File: hardware/turbofrank/turbofrank.kicad_pcb (KiCad board)
At the start: 2 copper layers, 99 x 99 mm, 201 parts, among them CON1 Pin Header 1x03, CON2 Pin Header 1x03, CON3 Pin Header 1x08, J1 Pin Header 2x18, Q1 BC850, Q2 BC850, Q3 BC850, SW1 KLS7-TS3302, SW2 KLS7-TS3302, SW3 KLS7-TS3302, U1 LM358, U2 JFC95101, U3 JFC95101, U4 74HC595, U5 74HC595, U6 74HC74, U7 NCP1117 3.3, X1 3.58 MHz

Commit message: Bugfixes
Connections:
- net /Zero/ZGPIO10 renamed /Zero/ZGPIO10_1
- net /Zero/ZGPIO26_1 renamed /Zero/ZGPIO26
- net /Zero/ZGPIO28 renamed /Zero/ZGPIO28_1
- net /Zero/ZGPIO29_1 renamed /Zero/ZGPIO29
- net /Zero/ZGPIO8 renamed /Zero/ZGPIO8_1
- net /Zero/ZGPIO9_1 renamed /Zero/ZGPIO9
- AJ2 pad T: /LOAD_IN_D -> Net-(AJ2-PadT)
- C29 pad 1: /LOAD_IN_D -> Net-(AJ2-PadT)
- R81 pad 1: /LOAD_IN_D -> Net-(AJ2-PadT)
Routing:
- net /LOAD_IN_D: track 94.1 -> 9.27 mm, vias 7 -> 0
- net VBUS: track 603.4 -> 596.9 mm
- net Net-(GP2-Pad2): track 26.1 -> 22.7 mm
- net /GPIO9: track 111.0 -> 108.1 mm
- net /GPIO28: track 127.4 -> 124.7 mm
- net /GPIO11: track 109.9 -> 107.5 mm
- net /GPIO27: track 123.8 -> 121.5 mm
- net /GPIO7: track 102.8 -> 100.4 mm
- net /GPIO6: track 99.4 -> 97.1 mm
- net /GPIO19: track 65.3 -> 63.1 mm
- net /GPIO12: track 92.0 -> 89.8 mm
- net /GPIO8: track 113.1 -> 111.0 mm
- net /GPIO17: track 55.5 -> 53.4 mm
- net /RUN: track 121.9 -> 119.8 mm
- net /GPIO0: track 122.7 -> 120.7 mm
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
Commit message: TurboFRANK HW 1.03
Parts:
- PSR1, TDA1: footprint FRANK:SOIC-8 -> FRANK:SO-8
Routing:
- net /LOAD_IN_D: track 9.27 -> 77.1 mm, vias 0 -> 7
- net Net-(AJ2-PadT): track 0.00 -> 34.8 mm, vias 0 -> 2
- net /KB_CLK: track 56.4 -> 60.6 mm
- net /A_TDAL: track 98.5 -> 101.9 mm
- net /RUN: track 119.8 -> 123.1 mm
- net /GPIO19: track 63.1 -> 65.6 mm
- net /GPIO0: track 120.7 -> 123.0 mm
- net /GPIO26: track 110.3 -> 112.4 mm
- net /RS232/C2-: track 20.3 -> 18.4 mm
- net VBUS: track 596.9 -> 598.1 mm
- net /MS_CLK: track 46.4 -> 47.3 mm
- net Net-(TDA1-FLT): track 46.4 -> 45.6 mm
- net +3V3: track 299.9 -> 300.7 mm
- net /GPIO20: track 14.6 -> 15.4 mm
- net /GP2_DATA: track 130.3 -> 130.9 mm
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Other:
- board text added: "HW Revision 1.03"
- board text removed: "HW Revision 1.02"

Commit message: TurboFRANK 1.04 WIP
Parts:
- removed AJ1, AJ2: SJ1-353XNG, FRANK:Jack (3.5mm)
- removed COM1, GP1, GP2: D-SUB 9 Male, FRANK:D-SUB (9 pin, male, top mount)
- removed CON1, CON2: Pin Header 1x03, FRANK:Pin Header (1x03)
- removed CON3: Pin Header 1x08, FRANK:Pin Header (1x08)
- removed HDMI1: DC3RX19JA2, FRANK:HDMI (female)
- removed KB1: MDC-036, FRANK:MiniDIN (6 Pin, female)
- removed L3: Green, FRANK:LED (0805)
- removed MAX1: MAX232CSE+, FRANK:SOIC127P600X175-16N
- removed PSR1: ESP-PSRAM32, FRANK:SO-8
- removed RP1: Rasberry Pi Pico, FRANK:Raspberry Pi Pico
- removed RP2: RP2040-Zero, FRANK:Raspberry Pi Zero
- removed SC1: RCA-103, FRANK:RCA
- removed SD1: 0475710001, FRANK:MicroSD (SMD, short)
- removed SD2: 104031-0811, FRANK:MicroSD (SMD, long)
- removed SW3: KLS7-TS3302, FRANK:Button (SMD, 3x3mm)
- removed TDA1: TDA1387T, FRANK:SO-8
- removed USB1: USB4215, FRANK:USB Type C
- removed USB2: SS-52100-004, FRANK:USB Type A (stacked)
- removed VGA1: D-SUB 15 Female, FRANK:D-SUB (15 pin, female)
- added C37: 10u, FRANK:Capacitor (0805), F.Cu at (50.7, 76.9)
- added C38: 10u, FRANK:Capacitor (0805), F.Cu at (50.7, 79.9)
- added C39: 10u, FRANK:Capacitor (0805), F.Cu at (50.7, 82.9)
- added C40: 10u, FRANK:Capacitor (0805), F.Cu at (-25.6, 135.8)
- added C41: 10u, FRANK:Capacitor (0805), F.Cu at (-25.6, 138.8)
- added C42: 100n, FRANK:Capacitor (0805), F.Cu at (-25.6, 141.8)
- added J10: DC3RX19JA2, FRANK:HDMI (female), F.Cu at (-4.30, 21.6)
- added J11: PAM L, FRANK:Connector Female ZH 1.50mm (2 pins), F.Cu at (31.6, 52.0)
- added J12: ~, FRANK:Jack (3.5mm, PJ-320D), F.Cu at (38.4, 44.2)
- added J13: PAM R, FRANK:Connector Female ZH 1.50mm (2 pins), F.Cu at (31.6, 57.6)
- added J14: ~, FRANK:Jack (3.5mm, PJ-320D), F.Cu at (20.3, 44.2)
- added J15: Rasberry Pi Pico, FRANK:Raspberry Pi Pico, F.Cu at (-77.2, 75.7)
- added J16: RP2040-Zero, FRANK:Raspberry Pi Zero, F.Cu at (-7.63, 55.9)
- added J17: SS-52100-004, FRANK:USB Type A (stacked), F.Cu at (46.8, 23.8)
- added J18: D-SUB 15 Female, FRANK:D-SUB (15 pin, female), F.Cu at (10.3, 75.1)
- added J19: Pin Header 1x08, FRANK:Pin Header (1x08), F.Cu at (-55.2, 130.3)
- added J2: Power, FRANK:Pin Header (1x03), F.Cu at (-1.06, 100.3)
- added J20: RCA-103, FRANK:RCA, F.Cu at (-72.9, 148.2)
- added J21: USB HUB Data, FRANK:Connector Female ZH 1.50mm (2 pins), F.Cu at (51.2, 100.3)
- added J22: D-SUB 9 Male, FRANK:D-SUB (9 pin, male, top mount), F.Cu at (-39.3, 76.2)
- added J3: USB4215, FRANK:USB Type C, F.Cu at (-44.9, 143.2)
- added J4: MDC-036, FRANK:MiniDIN (6 Pin, female), F.Cu at (-35.1, 111.0)
- added J5: 0475710001, FRANK:MicroSD (SMD, short), F.Cu at (45.6, 144.4)
- added J6: 104031-0811, FRANK:MicroSD (SMD, long), F.Cu at (47.3, 138.4)
- added J7: SS-52100-004, FRANK:USB Type A (stacked), F.Cu at (20.2, 23.8)
- added J8: D-SUB 9 Male, FRANK:D-SUB (9 pin, male, top mount), F.Cu at (14.2, 101.8)
- added J9: D-SUB 9 Male, FRANK:D-SUB (9 pin, male, top mount), F.Cu at (14.2, 125.7)
- added JP3: Jumper (Solder), FRANK:Jumper (solder), F.Cu at (-54.4, 74.2)
- added LD1: Green, FRANK:LED (0805), F.Cu at (-37.1, 141.9)
- added R110: 10K, FRANK:Resistor (0805), F.Cu at (-30.4, 135.8)
- added R111: 10K, FRANK:Resistor (0805), F.Cu at (-30.4, 138.8)
- added R112: 10K, FRANK:Resistor (0805), F.Cu at (-30.4, 141.7)
- added R113: 470R, FRANK:Resistor (0805), F.Cu at (-30.4, 144.7)
- added R114: 470R, FRANK:Resistor (0805), F.Cu at (-30.4, 147.6)
- added U10: PAM8403D, FRANK:SOIC127P600X175-16N, F.Cu at (43.0, 90.2)
- added U12: TDA1387T, FRANK:SO-8, F.Cu at (-23.8, 146.7)
- added U8: 74HC595, FRANK:SOP-16, F.Cu at (-30.5, 47.5)
- added U9: 74HC74, FRANK:74HCT74D, F.Cu at (-37.4, 64.7)
- C1, C2: value 100u -> 10u; footprint FRANK:Capacitor (3528, tantalum, polar) -> FRANK:Capacitor (0805)
- C11, C23, C8: value 10u -> 100n; footprint FRANK:Capacitor (3528, tantalum, polar) -> FRANK:Capacitor (0805)
- C12: footprint FRANK:Capacitor (3528, tantalum, polar) -> FRANK:Capacitor (0805)
- C13, C7: value 100n -> 10u; moved to F.Cu
- C14: value 22p -> 220u; footprint FRANK:Capacitor (0805) -> FRANK:Capacitor (3528, tantalum, polar)
- C15: value 22p -> 1u
- C16, C17: value 10u -> 1u
- C18, C28, C29: value 100n -> 1u
- C19, C20: value 100n -> 100u; footprint FRANK:Capacitor (0805) -> FRANK:Capacitor (3528, tantalum, polar)
- C21, C5, C6, L1, L2: moved to F.Cu
- C24: value 10n -> 22p
- C25: value 10u -> 22p; footprint FRANK:Capacitor (3528, tantalum, polar) -> FRANK:Capacitor (0805)
- C26: value 10u -> 47n; footprint FRANK:Capacitor (3528, tantalum, polar) -> FRANK:Capacitor (0805)
- C27: value 10n -> 47n
- C30: value 10u -> 100u; moved to F.Cu
- C31, C4: value 10u -> 100n; moved to F.Cu
- C32: value 220u -> 1u; footprint FRANK:Capacitor (3528, tantalum, polar) -> FRANK:Capacitor (0805)
- C33, C35, C36: value 1u -> 10u; moved to F.Cu
- C34: value 1u -> 100n; moved to F.Cu
- C9: value 10u -> 100n; footprint FRANK:Capacitor (3528, tantalum, polar) -> FRANK:Capacitor (0805); moved to F.Cu
- D1, D2: value 1N4148 -> 3V3; moved to F.Cu
- D7, D8: value 3V3 -> 1N4148
- J1: value Pin Header 2x18 -> UART; footprint FRANK:Pin Header (2x18) -> FRANK:Pin Header (1x03)
- JP1: value Jumper (Solder) -> Pin Header 2x18; footprint FRANK:Jumper (solder) -> FRANK:Pin Header (2x18)
- R1, R2: value 100K -> 5.1K; moved to F.Cu
- R10, R11, R5, R6: value 2K -> 100R; moved to F.Cu
- R100, R102, R104, R106, R98: value 270R -> 10K
- R101, R97, R99: value 150R -> 10K
- R103: value 150R -> 20K
- R105: value 150R -> 47K
- R107: value 300R -> 47K
- R108: value 1K -> 20K
- R109, R75, R89, R90: value 1K -> 10K
- R12, R13, R14: value 2K -> 22R; moved to F.Cu
- R15: value 10K -> 22R; moved to F.Cu
- R16: value 47K -> 1K; moved to F.Cu
- R17: value 120R -> 1K; moved to F.Cu
- R18, R24: value 1K -> 270R; moved to F.Cu
- R19, R53: value 1K -> 270R
- R20, R21: value 10K -> 270R
- R22: value 47K -> 270R
- R23: value 120R -> 270R; moved to F.Cu
- R25: value 2R -> 270R; moved to F.Cu
- R26: value 1K -> 10K; moved to F.Cu
- R27: value 1R -> 1K; moved to F.Cu
- R28, R29: value 1R -> 10K; moved to F.Cu
- R3, R4, R7, R8, R9: value 2K -> 1K; moved to F.Cu
- R30: value 1R -> 100R; moved to F.Cu
- R31, R32, R33: value 1R -> 22R; moved to F.Cu
- R34: value 2R -> 22R; moved to F.Cu
- R35, R36, R37: value 2R -> 330R; moved to F.Cu
- R38, R39, R40: value 2R -> 1K; moved to F.Cu
- R41: value 2R -> 100R; moved to F.Cu
- R42: value 1K -> 100R
- R43: value 10K -> 750R
- R44: value 10K -> 51R; moved to F.Cu
- R45, R47, R49: value 10K -> 270R; moved to F.Cu
- R46: value 100K -> 150R
- R48: value 10K -> 150R; moved to F.Cu
- R50: value 5.1K -> 150R
- R51: value 5.1K -> 270R
- R52: value 1K -> 150R; moved to F.Cu
- R54: value 100R -> 150R
- R55: value 100R -> 270R
- R56: value 1K -> 300R
- R59: value 100R -> 120R
- R60, R92, R93: value 100R -> 2K
- R61, R62, R71: value 1K -> 2K
- R63, R65, R66, R67, R68, R69, R70, R96: value 270R -> 2K
- R64: value 270R -> 120R
- R72, R87, R88: value 330R -> 2K
- R73, R74: value 2K -> 10K
- R76: value 330R -> 1K
- R77, R79: value 10K -> 1K
- R81: value 100R -> 10K
- R82, R83, R84: value 22R -> 10K
- R85: value 22R -> 1K; moved to F.Cu
- R86: value 330R -> 100K
- R94: value 750R -> 2K
- R95: value 51R -> 2K
- U1: value LM358 -> NCP1117 3.3; footprint FRANK:SO-8 -> FRANK:SOT-223; moved to F.Cu
- U2: value JFC95101 -> ESP-PSRAM32; footprint FRANK:DIP-40 -> FRANK:SOIC-8
- U3: value JFC95101 -> MW7211A; footprint FRANK:DIP-40 -> FRANK:SO-16
- U4: value 74HC595 -> MAX232CSE+; footprint FRANK:SOP-16 -> FRANK:SOIC127P600X175-16N; moved to F.Cu
- U5: value 74HC595 -> JFC95101; footprint FRANK:SOP-16 -> FRANK:DIP-40; moved to F.Cu
- U6: value 74HC74 -> JFC95101; footprint FRANK:74HCT74D -> FRANK:DIP-40; moved to F.Cu
- U7: value NCP1117 3.3 -> 74HC595; footprint FRANK:SOT-223 -> FRANK:SOP-16
- moved R52 275.5 mm to (-73.0, 141.2)
- moved R51 261.7 mm to (-73.0, 138.3)
- moved R50 258.1 mm to (-73.0, 135.3)
- moved R46 254.3 mm to (-77.7, 138.3)
- moved U6 246.0 mm to (-60.1, 20.1), turned to 0 degrees
- moved U5 242.4 mm to (-78.5, 20.1), turned to 0 degrees
- moved R61 239.8 mm to (-40.9, 25.4), turned to 0 degrees
- moved C14 237.1 mm to (-62.7, 130.1)
- moved R62 235.8 mm to (-40.9, 28.3), turned to 0 degrees
- moved C16 226.7 mm to (-47.8, 95.9)
- moved C17 226.7 mm to (-47.8, 98.9)
- moved R63 225.7 mm to (-40.9, 31.3), turned to 0 degrees
- moved C15 224.5 mm to (-47.8, 92.9), turned to 0 degrees
- moved R64 222.5 mm to (-40.9, 34.2), turned to 0 degrees
- moved R65 219.3 mm to (-40.9, 37.2), turned to 0 degrees
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Connections:
- C10 pad 1: /Audio Out/TurboSound/R_IN -> +3V3
- C10 pad 2: Net-(C10-Pad2) -> GND
- C11 pad 2: /A_TSR -> Net-(C11-Pad2)
- C12 pad 1: Net-(C10-Pad2) -> VBUS
- C12 pad 2: /Audio Out/TurboSound/R_IN -> GND
- C14 pad 1: GND -> Net-(C14-Pad1)
- C14 pad 2: Net-(Q1-C) -> /Composite/CVBS
- C15 pad 1: GND -> /RS232/V+
- C15 pad 2: Net-(Q1-B) -> VBUS
- C16 pad 1: VBUS -> /RS232/C1-
- C16 pad 2: GND -> /RS232/C1+
- C17 pad 1: +3V3 -> /RS232/C2-
- C17 pad 2: GND -> /RS232/C2+
- C18 pad 1: VBUS -> /RS232/V-
- C2 pad 1: VBUS -> +3V3
- C20 pad 1: GND -> VBUS
- C20 pad 2: +3V3 -> GND
- C22 pad 1: +3V3 -> VBUS
- C23 pad 1: Net-(C23-Pad1) -> VBUS
- C23 pad 2: /Audio Out/L -> GND
- C24 pad 1: Net-(C23-Pad1) -> GND
- C24 pad 2: GND -> Net-(Q3-C)
- C25 pad 1: Net-(TDA1-FLT) -> GND
- C25 pad 2: GND -> Net-(Q3-B)
- C26 pad 2: /Audio Out/R -> GND
- C27 pad 1: Net-(C26-Pad1) -> /GPIO28
- C28 pad 1: +3V3 -> VBUS
- C29 pad 1: Net-(AJ2-PadT) -> Net-(C29-Pad1)
- C31 pad 1: VBUS -> Net-(U10-VREF)
- C32 pad 2: /Composite/CVBS -> Net-(C32-Pad2)
- C33 pad 1: /RS232/V+ -> GND
- C34 pad 1: /RS232/C1- -> GND
- C34 pad 2: /RS232/C1+ -> VBUS
- C35 pad 1: /RS232/C2- -> /AMP_IN_L
- C35 pad 2: /RS232/C2+ -> Net-(C35-Pad2)
- C36 pad 1: /RS232/V- -> Net-(C36-Pad1)
- C36 pad 2: GND -> /Audio Out/AMP_OUTL
- C5 pad 1: VBUS -> GND
- C5 pad 2: GND -> +3V3
- C6 pad 1: Net-(U1A-+) -> VBUS
- C7 pad 1: /Audio Out/TurboSound/L_IN -> VBUS
- C7 pad 2: Net-(C7-Pad2) -> GND
- C8 pad 1: Net-(C8-Pad1) -> VBUS
- C8 pad 2: /A_TSL -> GND
- C9 pad 1: Net-(C7-Pad2) -> +3V3
- C9 pad 2: /Audio Out/TurboSound/L_IN -> GND
- D1 pad 1: Net-(D1-K) -> /GPIO0
- D1 pad 2: /Audio Out/TurboSound/YM_RST -> GND
- D10 pad 1: /RS232/CTS_MAX -> Net-(D10-K)
- D10 pad 2: /RS232_CTS -> /Audio Out/TS/YM_RST
- D11 pad 1: /RS232/RX_MAX -> Net-(D11-K)
- D11 pad 2: /RS232_RX -> /Audio Out/TS/YM_RST
- D2 pad 1: Net-(D2-K) -> /GPIO1
- D2 pad 2: /Audio Out/TurboSound/YM_RST -> GND
- D3 pad 1: /GPIO0 -> /MS_DATA_3V
- D4 pad 1: /GPIO1 -> /MS_CLK_3V
- D5 pad 1: /MS_DATA_3V -> /GP1_DATA
- D6 pad 1: /MS_CLK_3V -> /GP2_DATA
- D7 pad 1: /GP1_DATA -> Net-(D7-K)
- D7 pad 2: GND -> Net-(D7-A)
- D8 pad 1: /GP2_DATA -> /RS232/CTS_MAX
- D8 pad 2: GND -> /RS232_CTS
- D9 pad 1: Net-(D9-K) -> /RS232/RX_MAX
- D9 pad 2: Net-(D9-A) -> /RS232_RX
- J1 pad 1: /A_OUTL -> GND
- J1 pad 2: /GPIO27 -> /GPIO0
- J1 pad 3: /A_OUTR -> /GPIO1
- JP1 pad 1: Net-(JP1-A) -> /PWM_OUT_L
- JP1 pad 2: /PSR_SOSIO -> /AMP_IN_L
- JP2 pad 2: +3V3 -> /PSR_SOSIO
- L1 pad 2: /Audio Out/TurboSound/YM_CS1 -> /Audio Out/TS/YM_CS1
- L2 pad 2: /Audio Out/TurboSound/YM_CS2 -> /Audio Out/TS/YM_CS2
- Q1 pad 3: Net-(Q1-C) -> /LOAD_IN_D
- Q2 pad 1: Net-(Q2-B) -> Net-(D7-K)
- Q2 pad 3: /LOAD_IN_D -> Net-(D7-A)
- Q3 pad 1: Net-(D9-K) -> Net-(Q3-B)
- Q3 pad 3: Net-(D9-A) -> Net-(Q3-C)
- R1 pad 1: VBUS -> GND
- R1 pad 2: Net-(U1A-+) -> Net-(J3-CC1)
- R10 pad 1: /Audio Out/TurboSound/L_IN -> /MS_DATA
- R10 pad 2: /Audio Out/TurboSound/A2 -> /MS_DATA_3V
- R100 pad 1: /GPIO11 -> /AMP_IN_L
- R100 pad 2: Net-(R100-Pad2) -> Net-(C29-Pad1)
- R101 pad 1: Net-(R101-Pad1) -> /AMP_IN_R
- R101 pad 2: Net-(R100-Pad2) -> Net-(C32-Pad1)
- R102 pad 1: /GPIO10 -> Net-(U11A-+)
- R102 pad 2: Net-(R101-Pad1) -> VBUS
- R103 pad 1: Net-(R103-Pad1) -> GND
- R103 pad 2: Net-(R101-Pad1) -> /Audio Out/AMP_OUTL
- R104 pad 1: /GPIO7 -> Net-(U11B--)
- R104 pad 2: Net-(R103-Pad1) -> Net-(C35-Pad2)
- R105 pad 1: Net-(R105-Pad1) -> Net-(C36-Pad1)
- R105 pad 2: Net-(R103-Pad1) -> Net-(U11B--)
- R106 pad 1: /GPIO6 -> Net-(U11A--)
- R106 pad 2: Net-(R105-Pad1) -> Net-(C37-Pad2)
- R107 pad 1: GND -> Net-(C38-Pad1)
- R107 pad 2: Net-(R105-Pad1) -> Net-(U11A--)
- R108 pad 1: /RS232_CTS -> GND
- R108 pad 2: +3V3 -> /Audio Out/AMP_OUTR
- R109 pad 1: /RS232_RX -> GND
- R109 pad 2: +3V3 -> Net-(U11A-+)
- R11 pad 1: /Audio Out/TurboSound/R_IN -> /MS_CLK
- R11 pad 2: /Audio Out/TurboSound/C1 -> /MS_CLK_3V
- R12 pad 1: /Audio Out/TurboSound/R_IN -> /UH_DP1
- R12 pad 2: /Audio Out/TurboSound/C2 -> Net-(J7-D1+)
- R13 pad 1: /Audio Out/TurboSound/L_IN -> /UH_DP2
- R13 pad 2: /Audio Out/TurboSound/C1 -> Net-(J7-D2+)
- R14 pad 1: /Audio Out/TurboSound/L_IN -> /UH_DM1
- R14 pad 2: /Audio Out/TurboSound/C2 -> Net-(J7-D1-)
- R15 pad 1: Net-(U1A--) -> /UH_DM2
- R15 pad 2: Net-(C7-Pad2) -> Net-(J7-D2-)
- R16 pad 1: Net-(C8-Pad1) -> /GP1_DATA
- R16 pad 2: Net-(U1A--) -> Net-(J8-Pad2)
- R17 pad 1: /Audio Out/TurboSound/L_IN -> /GP2_DATA
- R17 pad 2: GND -> Net-(J9-Pad2)
- R18 pad 1: VBUS -> Net-(J10-CLKN)
- R18 pad 2: /Audio Out/TurboSound/YM_SEL1 -> /GPIO6
- R19 pad 1: VBUS -> Net-(J10-CLKP)
- R19 pad 2: /Audio Out/TurboSound/YM_SEL2 -> /GPIO7
- R2 pad 1: Net-(U1A-+) -> GND
- R2 pad 2: GND -> Net-(J3-CC2)
- R20 pad 1: /Audio Out/TurboSound/YM_RST -> Net-(J10-D0N)
- R20 pad 2: VBUS -> /GPIO8
- R21 pad 1: Net-(U1B--) -> Net-(J10-D0P)
- R21 pad 2: Net-(C10-Pad2) -> /GPIO9
- R22 pad 1: Net-(C11-Pad1) -> Net-(J10-D1N)
- R22 pad 2: Net-(U1B--) -> /GPIO10
- R23 pad 1: /Audio Out/TurboSound/R_IN -> Net-(J10-D1P)
- R23 pad 2: GND -> /GPIO11
- R24 pad 1: GND -> Net-(J10-D2N)
- R24 pad 2: Net-(L1-K) -> /GPIO12
- R25 pad 1: GND -> Net-(J10-D2P)
- R25 pad 2: Net-(R25-Pad2) -> /GPIO13
- R26 pad 1: GND -> +3V3
- R26 pad 2: Net-(L2-K) -> Net-(D7-A)
- R27 pad 1: Net-(R25-Pad2) -> +3V3
- R27 pad 2: Net-(R27-Pad2) -> /LOAD_IN_D
- R28 pad 1: Net-(R27-Pad2) -> Net-(D7-A)
- R28 pad 2: Net-(R28-Pad2) -> Net-(Q1-B)
- R29 pad 1: Net-(R28-Pad2) -> Net-(C11-Pad2)
- R29 pad 2: Net-(R29-Pad2) -> Net-(D7-K)
- R3 pad 1: /Audio Out/TurboSound/R_IN -> Net-(LD1-A)
- R3 pad 2: /Audio Out/TurboSound/B1 -> +3V3
- R30 pad 1: Net-(R29-Pad2) -> Net-(C11-Pad1)
- R30 pad 2: Net-(R30-Pad2) -> GND
- R31 pad 1: Net-(R30-Pad2) -> /USB_D1P
- R31 pad 2: Net-(R31-Pad2) -> Net-(J17-D1+)
- R32 pad 1: Net-(R31-Pad2) -> /USB_D2P
- R32 pad 2: Net-(R32-Pad2) -> Net-(J17-D2+)
- R33 pad 1: Net-(R32-Pad2) -> /USB_D1M
- R33 pad 2: /Audio Out/TurboSound/COVOX_OUT -> Net-(J17-D1-)
- R34 pad 1: Net-(R25-Pad2) -> /USB_D2M
- R34 pad 2: /Audio Out/TurboSound/DAC0 -> Net-(J17-D2-)
- R35 pad 1: Net-(R27-Pad2) -> /GPIO11
- R35 pad 2: /Audio Out/TurboSound/DAC1 -> Net-(J18-Pad1)
- R36 pad 1: Net-(R28-Pad2) -> /GPIO9
- R36 pad 2: /Audio Out/TurboSound/DAC2 -> Net-(J18-Pad2)
- R37 pad 1: Net-(R29-Pad2) -> /GPIO7
- R37 pad 2: /Audio Out/TurboSound/DAC3 -> Net-(J18-Pad3)
- R38 pad 1: Net-(R30-Pad2) -> /GPIO10
- R38 pad 2: /Audio Out/TurboSound/DAC4 -> Net-(J18-Pad1)
- R39 pad 1: Net-(R31-Pad2) -> /GPIO8
- R39 pad 2: /Audio Out/TurboSound/DAC5 -> Net-(J18-Pad2)
- R4 pad 1: /Audio Out/TurboSound/R_IN -> VBUS
- R4 pad 2: /Audio Out/TurboSound/B2 -> /KB_CLK
- R40 pad 1: Net-(R32-Pad2) -> /GPIO6
- R40 pad 2: /Audio Out/TurboSound/DAC6 -> Net-(J18-Pad3)
- R41 pad 1: /Audio Out/TurboSound/COVOX_OUT -> Net-(J18-Pad13)
- R41 pad 2: /Audio Out/TurboSound/DAC7 -> /GPIO12
- R42 pad 1: Net-(Q1-C) -> Net-(J18-Pad14)
- R42 pad 2: VBUS -> /GPIO13
- R43 pad 1: /Audio Out/TurboSound/R_IN -> /GPIO12
- R43 pad 2: /Audio Out/TurboSound/COVOX_OUT -> Net-(R43-Pad2)
- R44 pad 1: /Audio Out/TurboSound/L_IN -> Net-(R43-Pad2)
- R44 pad 2: /Audio Out/TurboSound/COVOX_OUT -> Net-(C14-Pad1)
- R45 pad 1: /Audio Out/TurboSound/R_IN -> /GPIO9
- R45 pad 2: /Audio Out/TurboSound/BEEP -> Net-(R43-Pad2)
- R46 pad 1: Net-(Q1-B) -> Net-(R46-Pad1)
- R46 pad 2: Net-(Q1-C) -> Net-(R43-Pad2)
- R47 pad 1: /Audio Out/TurboSound/L_IN -> /GPIO8
- R47 pad 2: /Audio Out/TurboSound/BEEP -> Net-(R46-Pad1)
- R48 pad 1: /Audio Out/TurboSound/R_IN -> Net-(R48-Pad1)
- R48 pad 2: /Audio Out/TurboSound/SAVE -> Net-(R46-Pad1)
- R49 pad 1: /Audio Out/TurboSound/L_IN -> /GPIO11
- R49 pad 2: /Audio Out/TurboSound/SAVE -> Net-(R48-Pad1)
- R5 pad 1: /Audio Out/TurboSound/L_IN -> /KB_CLK
- R5 pad 2: /Audio Out/TurboSound/B1 -> /GPIO0
- R50 pad 1: GND -> Net-(R50-Pad1)
- R50 pad 2: Net-(USB1-CC1) -> Net-(R48-Pad1)
- R51 pad 1: GND -> /GPIO10
- R51 pad 2: Net-(USB1-CC2) -> Net-(R50-Pad1)
- R52 pad 1: Net-(L3-A) -> Net-(R52-Pad1)
- R52 pad 2: +3V3 -> Net-(R50-Pad1)
- R53 pad 1: VBUS -> /GPIO7
- R53 pad 2: /KB_CLK -> Net-(R52-Pad1)
- R54 pad 1: /KB_CLK -> Net-(R54-Pad1)
- R54 pad 2: /GPIO0 -> Net-(R52-Pad1)
- R55 pad 1: /KB_DATA -> /GPIO6
- R55 pad 2: /GPIO1 -> Net-(R54-Pad1)
- R56 pad 1: VBUS -> GND
- R56 pad 2: /KB_DATA -> Net-(R54-Pad1)
- R57 pad 1: VBUS -> /RS232_CTS
- R57 pad 2: /MS_DATA -> +3V3
- R58 pad 1: VBUS -> /RS232_RX
- R58 pad 2: /MS_CLK -> +3V3
- R59 pad 1: /MS_DATA -> /TS_L
- R59 pad 2: /MS_DATA_3V -> GND
- R6 pad 1: /Audio Out/TurboSound/L_IN -> /KB_DATA
- R6 pad 2: /Audio Out/TurboSound/B2 -> /GPIO1
- R60 pad 1: /MS_CLK -> /TS_R
- R60 pad 2: /MS_CLK_3V -> /Audio Out/TS/B1
- R61 pad 1: /GP1_DATA -> /TS_R
- R61 pad 2: Net-(GP1-Pad2) -> /Audio Out/TS/B2
- R62 pad 1: /GP2_DATA -> /TS_L
- R62 pad 2: Net-(GP2-Pad2) -> /Audio Out/TS/B1
- R63 pad 1: Net-(HDMI1-CLKN) -> /TS_L
- R63 pad 2: /GPIO6 -> /Audio Out/TS/B2
- R64 pad 1: Net-(HDMI1-CLKP) -> /TS_R
- R64 pad 2: /GPIO7 -> GND
- R65 pad 1: Net-(HDMI1-D0N) -> /TS_R
- R65 pad 2: /GPIO8 -> /Audio Out/TS/A1
- R66 pad 1: Net-(HDMI1-D0P) -> /TS_R
- R66 pad 2: /GPIO9 -> /Audio Out/TS/A2
- R67 pad 1: Net-(HDMI1-D1N) -> /TS_L
- R67 pad 2: /GPIO10 -> /Audio Out/TS/A1
- R68 pad 1: Net-(HDMI1-D1P) -> /TS_L
- R68 pad 2: /GPIO11 -> /Audio Out/TS/A2
- R69 pad 1: Net-(HDMI1-D2N) -> /TS_R
- R69 pad 2: /GPIO12 -> /Audio Out/TS/C1
- R7 pad 1: /Audio Out/TurboSound/R_IN -> VBUS
- R7 pad 2: /Audio Out/TurboSound/A1 -> /KB_DATA
- R70 pad 1: Net-(HDMI1-D2P) -> /TS_R
- R70 pad 2: /GPIO13 -> /Audio Out/TS/C2
- R71 pad 1: Net-(C23-Pad1) -> /TS_L
- R71 pad 2: /A_OUTL -> /Audio Out/TS/C1
- R72 pad 1: /Audio Out/L -> /TS_L
- R72 pad 2: GND -> /Audio Out/TS/C2
- R73 pad 1: Net-(C23-Pad1) -> GND
- R73 pad 2: /A_OUTB -> /GPIO28
- R74 pad 1: Net-(C26-Pad1) -> GND
- R74 pad 2: /A_OUTB -> /GPIO27
- R75 pad 1: Net-(C26-Pad1) -> GND
- R75 pad 2: /A_OUTR -> /GPIO26
- R76 pad 1: /Audio Out/R -> GND
- R76 pad 2: GND -> Net-(L1-K)
- R77 pad 1: +3V3 -> GND
- R77 pad 2: Net-(D9-A) -> Net-(L2-K)
- R78 pad 1: +3V3 -> VBUS
- R78 pad 2: /LOAD_IN_D -> /Audio Out/TS/YM_SEL1
- R79 pad 1: Net-(D9-A) -> VBUS
- R79 pad 2: Net-(Q2-B) -> /Audio Out/TS/YM_SEL2
- R8 pad 1: /Audio Out/TurboSound/R_IN -> VBUS
- R8 pad 2: /Audio Out/TurboSound/A2 -> /MS_DATA
- R80 pad 1: Net-(C29-Pad2) -> /Audio Out/TS/YM_RST
- R80 pad 2: Net-(D9-K) -> VBUS
- R81 pad 1: Net-(AJ2-PadT) -> /TS_R
- R81 pad 2: GND -> /Audio Out/TS/BEEP
- R82 pad 1: /USB_D1P -> /TS_L
- R82 pad 2: Net-(USB2-D1+) -> /Audio Out/TS/BEEP
- R83 pad 1: /USB_D2P -> /TS_R
- R83 pad 2: Net-(USB2-D2+) -> /Audio Out/TS/SAVE
- R84 pad 1: /USB_D1M -> /TS_L
- R84 pad 2: Net-(USB2-D1-) -> /Audio Out/TS/SAVE
- R85 pad 1: /USB_D2M -> Net-(Q3-C)
- R85 pad 2: Net-(USB2-D2-) -> VBUS
- R86 pad 1: /GPIO11 -> Net-(Q3-B)
- R86 pad 2: Net-(R86-Pad2) -> Net-(Q3-C)
- R87 pad 1: /GPIO9 -> Net-(R87-Pad1)
- R87 pad 2: Net-(R87-Pad2) -> Net-(C26-Pad1)
- R88 pad 1: /GPIO7 -> Net-(R87-Pad1)
- R88 pad 2: Net-(R88-Pad2) -> /GPIO28
- R89 pad 1: /GPIO10 -> Net-(C26-Pad1)
- R89 pad 2: Net-(R86-Pad2) -> /PWM_OUT_R
- R9 pad 1: /Audio Out/TurboSound/L_IN -> VBUS
- R9 pad 2: /Audio Out/TurboSound/A1 -> /MS_CLK
- R90 pad 1: /GPIO8 -> /GPIO28
- R90 pad 2: Net-(R87-Pad2) -> /PWM_OUT_L
- R91 pad 1: /GPIO6 -> /GPIO28
- R91 pad 2: Net-(R88-Pad2) -> /GPIO27
- R92 pad 1: Net-(R92-Pad1) -> Net-(C26-Pad1)
- R92 pad 2: /GPIO12 -> /GPIO26
- R93 pad 1: Net-(R93-Pad1) -> /PWM_OUT_R
- R93 pad 2: /GPIO13 -> GND
- R94 pad 1: /GPIO12 -> /PWM_OUT_L
- R94 pad 2: Net-(R94-Pad2) -> GND
- R95 pad 1: Net-(R94-Pad2) -> Net-(C29-Pad1)
- R95 pad 2: Net-(C32-Pad1) -> GND
- R96 pad 1: /GPIO9 -> Net-(C32-Pad1)
- R96 pad 2: Net-(R94-Pad2) -> GND
- R97 pad 1: Net-(R97-Pad1) -> Net-(U10-INL)
- R97 pad 2: Net-(R94-Pad2) -> Net-(C29-Pad2)
- R98 pad 1: /GPIO8 -> VBUS
- R98 pad 2: Net-(R97-Pad1) -> /SHND
- R99 pad 1: Net-(R100-Pad2) -> Net-(U10-INR)
- R99 pad 2: Net-(R97-Pad1) -> Net-(C32-Pad2)
- SW1 pad 1: Net-(D1-K) -> Net-(D10-K)
- SW2 pad 1: Net-(D1-K) -> Net-(D10-K)
- U1 pad 1: Net-(C8-Pad1) -> GND
- U1 pad 2: Net-(U1A--) -> +3V3
- U1 pad 3: Net-(U1A-+) -> VBUS
- U2 pad 1: GND -> /GPIO18
- U2 pad 2: unconnected-(U2-NC-Pad2) -> Net-(JP2-A)
- U2 pad 3: /Audio Out/TurboSound/B1 -> unconnected-(U2-SIO2-Pad3)
- U2 pad 4: /Audio Out/TurboSound/A1 -> GND
- U2 pad 5: unconnected-(U2-NC-Pad5) -> /GPIO20
- U2 pad 6: unconnected-(U2-IOB7-Pad6) -> /GPIO19
- U2 pad 8: unconnected-(U2-IOB5-Pad8) -> +3V3
- U3 pad 1: GND -> /UH_DM4
- U3 pad 10: /Audio Out/TurboSound/DAC3 -> /USB Hub/DM_IN
- U3 pad 11: /Audio Out/TurboSound/DAC2 -> /USB Hub/DP_IN
- U3 pad 12: /Audio Out/TurboSound/DAC1 -> Net-(U3-VD3)
- U3 pad 13: /Audio Out/TurboSound/DAC0 -> VBUS
- U3 pad 14: unconnected-(U3-IOA7-Pad14) -> Net-(U3-VD3)
- U3 pad 15: unconnected-(U3-IOA6-Pad15) -> GND
- U3 pad 16: unconnected-(U3-IOA5-Pad16) -> GND
- U3 pad 2: unconnected-(U3-NC-Pad2) -> /UH_DP4
- U3 pad 3: /Audio Out/TurboSound/B2 -> /UH_DM3
- U3 pad 4: /Audio Out/TurboSound/A2 -> /UH_DP3
- U3 pad 5: unconnected-(U3-NC-Pad5) -> /UH_DM2
- U3 pad 6: /Audio Out/TurboSound/DAC7 -> /UH_DP2
- U3 pad 7: /Audio Out/TurboSound/DAC6 -> /UH_DM1
- U3 pad 8: /Audio Out/TurboSound/DAC5 -> /UH_DP1
- U3 pad 9: /Audio Out/TurboSound/DAC4 -> unconnected-(U3-LED-Pad9)
- U4 pad 1: /Audio Out/TurboSound/DA1 -> /RS232/C1+
- U4 pad 10: VBUS -> /RS232_RTS
- U4 pad 11: /GPIO27 -> /RS232_TX
- U4 pad 12: /GPIO26 -> /RS232/RX_MAX
- U4 pad 13: GND -> /RS232/TX_IN
- U4 pad 14: /GPIO28 -> /RS232/RX_IN
- U4 pad 15: /Audio Out/TurboSound/DA0 -> GND
- U4 pad 2: /Audio Out/TurboSound/DA2 -> /RS232/V+
- U4 pad 3: /Audio Out/TurboSound/DA3 -> /RS232/C1-
- U4 pad 4: /Audio Out/TurboSound/DA4 -> /RS232/C2+
- U4 pad 5: /Audio Out/TurboSound/DA5 -> /RS232/C2-
- U4 pad 6: /Audio Out/TurboSound/DA6 -> /RS232/V-
- U4 pad 7: /Audio Out/TurboSound/DA7 -> /RS232/CTS_IN
- U4 pad 8: GND -> /RS232/RTS_IN
- U4 pad 9: Net-(U4-QH') -> /RS232/CTS_MAX
- U5 pad 1: /Audio Out/TurboSound/YM_BDIR -> GND
- U5 pad 10: VBUS -> unconnected-(U5-IOB3-Pad10)
- U5 pad 11: /GPIO27 -> unconnected-(U5-IOB2-Pad11)
- U5 pad 12: /GPIO26 -> unconnected-(U5-IOB1-Pad12)
- U5 pad 13: GND -> unconnected-(U5-IOB0-Pad13)
- U5 pad 14: Net-(U4-QH') -> unconnected-(U5-IOA7-Pad14)
- U5 pad 15: /Audio Out/TurboSound/YM_BC1 -> unconnected-(U5-IOA6-Pad15)
- U5 pad 16: VBUS -> unconnected-(U5-IOA5-Pad16)
- U5 pad 2: /Audio Out/TurboSound/YM_CS1 -> unconnected-(U5-NC-Pad2)
- U5 pad 3: /Audio Out/TurboSound/YM_CS2 -> /Audio Out/TS/B1
- U5 pad 4: /Audio Out/TurboSound/BEEP -> /Audio Out/TS/A1
- U5 pad 5: /Audio Out/TurboSound/SAVE -> unconnected-(U5-NC-Pad5)
- U5 pad 6: Net-(D2-K) -> unconnected-(U5-IOB7-Pad6)
- U5 pad 8: GND -> unconnected-(U5-IOB5-Pad8)
- U6 pad 1: VBUS -> GND
- U6 pad 10: (no net) -> unconnected-(U6-IOB3-Pad10)
- U6 pad 11: (no net) -> unconnected-(U6-IOB2-Pad11)
- U6 pad 12: (no net) -> unconnected-(U6-IOB1-Pad12)
- U6 pad 13: (no net) -> unconnected-(U6-IOB0-Pad13)
- U6 pad 14: VBUS -> unconnected-(U6-IOA7-Pad14)
- U6 pad 2: Net-(U6A-D) -> unconnected-(U6-NC-Pad2)
- U6 pad 3: Net-(Q1-C) -> /Audio Out/TS/B2
- U6 pad 4: VBUS -> /Audio Out/TS/A2
- U6 pad 5: /Audio Out/TurboSound/CLK_1.75M -> unconnected-(U6-NC-Pad5)
- U6 pad 6: Net-(U6A-D) -> unconnected-(U6-IOB7-Pad6)
- U6 pad 7: GND -> unconnected-(U6-IOB6-Pad7)
- U6 pad 8: (no net) -> unconnected-(U6-IOB5-Pad8)
- U6 pad 9: (no net) -> unconnected-(U6-IOB4-Pad9)
- U7 pad 1: GND -> /Audio Out/TS/DA1
- U7 pad 2: +3V3 -> /Audio Out/TS/DA2
- U7 pad 3: VBUS -> /Audio Out/TS/DA3
- X1 pad 1: Net-(Q1-B) -> Net-(Q3-B)
- X1 pad 2: Net-(Q1-C) -> Net-(Q3-C)
Routing:
- net VBUS: track 598.1 -> 0.00 mm, vias 1 -> 0
- net +3V3: track 300.7 -> 0.00 mm, vias 7 -> 0
- net /GPIO15: track 182.6 -> 0.00 mm, vias 8 -> 0
- net /GPIO14: track 154.6 -> 0.00 mm, vias 8 -> 0
- net /Audio Out/TurboSound/R_IN: track 149.5 -> 0.00 mm, vias 3 -> 0
- net /A_OUTB: track 145.9 -> 0.00 mm, vias 8 -> 0
- net /GPIO1: track 134.9 -> 0.00 mm, vias 6 -> 0
- net /GP2_DATA: track 130.9 -> 0.00 mm, vias 4 -> 0
- net /GPIO28: track 125.2 -> 0.00 mm, vias 2 -> 0
- net /RUN: track 123.1 -> 0.00 mm, vias 8 -> 0
- net /GPIO0: track 123.0 -> 0.00 mm, vias 7 -> 0
- net /GPIO27: track 121.3 -> 0.00 mm, vias 2 -> 0
- net /Audio Out/TurboSound/DA4: track 116.6 -> 0.00 mm, vias 6 -> 0
- net /GPIO26: track 112.4 -> 0.00 mm, vias 4 -> 0
- net /GPIO8: track 111.0 -> 0.00 mm, vias 4 -> 0
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- removed copper zone on B.Cu, net GND
- removed copper zone on F.Cu, net GND
Other:
- board text removed: "+5V"
- board text removed: "3"
- board text removed: "5"
- board text removed: "Audio In"
- board text removed: "Audio Out"
- board text removed: "BL"
- board text removed: "BP"
- board text removed: "CS"
- board text removed: "CTS"
- board text removed: "DC"
- board text removed: "G"
- board text removed: "GND"
- board text removed: "GP1"
- board text removed: "GP2"
- board text removed: "Gamepad 1"
- board text removed: "Gamepad 2"
- board text removed: "HDMI"
- board text removed: "HW Revision 1.03"
- board text removed: "IL"
- board text removed: "IR"
- board text removed: "MS"
- board text removed: "MicroSD Card"
- board text removed: "PL"
- board text removed: "PR"
- board text removed: "PS/2"
- board text removed: "PSR"
- board text removed: "Pi Pico"
- board text removed: "RP2040-Zero"
- board text removed: "RS232"
- board text removed: "RST"
- board text removed: "RTS"
- board text removed: "RX"
- board text removed: "Reset"
- board text removed: "SCL"
- board text removed: "SDA"
- board text removed: "Soft Composite"
- board text removed: "TAPE"
- board text removed: "TL"
- board text removed: "TR"
- board text removed: "TURBO"
- board text removed: "TX"
- board text removed: "USB KB/Mouse"
- board text removed: "USB Power"
- board text removed: "VGA"
- board text removed: "ZERO"
- board text removed: "rh1.tech"

Commit message: TurboFRANK 1.04 WIP
Parts:
- removed C4: 100n, FRANK:Capacitor (0805)
- removed R109, R110, R111, R112: 10K, FRANK:Resistor (0805)
- removed R113, R114: 470R, FRANK:Resistor (0805)
- added C43: 4.7u, FRANK:Capacitor (0805), B.Cu at (178.0, 107.5)
- added J23: D-SUB 9 Male, FRANK:D-SUB (9 pin, male, top mount), F.Cu at (96.4, 101.9)
- added U11: LM358, FRANK:SO-8, B.Cu at (170.1, 79.8)
- C12, C13, C15, C16, C17, C18, C21, C22, C23, C24, C25, C26, C27, C28, C29, C3, C30, C31, C32, C33, C34, C35, C36, C37, C38, C39, C40, C41, C42, C6, C7, D10, D11, D5, D6, D8, D9, Q3, R101, R106, R12, R13, R14, R15, R16, R17, R57, R58, R59, R60, R61, R62, R63, R67, R69, R70, R71, R72, R76, R80, R81, R92, R93, R97, R98, R99, U10, U12, U3, U4, U7, U8, U9: moved to B.Cu
- J14: value ~ -> Mono; footprint FRANK:Jack (3.5mm, PJ-320D) -> FRANK:Pin Header (1x02)
- J15: value Rasberry Pi Pico -> ~; footprint FRANK:Raspberry Pi Pico -> FRANK:Jack (3.5mm, PJ-320D)
- J16: value RP2040-Zero -> Rasberry Pi Pico; footprint FRANK:Raspberry Pi Zero -> FRANK:Raspberry Pi Pico
- J17: value SS-52100-004 -> RP2040-Zero; footprint FRANK:USB Type A (stacked) -> FRANK:Raspberry Pi Zero
- J18: value D-SUB 15 Female -> SS-52100-004; footprint FRANK:D-SUB (15 pin, female) -> FRANK:USB Type A (stacked)
- J19: value Pin Header 1x08 -> D-SUB 15 Female; footprint FRANK:Pin Header (1x08) -> FRANK:D-SUB (15 pin, female)
- J20: value RCA-103 -> Pin Header 1x08; footprint FRANK:RCA -> FRANK:Pin Header (1x08)
- J21: value USB HUB Data -> RCA-103; footprint FRANK:Connector Female ZH 1.50mm (2 pins) -> FRANK:RCA
- J22: value D-SUB 9 Male -> USB HUB Data; footprint FRANK:D-SUB (9 pin, male, top mount) -> FRANK:Connector Female ZH 1.50mm (2 pins)
- R100: value 10K -> 20K; moved to B.Cu
- R102, R104: value 10K -> 47K; moved to B.Cu
- R103: value 20K -> 10K; moved to B.Cu
- R105: value 47K -> 20K; moved to B.Cu
- R107: value 47K -> 470R; moved to B.Cu
- R108: value 20K -> 470R
- R64: value 120R -> 2K
- R68: value 2K -> 120R; moved to B.Cu
- R73, R74: value 10K -> 1K
- R75, R82: value 10K -> 1K; moved to B.Cu
- R77: value 1K -> 10K; moved to B.Cu
- R78, R79: value 1K -> 10K
- R83: value 10K -> 100K; moved to B.Cu
- R84, R89, R90: value 10K -> 2K; moved to B.Cu
- R85, R91: value 1K -> 2K; moved to B.Cu
- R86: value 100K -> 10K; moved to B.Cu
- R87, R94, R95, R96: value 2K -> 10K; moved to B.Cu
- R88: value 2K -> 1K; moved to B.Cu
- U2: footprint FRANK:SOIC-8 -> FRANK:SO-8
- moved J15 259.7 mm to (181.3, 100.2), turned to 180 degrees
- moved J3 247.0 mm to (189.0, 63.8), turned to 90 degrees
- moved U1 232.5 mm to (170.2, 61.0), turned to 180 degrees
- moved LD1 232.2 mm to (183.8, 70.2), turned to 180 degrees
- moved R2 230.9 mm to (177.0, 64.0)
- moved R3 230.9 mm to (178.2, 70.2), turned to 180 degrees
- moved R1 228.7 mm to (177.0, 67.2)
- moved C1 227.8 mm to (177.0, 58.2)
- moved JP3 227.7 mm to (173.2, 69.1), turned to 90 degrees
- moved J20 223.6 mm to (130.3, 55.0)
- moved J19 217.1 mm to (143.3, 42.3), turned to 180 degrees
- moved R47 217.0 mm to (125.0, 63.8), turned to 180 degrees
- moved C2 215.8 mm to (163.0, 58.2), turned to 180 degrees
- moved U5 215.0 mm to (114.4, 115.0), turned to 90 degrees
- moved R43 214.1 mm to (125.0, 60.8), turned to 180 degrees
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Connections:
- C27 pad 1: /GPIO28 -> Net-(C27-Pad1)
- C29 pad 1: Net-(C29-Pad1) -> /AMP_IN_L
- C32 pad 1: Net-(C32-Pad1) -> /AMP_IN_R
- J16 pad 1: /Zero/ZGPIO0_1 -> /GPIO0
- J16 pad 10: /Zero/ZGPIO9_1 -> /GPIO7
- J16 pad 11: /Zero/ZGPIO10_1 -> /GPIO8
- J16 pad 12: /KB_DATA -> /GPIO9
- J16 pad 13: /KB_CLK -> GND
- J16 pad 14: /Zero/ZGPIO13_1 -> /GPIO10
- J16 pad 15: /MS_DATA -> /GPIO11
- J16 pad 16: /MS_CLK -> /GPIO12
- J16 pad 17: /Zero/ZGPIO26_1 -> /GPIO13
- J16 pad 18: /Zero/ZGPIO27 -> GND
- J16 pad 19: /Zero/ZGPIO28 -> /GPIO14
- J16 pad 2: /Zero/ZGPIO1 -> /GPIO1
- J16 pad 20: /Zero/ZGPIO29 -> /GPIO15
- J16 pad 21: unconnected-(J16-3V3-Pad21)_1 -> /GPIO16
- J16 pad 22: GND -> /GPIO17
- J16 pad 23: /ZERO_VBUS -> GND
- J16 pad 3: /USB_D1P -> GND
- J16 pad 4: /USB_D1M -> /GPIO2
- J16 pad 5: /USB_D2P -> /GPIO3
- J16 pad 6: /USB_D2M -> /GPIO4
- J16 pad 7: /Zero/ZGPIO6 -> /GPIO5
- J16 pad 8: /Zero/ZGPIO7_1 -> GND
- J16 pad 9: /Zero/ZGPIO8 -> /GPIO6
- J17 pad 1: VBUS -> /Zero/ZGPIO0
- J17 pad 2: Net-(J17-D1-) -> /Zero/ZGPIO1
- J17 pad 3: Net-(J17-D1+) -> /USB_D1P
- J17 pad 4: GND -> /USB_D1M
- J17 pad 5: VBUS -> /USB_D2P
- J17 pad 6: Net-(J17-D2-) -> /USB_D2M
- J17 pad 7: Net-(J17-D2+) -> /Zero/ZGPIO6
- J17 pad 8: GND -> /Zero/ZGPIO7_1
- J17 pad 9: GND -> /Zero/ZGPIO8_1
- J18 pad 1: Net-(J18-Pad1) -> VBUS
- J18 pad 2: Net-(J18-Pad2) -> Net-(J18-D1-)
- J18 pad 3: Net-(J18-Pad3) -> Net-(J18-D1+)
- J18 pad 4: unconnected-(J18-Pad4) -> GND
- J18 pad 5: GND -> VBUS
- J18 pad 6: GND -> Net-(J18-D2-)
- J18 pad 7: GND -> Net-(J18-D2+)
- J18 pad 9: unconnected-(J18-Pad9) -> GND
- J19 pad 1: GND -> Net-(J19-Pad1)
- J19 pad 2: VBUS -> Net-(J19-Pad2)
- J19 pad 3: /GPIO13 -> Net-(J19-Pad3)
- J19 pad 4: /GPIO12 -> unconnected-(J19-Pad4)
- J19 pad 5: /GPIO8 -> GND
- J19 pad 6: /GPIO10 -> GND
- J19 pad 7: /GPIO6 -> GND
- J19 pad 8: /GPIO9 -> GND
- J20 pad 1: /Composite/CVBS -> GND
- J20 pad 2: GND -> VBUS
- J21 pad 1: /USB Hub/DP_IN -> /Composite/CVBS
- J21 pad 2: /USB Hub/DM_IN -> GND
- J22 pad 1: Net-(J22-Pad1) -> /USB Hub/DP_IN
- J22 pad 2: /RS232/TX_IN -> /USB Hub/DM_IN
- JP3 pad 1: Net-(J15-3V3) -> Net-(J16-3V3)
- R100 pad 1: /AMP_IN_L -> GND
- R100 pad 2: Net-(C29-Pad1) -> /Audio Out/AMP_OUTL
- R101 pad 1: /AMP_IN_R -> Net-(U11B--)
- R101 pad 2: Net-(C32-Pad1) -> Net-(C35-Pad2)
- R102 pad 1: Net-(U11A-+) -> Net-(C36-Pad1)
- R102 pad 2: VBUS -> Net-(U11B--)
- R103 pad 1: GND -> Net-(U11A--)
- R103 pad 2: /Audio Out/AMP_OUTL -> Net-(C37-Pad2)
- R104 pad 1: Net-(U11B--) -> Net-(C38-Pad1)
- R104 pad 2: Net-(C35-Pad2) -> Net-(U11A--)
- R105 pad 1: Net-(C36-Pad1) -> GND
- R105 pad 2: Net-(U11B--) -> /Audio Out/AMP_OUTR
- R106 pad 1: Net-(U11A--) -> GND
- R106 pad 2: Net-(C37-Pad2) -> Net-(U11A-+)
- R107 pad 1: Net-(C38-Pad1) -> /TDA_R
- R107 pad 2: Net-(U11A--) -> GND
- R108 pad 2: /Audio Out/AMP_OUTR -> /TDA_L
- R31 pad 2: Net-(J17-D1+) -> Net-(J18-D1+)
- R32 pad 2: Net-(J17-D2+) -> Net-(J18-D2+)
- R33 pad 2: Net-(J17-D1-) -> Net-(J18-D1-)
- R34 pad 2: Net-(J17-D2-) -> Net-(J18-D2-)
- R35 pad 2: Net-(J18-Pad1) -> Net-(J19-Pad1)
- R36 pad 2: Net-(J18-Pad2) -> Net-(J19-Pad2)
- R37 pad 2: Net-(J18-Pad3) -> Net-(J19-Pad3)
- R38 pad 2: Net-(J18-Pad1) -> Net-(J19-Pad1)
- R39 pad 2: Net-(J18-Pad2) -> Net-(J19-Pad2)
- R40 pad 2: Net-(J18-Pad3) -> Net-(J19-Pad3)
- R41 pad 1: Net-(J18-Pad13) -> Net-(J19-Pad13)
- R42 pad 1: Net-(J18-Pad14) -> Net-(J19-Pad14)
- R64 pad 2: GND -> /Audio Out/TS/A1
- R65 pad 2: /Audio Out/TS/A1 -> /Audio Out/TS/A2
- R66 pad 1: /TS_R -> /TS_L
- R66 pad 2: /Audio Out/TS/A2 -> /Audio Out/TS/A1
- R67 pad 2: /Audio Out/TS/A1 -> /Audio Out/TS/A2
- R68 pad 1: /TS_L -> /TS_R
- R68 pad 2: /Audio Out/TS/A2 -> GND
- R73 pad 2: /GPIO28 -> Net-(L1-K)
- R74 pad 2: /GPIO27 -> Net-(L2-K)
- R75 pad 1: GND -> VBUS
- R75 pad 2: /GPIO26 -> /Audio Out/TS/YM_SEL1
- R76 pad 1: GND -> VBUS
- R76 pad 2: Net-(L1-K) -> /Audio Out/TS/YM_SEL2
- R77 pad 1: GND -> /Audio Out/TS/YM_RST
- R77 pad 2: Net-(L2-K) -> VBUS
- R78 pad 1: VBUS -> /TS_R
- R78 pad 2: /Audio Out/TS/YM_SEL1 -> /Audio Out/TS/BEEP
- R79 pad 1: VBUS -> /TS_L
- R79 pad 2: /Audio Out/TS/YM_SEL2 -> /Audio Out/TS/BEEP
- R80 pad 1: /Audio Out/TS/YM_RST -> /TS_R
- R80 pad 2: VBUS -> /Audio Out/TS/SAVE
- R81 pad 1: /TS_R -> /TS_L
- R81 pad 2: /Audio Out/TS/BEEP -> /Audio Out/TS/SAVE
- R82 pad 1: /TS_L -> Net-(Q3-C)
- R82 pad 2: /Audio Out/TS/BEEP -> VBUS
- R83 pad 1: /TS_R -> Net-(Q3-B)
- R83 pad 2: /Audio Out/TS/SAVE -> Net-(Q3-C)
- R84 pad 1: /TS_L -> /GPIO28
- R84 pad 2: /Audio Out/TS/SAVE -> Net-(C26-Pad1)
- R85 pad 1: Net-(Q3-C) -> /GPIO28
- R85 pad 2: VBUS -> Net-(C27-Pad1)
- R86 pad 1: Net-(Q3-B) -> Net-(C26-Pad1)
- R86 pad 2: Net-(Q3-C) -> /PWM_OUT_R
- R87 pad 1: Net-(R87-Pad1) -> Net-(C27-Pad1)
- R87 pad 2: Net-(C26-Pad1) -> /PWM_OUT_L
- R88 pad 1: Net-(R87-Pad1) -> Net-(C27-Pad1)
- R88 pad 2: /GPIO28 -> /GPIO27
- R89 pad 2: /PWM_OUT_R -> /GPIO26
- R90 pad 1: /GPIO28 -> /PWM_OUT_R
- R90 pad 2: /PWM_OUT_L -> GND
- R91 pad 1: /GPIO28 -> /PWM_OUT_L
- R91 pad 2: /GPIO27 -> GND
- R92 pad 1: Net-(C26-Pad1) -> /AMP_IN_L
- R92 pad 2: /GPIO26 -> GND
- R93 pad 1: /PWM_OUT_R -> /AMP_IN_R
- R94 pad 1: /PWM_OUT_L -> Net-(U10-INL)
- R94 pad 2: GND -> Net-(C29-Pad2)
- R95 pad 1: Net-(C29-Pad1) -> VBUS
- R95 pad 2: GND -> /SHND
- R96 pad 1: Net-(C32-Pad1) -> Net-(U10-INR)
- R96 pad 2: GND -> Net-(C32-Pad2)
- R97 pad 1: Net-(U10-INL) -> /AMP_IN_L
- R97 pad 2: Net-(C29-Pad2) -> /AMP_IN_L
- R98 pad 1: VBUS -> /AMP_IN_R
- R98 pad 2: /SHND -> /AMP_IN_R
- R99 pad 1: Net-(U10-INR) -> Net-(U11A-+)
- R99 pad 2: Net-(C32-Pad2) -> VBUS
Routing:
- net VBUS: track 0.00 -> 831.6 mm, vias 0 -> 3
- net +3V3: track 0.00 -> 266.3 mm, vias 0 -> 1
- net /GPIO9: track 0.00 -> 74.7 mm, vias 0 -> 2
- net /GPIO6: track 0.00 -> 73.4 mm, vias 0 -> 1
- net /GPIO7: track 0.00 -> 69.1 mm, vias 0 -> 1
- net /GPIO10: track 0.00 -> 68.2 mm, vias 0 -> 1
- net /GPIO8: track 0.00 -> 66.9 mm, vias 0 -> 1
- net /GPIO13: track 0.00 -> 61.7 mm
- net /GPIO12: track 0.00 -> 61.0 mm, vias 0 -> 2
- net /GPIO11: track 0.00 -> 53.4 mm, vias 0 -> 3
- net Net-(J19-Pad14): track 0.00 -> 22.7 mm
- net Net-(J19-Pad13): track 0.00 -> 21.1 mm
- net Net-(J19-Pad3): track 0.00 -> 14.2 mm
- net Net-(J10-CLKN): track 0.00 -> 12.6 mm
- net Net-(J19-Pad2): track 0.00 -> 12.4 mm
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- added copper zone on B.Cu, net GND
- added copper zone on F.Cu, net GND
