File: hardware/turbofrank/tape.kicad_sch (KiCad schematic)
At the start: 11 parts, among them Q2 BC850, Q3 BC850

Commit message: Bugfixes
Connections:
- net LOAD_IN: no longer AJ2.T, C29.1, R81.1
- new net: AJ2.T, C29.1, R81.1
Changed lines of the file:
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@@
-		)
-	)
-	(label "LOAD_IN"
-		(at 49.53 72.39 0)
-		(effects
-			(font
-				(size 1.27 1.27)
-			)
-			(justify left bottom)
 		)
 	)

Commit message: TurboFRANK 1.04 WIP
Parts:
- J15: renamed from AJ2; value SJ1-353XNG -> ~; footprint FRANK:Jack (3.5mm) -> FRANK:Jack (3.5mm, PJ-320D); AliExpress https://www.aliexpress.com/item/1005006710837751.html -> (none)
- renumbered C28 to C10, C29 to C11, D9 to D7, Q2 to Q1, Q3 to Q2, R77 to R26, R78 to R27, R79 to R28, R80 to R29, R81 to R30
Connections:
- no-connect marks 3 -> 1
Other:
- note removed: "This schematics is used to load data from external audio source, e.g. tape."
Changed lines of the file:
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@@
 	(title_block
 		(title "TurboFRANK")
-		(date "2025-03-03")
-		(rev "1.03")
+		(date "2025-03-17")
+		(rev "1.04")
 		(company "Mikhail Matveev")
 		(comment 1 "https://github.com/xtremespb/frank")
-	)
-	(text "This schematics is used to load data from\nexternal audio source, e.g. tape."
-		(exclude_from_sim no)
-		(at 38.1 27.178 0)
-		(effects
-			(font
-				(size 1.27 1.27)
-			)
-			(justify left)
-		)
 	)
 	(junction
@@
 		(diameter 0)
 		(color 0 0 0 0)
-	)
-	(no_connect
-		(at 49.53 69.85)
-	)
-	(no_connect
-		(at 49.53 74.93)
 	)
 	(no_connect
@@
 		(dnp no)
 		(fields_autoplaced yes)
-		(property "Reference" "D9"
+		(property "Reference" "D7"
 			(at 93.98 58.42 0)
 			(effects
@@
 			(project ""
 				(path "/8c0b3d8b-46d3-4173-ab1e-a61765f77d61/599e2208-d0f7-4f1d-beb8-3b4e6272cb10"
-					(reference "D9")
+					(reference "D7")
 					(unit 1)
 				)
@@
 		(dnp no)
 		(fields_autoplaced yes)
-		(property "Reference" "#PWR085"
+		(property "Reference" "#PWR055"
 			(at 99.06 93.98 0)
 			(effects
@@
 			(project ""
 				(path "/8c0b3d8b-46d3-4173-ab1e-a61765f77d61/599e2208-d0f7-4f1d-beb8-3b4e6272cb10"
-					(reference "#PWR085")
+					(reference "#PWR055")
 					(unit 1)
 				)
@@
 		(dnp no)
 		(fields_autoplaced yes)
-		(property "Reference" "R79"
+		(property "Reference" "R28"
 			(at 105.41 58.42 90)
 			(effects
@@
 			(project "38NJU24"
 				(path "/8c0b3d8b-46d3-4173-ab1e-a61765f77d61/599e2208-d0f7-4f1d-beb8-3b4e6272cb10"
-					(reference "R79")
+					(reference "R28")
 					(unit 1)
 				)
@@
 		(dnp no)
 		(fields_autoplaced yes)
-		(property "Reference" "#PWR084"
+		(property "Reference" "#PWR054"
 			(at 66.04 93.98 0)
 			(effects
@@
 			(project ""
 				(path "/8c0b3d8b-46d3-4173-ab1e-a61765f77d61/599e2208-d0f7-4f1d-beb8-3b4e6272cb10"
-					(reference "#PWR084")
+					(reference "#PWR054")
 					(unit 1)
 				)
@@
 		(dnp no)
 		(fields_autoplaced yes)
-		(property "Reference" "R78"
+		(property "Reference" "R27"
 			(at 119.38 52.0699 0)
 			(effects
@@
 			(project "38NJU24"
 				(path "/8c0b3d8b-46d3-4173-ab1e-a61765f77d61/599e2208-d0f7-4f1d-beb8-3b4e6272cb10"
-					(reference "R78")
+					(reference "R27")
 					(unit 1)
 				)
@@
 		(on_board yes)
 		(dnp no)
-		(property "Reference" "AJ2"
+		(property "Reference" "J15"
 			(at 37.3381 73.4603 0)
 			(effects
@@
 			)
 		)
-		(property "Value" "SJ1-353XNG"
+		(property "Value" "~"
 			(at 46.99 66.04 0)
 			(effects
@@
 			)
 		)
-		(property "Footprint" "FRANK:Jack (3.5mm)"
+		(property "Footprint" "FRANK:Jack (3.5mm, PJ-320D)"
 			(at 44.45 77.47 0)
 			(effects
@@
 			)
 		)
-		(property "Datasheet" "https://eu.mouser.com/datasheet/2/1628/sj1_353xng-3511142.pdf"
+		(property "Datasheet" "~"
 			(at 44.45 77.47 0)
 			(effects
@@
 			)
 		)
-		(property "Description" "Audio Jack, 3 Poles (Stereo / TRS), Switched TR Poles (Normalling)"
+		(property "Description" ""
 			(at 44.45 77.47 0)
 			(effects
@@
 			)
 		)
-		(property "AliExpress" "https://www.aliexpress.com/item/1005006710837751.html"
+		(property "AliExpress" ""
 			(at 44.45 77.47 0)
 			(effects
@@
 		(pin "R"
 		)
-		(pin "RN"
-		)
 		(pin "S"
 		)
 		(pin "T"
-		)
-		(pin "TN"
 		)
 		(instances
@@
 			(project "38NJU24"
 				(path "/8c0b3d8b-46d3-4173-ab1e-a61765f77d61/599e2208-d0f7-4f1d-beb8-3b4e6272cb10"
-					(reference "AJ2")
+					(reference "J15")
 					(unit 1)
 				)
@@
 		(on_board yes)
 		(dnp no)
-		(property "Reference" "C29"
+		(property "Reference" "C11"
 			(at 71.12 68.58 90)
 			(effects
@@
 			(project "38NJU24"
 				(path "/8c0b3d8b-46d3-4173-ab1e-a61765f77d61/599e2208-d0f7-4f1d-beb8-3b4e6272cb10"
-					(reference "C29")
+					(reference "C11")
 					(unit 1)
 				)
@@
 		(dnp no)
 		(fields_autoplaced yes)
-		(property "Reference" "#PWR083"
+		(property "Reference" "#PWR053"
 			(at 55.88 80.01 0)
 			(effects
@@
 			(project ""
 				(path "/8c0b3d8b-46d3-4173-ab1e-a61765f77d61/599e2208-d0f7-4f1d-beb8-3b4e6272cb10"
-					(reference "#PWR083")
+					(reference "#PWR053")
 					(unit 1)
 				)
@@
 		(dnp no)
 		(fields_autoplaced yes)
-		(property "Reference" "R80"
+		(property "Reference" "R29"
 			(at 81.28 66.04 90)
 			(effects
@@
 			(project "38NJU24"
 				(path "/8c0b3d8b-46d3-4173-ab1e-a61765f77d61/599e2208-d0f7-4f1d-beb8-3b4e6272cb10"
-					(reference "R80")
+					(reference "R29")
 					(unit 1)
 				)
@@
 		(dnp no)
 		(fields_autoplaced yes)
-		(property "Reference" "#PWR082"
+		(property "Reference" "#PWR052"
 			(at 138.43 58.42 0)
 			(effects
@@
 			(project ""
 				(path "/8c0b3d8b-46d3-4173-ab1e-a61765f77d61/599e2208-d0f7-4f1d-beb8-3b4e6272cb10"
-					(reference "#PWR082")
+					(reference "#PWR052")
 					(unit 1)
 				)
@@
 		(dnp no)
 		(fields_autoplaced yes)
-		(property "Reference" "#PWR086"
+		(property "Reference" "#PWR056"
 			(at 116.84 93.98 0)
 			(effects
@@
 			(project ""
 				(path "/8c0b3d8b-46d3-4173-ab1e-a61765f77d61/599e2208-d0f7-4f1d-beb8-3b4e6272cb10"
-					(reference "#PWR086")
+					(reference "#PWR056")
 					(unit 1)
 				)
@@
 		(dnp no)
 		(fields_autoplaced yes)
-		(property "Reference" "#PWR081"
+		(property "Reference" "#PWR051"
 			(at 121.92 43.18 0)
 			(effects
@@
 			(project ""
 				(path "/8c0b3d8b-46d3-4173-ab1e-a61765f77d61/599e2208-d0f7-4f1d-beb8-3b4e6272cb10"
-					(reference "#PWR081")
+					(reference "#PWR051")
 					(unit 1)
 				)
@@
 		(on_board yes)
 		(dnp no)
-		(property "Reference" "C28"
+		(property "Reference" "C10"
 			(at 135.001 49.6316 0)
 			(effects
@@
 			(project "38NJU24"
 				(path "/8c0b3d8b-46d3-4173-ab1e-a61765f77d61/599e2208-d0f7-4f1d-beb8-3b4e6272cb10"
-					(reference "C28")
+					(reference "C10")
 					(unit 1)
 				)
@@
 		(dnp no)
 		(fields_autoplaced yes)
-		(property "Reference" "R81"
+		(property "Reference" "R30"
 			(at 67.818 82.6078 0)
 			(effects
@@
 			(project "38NJU24"
 				(path "/8c0b3d8b-46d3-4173-ab1e-a61765f77d61/599e2208-d0f7-4f1d-beb8-3b4e6272cb10"
-					(reference "R81")
+					(reference "R30")
 					(unit 1)
 				)
@@
 		(dnp no)
 		(fields_autoplaced yes)
-		(property "Reference" "Q3"
+		(property "Reference" "Q2"
 			(at 101.3714 71.5553 0)
 			(effects
@@
 			(project "38NJU24"
 				(path "/8c0b3d8b-46d3-4173-ab1e-a61765f77d61/599e2208-d0f7-4f1d-beb8-3b4e6272cb10"
-					(reference "Q3")
+					(reference "Q2")
 					(unit 1)
 				)
@@
 		(dnp no)
 		(fields_autoplaced yes)
-		(property "Reference" "R77"
+		(property "Reference" "R26"
 			(at 101.6 52.0699 0)
 			(effects
@@
 			(project "38NJU24"
 				(path "/8c0b3d8b-46d3-4173-ab1e-a61765f77d61/599e2208-d0f7-4f1d-beb8-3b4e6272cb10"
-					(reference "R77")
+					(reference "R26")
 					(unit 1)
 				)
@@
 		(dnp no)
 		(fields_autoplaced yes)
-		(property "Reference" "Q2"
+		(property "Reference" "Q1"
 			(at 119.1514 63.9353 0)
 			(effects
@@
 			(project "38NJU24"
 				(path "/8c0b3d8b-46d3-4173-ab1e-a61765f77d61/599e2208-d0f7-4f1d-beb8-3b4e6272cb10"
-					(reference "Q2")
-					(unit 1)
-				)
+					(reference "Q1")
+					(unit 1)
+				)

Commit message: TurboFRANK WIP
Parts:
- renumbered C10 to C7, C11 to C8, J15 to J13, R26 to R22, R27 to R23, R28 to R24, R29 to R25, R30 to R26
Other:
- moved on the sheet: C7, C8, D7, J13, Q1, Q2, R22, R23, R24, R25, R26

Commit message: TurboFRANK HW 1.05 Release
Parts:
- J13: value ~ -> PJ-320D; AliExpress (none) -> https://www.aliexpress.com/item/4001158231104.html
Changed lines of the file:
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@@
 			)
 		)
-		(property "Value" "~"
+		(property "Value" "PJ-320D"
 			(at 109.22 93.98 0)
 			(effects
@@
 			)
 		)
-		(property "Datasheet" "~"
+		(property "Datasheet" "https://www.lcsc.com/datasheet/lcsc_datasheet_1810121716_Korean-Hroparts-Elec-PJ-320D-4A_C95562.pdf"
 			(at 106.68 105.41 0)
 			(effects
@@
 			)
 		)
-		(property "AliExpress" ""
+		(property "AliExpress" "https://www.aliexpress.com/item/4001158231104.html"
 			(at 106.68 105.41 0)
 			(effects
