File: hardware/turbofrank/composite.kicad_sch (KiCad schematic)
At the start: 16 parts

Commit message: TurboFRANK 1.04 WIP
Parts:
- renumbered C32 to C14, SC1 to J21, R94 to R43, R95 to R44, R96 to R45, R97 to R46, R98 to R47, R99 to R48, R100 to R49, R101 to R50, R102 to R51, R103 to R52, R104 to R53, R105 to R54, R106 to R55, R107 to R56
Changed lines of the file:
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@@
 	(title_block
 		(title "TurboFRANK")
-		(date "2025-03-03")
-		(rev "1.03")
+		(date "2025-03-17")
+		(rev "1.04")
 		(company "Mikhail Matveev")
 		(comment 1 "https://github.com/xtremespb/frank")
@@
 		(on_board yes)
 		(dnp no)
-		(property "Reference" "R105"
+		(property "Reference" "R54"
 			(at 69.85 97.79 0)
 			(effects
@@
 			(project ""
 				(path "/8c0b3d8b-46d3-4173-ab1e-a61765f77d61/50e44d6f-5022-48d1-aa5c-5d8f0f1936d3"
-					(reference "R105")
+					(reference "R54")
 					(unit 1)
 				)
@@
 		(on_board yes)
 		(dnp no)
-		(property "Reference" "R104"
+		(property "Reference" "R53"
 			(at 49.53 92.71 90)
 			(effects
@@
 			(project ""
 				(path "/8c0b3d8b-46d3-4173-ab1e-a61765f77d61/50e44d6f-5022-48d1-aa5c-5d8f0f1936d3"
-					(reference "R104")
+					(reference "R53")
 					(unit 1)
 				)
@@
 		(dnp no)
 		(fields_autoplaced yes)
-		(property "Reference" "#PWR0106"
+		(property "Reference" "#PWR076"
 			(at 104.14 59.69 0)
 			(effects
@@
 			(project ""
 				(path "/8c0b3d8b-46d3-4173-ab1e-a61765f77d61/50e44d6f-5022-48d1-aa5c-5d8f0f1936d3"
-					(reference "#PWR0106")
+					(reference "#PWR076")
 					(unit 1)
 				)
@@
 		(on_board yes)
 		(dnp no)
-		(property "Reference" "R100"
+		(property "Reference" "R49"
 			(at 49.53 69.85 90)
 			(effects
@@
 			(project ""
 				(path "/8c0b3d8b-46d3-4173-ab1e-a61765f77d61/50e44d6f-5022-48d1-aa5c-5d8f0f1936d3"
-					(reference "R100")
+					(reference "R49")
 					(unit 1)
 				)
@@
 		(on_board yes)
 		(dnp no)
-		(property "Reference" "R96"
+		(property "Reference" "R45"
 			(at 49.53 46.99 90)
 			(effects
@@
 			(project ""
 				(path "/8c0b3d8b-46d3-4173-ab1e-a61765f77d61/50e44d6f-5022-48d1-aa5c-5d8f0f1936d3"
-					(reference "R96")
+					(reference "R45")
 					(unit 1)
 				)
@@
 		(on_board yes)
 		(dnp no)
-		(property "Reference" "R94"
+		(property "Reference" "R43"
 			(at 49.53 36.83 90)
 			(effects
@@
 			(project ""
 				(path "/8c0b3d8b-46d3-4173-ab1e-a61765f77d61/50e44d6f-5022-48d1-aa5c-5d8f0f1936d3"
-					(reference "R94")
+					(reference "R43")
 					(unit 1)
 				)
@@
 		(on_board yes)
 		(dnp no)
-		(property "Reference" "R101"
+		(property "Reference" "R50"
 			(at 69.85 74.93 0)
 			(effects
@@
 			(project ""
 				(path "/8c0b3d8b-46d3-4173-ab1e-a61765f77d61/50e44d6f-5022-48d1-aa5c-5d8f0f1936d3"
-					(reference "R101")
+					(reference "R50")
 					(unit 1)
 				)
@@
 		(on_board yes)
 		(dnp no)
-		(property "Reference" "R107"
+		(property "Reference" "R56"
 			(at 49.53 111.76 90)
 			(effects
@@
 			(project ""
 				(path "/8c0b3d8b-46d3-4173-ab1e-a61765f77d61/50e44d6f-5022-48d1-aa5c-5d8f0f1936d3"
-					(reference "R107")
+					(reference "R56")
 					(unit 1)
 				)
@@
 		(dnp no)
 		(fields_autoplaced yes)
-		(property "Reference" "C32"
+		(property "Reference" "C14"
 			(at 94.361 32.2412 90)
 			(effects
@@
 			(project ""
 				(path "/8c0b3d8b-46d3-4173-ab1e-a61765f77d61/50e44d6f-5022-48d1-aa5c-5d8f0f1936d3"
-					(reference "C32")
+					(reference "C14")
 					(unit 1)
 				)
@@
 		(on_board yes)
 		(dnp no)
-		(property "Reference" "R98"
+		(property "Reference" "R47"
 			(at 49.53 58.42 90)
 			(effects
@@
 			(project ""
 				(path "/8c0b3d8b-46d3-4173-ab1e-a61765f77d61/50e44d6f-5022-48d1-aa5c-5d8f0f1936d3"
-					(reference "R98")
+					(reference "R47")
 					(unit 1)
 				)
@@
 		(on_board yes)
 		(dnp no)
-		(property "Reference" "R95"
+		(property "Reference" "R44"
 			(at 72.39 36.83 90)
 			(effects
@@
 			(project ""
 				(path "/8c0b3d8b-46d3-4173-ab1e-a61765f77d61/50e44d6f-5022-48d1-aa5c-5d8f0f1936d3"
-					(reference "R95")
+					(reference "R44")
 					(unit 1)
 				)
@@
 		(on_board yes)
 		(dnp no)
-		(property "Reference" "R102"
+		(property "Reference" "R51"
 			(at 49.53 81.28 90)
 			(effects
@@
 			(project ""
 				(path "/8c0b3d8b-46d3-4173-ab1e-a61765f77d61/50e44d6f-5022-48d1-aa5c-5d8f0f1936d3"
-					(reference "R102")
+					(reference "R51")
 					(unit 1)
 				)
@@
 		(on_board yes)
 		(dnp no)
-		(property "Reference" "R103"
+		(property "Reference" "R52"
 			(at 69.85 86.36 0)
 			(effects
@@
 			(project ""
 				(path "/8c0b3d8b-46d3-4173-ab1e-a61765f77d61/50e44d6f-5022-48d1-aa5c-5d8f0f1936d3"
-					(reference "R103")
+					(reference "R52")
 					(unit 1)
 				)
@@
 		(on_board yes)
 		(dnp no)
-		(property "Reference" "R106"
+		(property "Reference" "R55"
 			(at 49.53 104.14 90)
 			(effects
@@
 			(project ""
 				(path "/8c0b3d8b-46d3-4173-ab1e-a61765f77d61/50e44d6f-5022-48d1-aa5c-5d8f0f1936d3"
-					(reference "R106")
+					(reference "R55")
 					(unit 1)
 				)
@@
 		(dnp no)
 		(fields_autoplaced yes)
-		(property "Reference" "SC1"
+		(property "Reference" "J21"
 			(at 107.95 43.1799 0)
 			(effects
@@
 			(project ""
 				(path "/8c0b3d8b-46d3-4173-ab1e-a61765f77d61/50e44d6f-5022-48d1-aa5c-5d8f0f1936d3"
-					(reference "SC1")
+					(reference "J21")
 					(unit 1)
 				)
@@
 		(on_board yes)
 		(dnp no)
-		(property "Reference" "R97"
+		(property "Reference" "R46"
 			(at 69.85 52.07 0)
 			(effects
@@
 			(project ""
 				(path "/8c0b3d8b-46d3-4173-ab1e-a61765f77d61/50e44d6f-5022-48d1-aa5c-5d8f0f1936d3"
-					(reference "R97")
+					(reference "R46")
 					(unit 1)
 				)
@@
 		(on_board yes)
 		(dnp no)
-		(property "Reference" "R99"
+		(property "Reference" "R48"
 			(at 69.85 63.5 0)
 			(effects
@@
 			(project ""
 				(path "/8c0b3d8b-46d3-4173-ab1e-a61765f77d61/50e44d6f-5022-48d1-aa5c-5d8f0f1936d3"
-					(reference "R99")
+					(reference "R48")
 					(unit 1)
 				)
@@
 		(dnp no)
 		(fields_autoplaced yes)
-		(property "Reference" "#PWR0107"
+		(property "Reference" "#PWR077"
 			(at 40.64 125.73 0)
 			(effects
@@
 			(project ""
 				(path "/8c0b3d8b-46d3-4173-ab1e-a61765f77d61/50e44d6f-5022-48d1-aa5c-5d8f0f1936d3"
-					(reference "#PWR0107")
+					(reference "#PWR077")
 					(unit 1)
 				)

Commit message: TurboFRANK WIP
Parts:
- renumbered C14 to C11, J21 to J19, R43 to R39, R44 to R40, R45 to R41, R46 to R42, R47 to R43, R48 to R44, R49 to R45, R50 to R46, R51 to R47, R52 to R48, R53 to R49, R54 to R50, R55 to R51, R56 to R52
Changed lines of the file:
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@@
 		(on_board yes)
 		(dnp no)
-		(property "Reference" "R54"
+		(property "Reference" "R50"
 			(at 69.85 97.79 0)
 			(effects
@@
 			(project ""
 				(path "/8c0b3d8b-46d3-4173-ab1e-a61765f77d61/50e44d6f-5022-48d1-aa5c-5d8f0f1936d3"
-					(reference "R54")
+					(reference "R50")
 					(unit 1)
 				)
@@
 		(on_board yes)
 		(dnp no)
-		(property "Reference" "R53"
+		(property "Reference" "R49"
 			(at 49.53 92.71 90)
 			(effects
@@
 			(project ""
 				(path "/8c0b3d8b-46d3-4173-ab1e-a61765f77d61/50e44d6f-5022-48d1-aa5c-5d8f0f1936d3"
-					(reference "R53")
+					(reference "R49")
 					(unit 1)
 				)
@@
 		(dnp no)
 		(fields_autoplaced yes)
-		(property "Reference" "#PWR076"
+		(property "Reference" "#PWR071"
 			(at 104.14 59.69 0)
 			(effects
@@
 			(project ""
 				(path "/8c0b3d8b-46d3-4173-ab1e-a61765f77d61/50e44d6f-5022-48d1-aa5c-5d8f0f1936d3"
-					(reference "#PWR076")
+					(reference "#PWR071")
 					(unit 1)
 				)
@@
 		(on_board yes)
 		(dnp no)
-		(property "Reference" "R49"
+		(property "Reference" "R45"
 			(at 49.53 69.85 90)
 			(effects
@@
 			(project ""
 				(path "/8c0b3d8b-46d3-4173-ab1e-a61765f77d61/50e44d6f-5022-48d1-aa5c-5d8f0f1936d3"
-					(reference "R49")
+					(reference "R45")
 					(unit 1)
 				)
@@
 		(on_board yes)
 		(dnp no)
-		(property "Reference" "R45"
+		(property "Reference" "R41"
 			(at 49.53 46.99 90)
 			(effects
@@
 			(project ""
 				(path "/8c0b3d8b-46d3-4173-ab1e-a61765f77d61/50e44d6f-5022-48d1-aa5c-5d8f0f1936d3"
-					(reference "R45")
+					(reference "R41")
 					(unit 1)
 				)
@@
 		(on_board yes)
 		(dnp no)
-		(property "Reference" "R43"
+		(property "Reference" "R39"
 			(at 49.53 36.83 90)
 			(effects
@@
 			(project ""
 				(path "/8c0b3d8b-46d3-4173-ab1e-a61765f77d61/50e44d6f-5022-48d1-aa5c-5d8f0f1936d3"
-					(reference "R43")
+					(reference "R39")
 					(unit 1)
 				)
@@
 		(on_board yes)
 		(dnp no)
-		(property "Reference" "R50"
+		(property "Reference" "R46"
 			(at 69.85 74.93 0)
 			(effects
@@
 			(project ""
 				(path "/8c0b3d8b-46d3-4173-ab1e-a61765f77d61/50e44d6f-5022-48d1-aa5c-5d8f0f1936d3"
-					(reference "R50")
+					(reference "R46")
 					(unit 1)
 				)
@@
 		(on_board yes)
 		(dnp no)
-		(property "Reference" "R56"
+		(property "Reference" "R52"
 			(at 49.53 111.76 90)
 			(effects
@@
 			(project ""
 				(path "/8c0b3d8b-46d3-4173-ab1e-a61765f77d61/50e44d6f-5022-48d1-aa5c-5d8f0f1936d3"
-					(reference "R56")
+					(reference "R52")
 					(unit 1)
 				)
@@
 		(dnp no)
 		(fields_autoplaced yes)
-		(property "Reference" "C14"
+		(property "Reference" "C11"
 			(at 94.361 32.2412 90)
 			(effects
@@
 			(project ""
 				(path "/8c0b3d8b-46d3-4173-ab1e-a61765f77d61/50e44d6f-5022-48d1-aa5c-5d8f0f1936d3"
-					(reference "C14")
+					(reference "C11")
 					(unit 1)
 				)
@@
 		(on_board yes)
 		(dnp no)
-		(property "Reference" "R47"
+		(property "Reference" "R43"
 			(at 49.53 58.42 90)
 			(effects
@@
 			(project ""
 				(path "/8c0b3d8b-46d3-4173-ab1e-a61765f77d61/50e44d6f-5022-48d1-aa5c-5d8f0f1936d3"
-					(reference "R47")
+					(reference "R43")
 					(unit 1)
 				)
@@
 		(on_board yes)
 		(dnp no)
-		(property "Reference" "R44"
+		(property "Reference" "R40"
 			(at 72.39 36.83 90)
 			(effects
@@
 			(project ""
 				(path "/8c0b3d8b-46d3-4173-ab1e-a61765f77d61/50e44d6f-5022-48d1-aa5c-5d8f0f1936d3"
-					(reference "R44")
+					(reference "R40")
 					(unit 1)
 				)
@@
 		(on_board yes)
 		(dnp no)
-		(property "Reference" "R51"
+		(property "Reference" "R47"
 			(at 49.53 81.28 90)
 			(effects
@@
 			(project ""
 				(path "/8c0b3d8b-46d3-4173-ab1e-a61765f77d61/50e44d6f-5022-48d1-aa5c-5d8f0f1936d3"
-					(reference "R51")
+					(reference "R47")
 					(unit 1)
 				)
@@
 		(on_board yes)
 		(dnp no)
-		(property "Reference" "R52"
+		(property "Reference" "R48"
 			(at 69.85 86.36 0)
 			(effects
@@
 			(project ""
 				(path "/8c0b3d8b-46d3-4173-ab1e-a61765f77d61/50e44d6f-5022-48d1-aa5c-5d8f0f1936d3"
-					(reference "R52")
+					(reference "R48")
 					(unit 1)
 				)
@@
 		(on_board yes)
 		(dnp no)
-		(property "Reference" "R55"
+		(property "Reference" "R51"
 			(at 49.53 104.14 90)
 			(effects
@@
 			(project ""
 				(path "/8c0b3d8b-46d3-4173-ab1e-a61765f77d61/50e44d6f-5022-48d1-aa5c-5d8f0f1936d3"
-					(reference "R55")
+					(reference "R51")
 					(unit 1)
 				)
@@
 		(dnp no)
 		(fields_autoplaced yes)
-		(property "Reference" "J21"
+		(property "Reference" "J19"
 			(at 107.95 43.1799 0)
 			(effects
@@
 			(project ""
 				(path "/8c0b3d8b-46d3-4173-ab1e-a61765f77d61/50e44d6f-5022-48d1-aa5c-5d8f0f1936d3"
-					(reference "J21")
+					(reference "J19")
 					(unit 1)
 				)
@@
 		(on_board yes)
 		(dnp no)
-		(property "Reference" "R46"
+		(property "Reference" "R42"
 			(at 69.85 52.07 0)
 			(effects
@@
 			(project ""
 				(path "/8c0b3d8b-46d3-4173-ab1e-a61765f77d61/50e44d6f-5022-48d1-aa5c-5d8f0f1936d3"
-					(reference "R46")
+					(reference "R42")
 					(unit 1)
 				)
@@
 		(on_board yes)
 		(dnp no)
-		(property "Reference" "R48"
+		(property "Reference" "R44"
 			(at 69.85 63.5 0)
 			(effects
@@
 			(project ""
 				(path "/8c0b3d8b-46d3-4173-ab1e-a61765f77d61/50e44d6f-5022-48d1-aa5c-5d8f0f1936d3"
-					(reference "R48")
+					(reference "R44")
 					(unit 1)
 				)
@@
 		(dnp no)
 		(fields_autoplaced yes)
-		(property "Reference" "#PWR077"
+		(property "Reference" "#PWR072"
 			(at 40.64 125.73 0)
 			(effects
@@
 			(project ""
 				(path "/8c0b3d8b-46d3-4173-ab1e-a61765f77d61/50e44d6f-5022-48d1-aa5c-5d8f0f1936d3"
-					(reference "#PWR077")
-					(unit 1)
-				)
+					(reference "#PWR072")
+					(unit 1)
+				)

Commit message: TurboFRANK HW 1.05 Release
Other:
- moved on the sheet: C11, J19, R39, R40, R41, R42, R43, R44, R45, R46, R47, R48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

Commit message: Bugfixes
Other:
- title: TurboFRANK -> ${NAME}
Changed lines of the file:
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@@
 	(paper "A4")
 	(title_block
-		(title "TurboFRANK")
-		(date "2025-04-04")
+		(title "${NAME}")
+		(date "2025-04-20")
 		(rev "${VERSION}")
 		(company "Mikhail Matveev")
