File: hardware/turbofrank/rs232.kicad_sch (KiCad schematic)
At the start: 10 parts

Commit message: TurboFRANK 1.04 WIP
Parts:
- renumbered C33 to C15, C34 to C16, C35 to C17, C36 to C18, D10 to D8, D11 to D9, COM1 to J23, R108 to R57, R109 to R58, MAX1 to U4
Changed lines of the file:
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@@
 	(title_block
 		(title "TurboFRANK")
-		(date "2025-03-03")
-		(rev "1.03")
+		(date "2025-03-17")
+		(rev "1.04")
 		(company "Mikhail Matveev")
 		(comment 1 "https://github.com/xtremespb/frank")
@@
 		(dnp no)
 		(fields_autoplaced yes)
-		(property "Reference" "C34"
+		(property "Reference" "C16"
 			(at 59.6963 62.23 90)
 			(effects
@@
 			(project "turbofrank"
 				(path "/8c0b3d8b-46d3-4173-ab1e-a61765f77d61/960439d1-a657-47b6-aee7-897565b7d217"
-					(reference "C34")
+					(reference "C16")
 					(unit 1)
 				)
@@
 		(dnp no)
 		(fields_autoplaced yes)
-		(property "Reference" "#PWR0108"
+		(property "Reference" "#PWR080"
 			(at 99.06 36.83 0)
 			(effects
@@
 			(project ""
 				(path "/8c0b3d8b-46d3-4173-ab1e-a61765f77d61/960439d1-a657-47b6-aee7-897565b7d217"
-					(reference "#PWR0108")
+					(reference "#PWR080")
 					(unit 1)
 				)
@@
 		(dnp no)
 		(fields_autoplaced yes)
-		(property "Reference" "#PWR0111"
+		(property "Reference" "#PWR083"
 			(at 116.84 54.61 0)
 			(effects
@@
 			(project ""
 				(path "/8c0b3d8b-46d3-4173-ab1e-a61765f77d61/960439d1-a657-47b6-aee7-897565b7d217"
-					(reference "#PWR0111")
+					(reference "#PWR083")
 					(unit 1)
 				)
@@
 		(dnp no)
 		(fields_autoplaced yes)
-		(property "Reference" "C35"
+		(property "Reference" "C17"
 			(at 48.2663 67.31 90)
 			(effects
@@
 			(project "turbofrank"
 				(path "/8c0b3d8b-46d3-4173-ab1e-a61765f77d61/960439d1-a657-47b6-aee7-897565b7d217"
-					(reference "C35")
+					(reference "C17")
 					(unit 1)
 				)
@@
 		(dnp no)
 		(fields_autoplaced yes)
-		(property "Reference" "C33"
+		(property "Reference" "C15"
 			(at 106.6863 50.8 90)
 			(effects
@@
 			(project ""
 				(path "/8c0b3d8b-46d3-4173-ab1e-a61765f77d61/960439d1-a657-47b6-aee7-897565b7d217"
-					(reference "C33")
+					(reference "C15")
 					(unit 1)
 				)
@@
 		(dnp no)
 		(fields_autoplaced yes)
-		(property "Reference" "#PWR0109"
+		(property "Reference" "#PWR081"
 			(at 146.05 36.83 0)
 			(effects
@@
 			(project "frank2"
 				(path "/8c0b3d8b-46d3-4173-ab1e-a61765f77d61/960439d1-a657-47b6-aee7-897565b7d217"
-					(reference "#PWR0109")
+					(reference "#PWR081")
 					(unit 1)
 				)
@@
 		(on_board yes)
 		(dnp no)
-		(property "Reference" "R109"
+		(property "Reference" "R58"
 			(at 144.78 41.91 90)
 			(effects
@@
 			(project "frank2"
 				(path "/8c0b3d8b-46d3-4173-ab1e-a61765f77d61/960439d1-a657-47b6-aee7-897565b7d217"
-					(reference "R109")
+					(reference "R58")
 					(unit 1)
 				)
@@
 		(on_board yes)
 		(dnp no)
-		(property "Reference" "C36"
+		(property "Reference" "C18"
 			(at 46.99 90.17 90)
 			(effects
@@
 			(project "turbofrank"
 				(path "/8c0b3d8b-46d3-4173-ab1e-a61765f77d61/960439d1-a657-47b6-aee7-897565b7d217"
-					(reference "C36")
+					(reference "C18")
 					(unit 1)
 				)
@@
 		(dnp no)
 		(fields_autoplaced yes)
-		(property "Reference" "#PWR0110"
+		(property "Reference" "#PWR082"
 			(at 187.96 53.34 0)
 			(effects
@@
 			(project "frank2"
 				(path "/8c0b3d8b-46d3-4173-ab1e-a61765f77d61/960439d1-a657-47b6-aee7-897565b7d217"
-					(reference "#PWR0110")
+					(reference "#PWR082")
 					(unit 1)
 				)
@@
 		(dnp no)
 		(fields_autoplaced yes)
-		(property "Reference" "D11"
+		(property "Reference" "D9"
 			(at 132.08 40.64 0)
 			(effects
@@
 			(project "frank2"
 				(path "/8c0b3d8b-46d3-4173-ab1e-a61765f77d61/960439d1-a657-47b6-aee7-897565b7d217"
-					(reference "D11")
+					(reference "D9")
 					(unit 1)
 				)
@@
 		(dnp no)
 		(fields_autoplaced yes)
-		(property "Reference" "MAX1"
+		(property "Reference" "U4"
 			(at 96.52 60.96 0)
 			(effects
@@
 			(project "frank2"
 				(path "/8c0b3d8b-46d3-4173-ab1e-a61765f77d61/960439d1-a657-47b6-aee7-897565b7d217"
-					(reference "MAX1")
+					(reference "U4")
 					(unit 1)
 				)
@@
 		(dnp no)
 		(fields_autoplaced yes)
-		(property "Reference" "#PWR0113"
+		(property "Reference" "#PWR085"
 			(at 33.02 83.82 0)
 			(effects
@@
 			(project "frank2"
 				(path "/8c0b3d8b-46d3-4173-ab1e-a61765f77d61/960439d1-a657-47b6-aee7-897565b7d217"
-					(reference "#PWR0113")
+					(reference "#PWR085")
 					(unit 1)
 				)
@@
 		(on_board yes)
 		(dnp no)
-		(property "Reference" "R108"
+		(property "Reference" "R57"
 			(at 97.79 41.91 90)
 			(effects
@@
 			(project "frank2"
 				(path "/8c0b3d8b-46d3-4173-ab1e-a61765f77d61/960439d1-a657-47b6-aee7-897565b7d217"
-					(reference "R108")
+					(reference "R57")
 					(unit 1)
 				)
@@
 		(on_board yes)
 		(dnp no)
-		(property "Reference" "#PWR0112"
+		(property "Reference" "#PWR084"
 			(at 118.11 71.12 0)
 			(effects
@@
 			(project "frank2"
 				(path "/8c0b3d8b-46d3-4173-ab1e-a61765f77d61/960439d1-a657-47b6-aee7-897565b7d217"
-					(reference "#PWR0112")
+					(reference "#PWR084")
 					(unit 1)
 				)
@@
 		(dnp no)
 		(fields_autoplaced yes)
-		(property "Reference" "D10"
+		(property "Reference" "D8"
 			(at 85.09 40.64 0)
 			(effects
@@
 			(project "frank2"
 				(path "/8c0b3d8b-46d3-4173-ab1e-a61765f77d61/960439d1-a657-47b6-aee7-897565b7d217"
-					(reference "D10")
+					(reference "D8")
 					(unit 1)
 				)
@@
 		(on_board yes)
 		(dnp no)
-		(property "Reference" "COM1"
+		(property "Reference" "J23"
 			(at 220.98 50.8 0)
 			(effects
@@
 			(project "frank2"
 				(path "/8c0b3d8b-46d3-4173-ab1e-a61765f77d61/960439d1-a657-47b6-aee7-897565b7d217"
-					(reference "COM1")
+					(reference "J23")
 					(unit 1)
 				)

Commit message: TurboFRANK WIP
Parts:
- renumbered C15 to C12, C16 to C13, C17 to C14, C18 to C15, J23 to J20, R57 to R53, R58 to R54, U4 to U3
Changed lines of the file:
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@@
 		(dnp no)
 		(fields_autoplaced yes)
-		(property "Reference" "C16"
+		(property "Reference" "C13"
 			(at 59.6963 62.23 90)
 			(effects
@@
 			(project "turbofrank"
 				(path "/8c0b3d8b-46d3-4173-ab1e-a61765f77d61/960439d1-a657-47b6-aee7-897565b7d217"
-					(reference "C16")
+					(reference "C13")
 					(unit 1)
 				)
@@
 		(dnp no)
 		(fields_autoplaced yes)
-		(property "Reference" "#PWR080"
+		(property "Reference" "#PWR073"
 			(at 99.06 36.83 0)
 			(effects
@@
 			(project ""
 				(path "/8c0b3d8b-46d3-4173-ab1e-a61765f77d61/960439d1-a657-47b6-aee7-897565b7d217"
-					(reference "#PWR080")
+					(reference "#PWR073")
 					(unit 1)
 				)
@@
 		(dnp no)
 		(fields_autoplaced yes)
-		(property "Reference" "#PWR083"
+		(property "Reference" "#PWR076"
 			(at 116.84 54.61 0)
 			(effects
@@
 			(project ""
 				(path "/8c0b3d8b-46d3-4173-ab1e-a61765f77d61/960439d1-a657-47b6-aee7-897565b7d217"
-					(reference "#PWR083")
+					(reference "#PWR076")
 					(unit 1)
 				)
@@
 		(dnp no)
 		(fields_autoplaced yes)
-		(property "Reference" "C17"
+		(property "Reference" "C14"
 			(at 48.2663 67.31 90)
 			(effects
@@
 			(project "turbofrank"
 				(path "/8c0b3d8b-46d3-4173-ab1e-a61765f77d61/960439d1-a657-47b6-aee7-897565b7d217"
-					(reference "C17")
+					(reference "C14")
 					(unit 1)
 				)
@@
 		(dnp no)
 		(fields_autoplaced yes)
-		(property "Reference" "C15"
+		(property "Reference" "C12"
 			(at 106.6863 50.8 90)
 			(effects
@@
 			(project ""
 				(path "/8c0b3d8b-46d3-4173-ab1e-a61765f77d61/960439d1-a657-47b6-aee7-897565b7d217"
-					(reference "C15")
+					(reference "C12")
 					(unit 1)
 				)
@@
 		(dnp no)
 		(fields_autoplaced yes)
-		(property "Reference" "#PWR081"
+		(property "Reference" "#PWR074"
 			(at 146.05 36.83 0)
 			(effects
@@
 			(project "frank2"
 				(path "/8c0b3d8b-46d3-4173-ab1e-a61765f77d61/960439d1-a657-47b6-aee7-897565b7d217"
-					(reference "#PWR081")
+					(reference "#PWR074")
 					(unit 1)
 				)
@@
 		(on_board yes)
 		(dnp no)
-		(property "Reference" "R58"
+		(property "Reference" "R54"
 			(at 144.78 41.91 90)
 			(effects
@@
 			(project "frank2"
 				(path "/8c0b3d8b-46d3-4173-ab1e-a61765f77d61/960439d1-a657-47b6-aee7-897565b7d217"
-					(reference "R58")
+					(reference "R54")
 					(unit 1)
 				)
@@
 		(on_board yes)
 		(dnp no)
-		(property "Reference" "C18"
+		(property "Reference" "C15"
 			(at 46.99 90.17 90)
 			(effects
@@
 			(project "turbofrank"
 				(path "/8c0b3d8b-46d3-4173-ab1e-a61765f77d61/960439d1-a657-47b6-aee7-897565b7d217"
-					(reference "C18")
+					(reference "C15")
 					(unit 1)
 				)
@@
 		(dnp no)
 		(fields_autoplaced yes)
-		(property "Reference" "#PWR082"
+		(property "Reference" "#PWR075"
 			(at 187.96 53.34 0)
 			(effects
@@
 			(project "frank2"
 				(path "/8c0b3d8b-46d3-4173-ab1e-a61765f77d61/960439d1-a657-47b6-aee7-897565b7d217"
-					(reference "#PWR082")
+					(reference "#PWR075")
 					(unit 1)
 				)
@@
 		(dnp no)
 		(fields_autoplaced yes)
-		(property "Reference" "U4"
+		(property "Reference" "U3"
 			(at 96.52 60.96 0)
 			(effects
@@
 			(project "frank2"
 				(path "/8c0b3d8b-46d3-4173-ab1e-a61765f77d61/960439d1-a657-47b6-aee7-897565b7d217"
-					(reference "U4")
+					(reference "U3")
 					(unit 1)
 				)
@@
 		(dnp no)
 		(fields_autoplaced yes)
-		(property "Reference" "#PWR085"
+		(property "Reference" "#PWR078"
 			(at 33.02 83.82 0)
 			(effects
@@
 			(project "frank2"
 				(path "/8c0b3d8b-46d3-4173-ab1e-a61765f77d61/960439d1-a657-47b6-aee7-897565b7d217"
-					(reference "#PWR085")
+					(reference "#PWR078")
 					(unit 1)
 				)
@@
 		(on_board yes)
 		(dnp no)
-		(property "Reference" "R57"
+		(property "Reference" "R53"
 			(at 97.79 41.91 90)
 			(effects
@@
 			(project "frank2"
 				(path "/8c0b3d8b-46d3-4173-ab1e-a61765f77d61/960439d1-a657-47b6-aee7-897565b7d217"
-					(reference "R57")
+					(reference "R53")
 					(unit 1)
 				)
@@
 		(on_board yes)
 		(dnp no)
-		(property "Reference" "#PWR084"
+		(property "Reference" "#PWR077"
 			(at 118.11 71.12 0)
 			(effects
@@
 			(project "frank2"
 				(path "/8c0b3d8b-46d3-4173-ab1e-a61765f77d61/960439d1-a657-47b6-aee7-897565b7d217"
-					(reference "#PWR084")
+					(reference "#PWR077")
 					(unit 1)
 				)
@@
 		(on_board yes)
 		(dnp no)
-		(property "Reference" "J23"
+		(property "Reference" "J20"
 			(at 220.98 50.8 0)
 			(effects
@@
 			(project "frank2"
 				(path "/8c0b3d8b-46d3-4173-ab1e-a61765f77d61/960439d1-a657-47b6-aee7-897565b7d217"
-					(reference "J23")
-					(unit 1)
-				)
+					(reference "J20")
+					(unit 1)
+				)

Commit message: TurboFRANK HW 1.05 Release
Other:
- moved on the sheet: C12, C13, C14, C15, D8, D9, J20, R53, R54, U3

Commit message: Bugfixes
Other:
- title: TurboFRANK -> ${NAME}
Changed lines of the file:
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@@
 	(paper "A4")
 	(title_block
-		(title "TurboFRANK")
-		(date "2025-04-04")
+		(title "${NAME}")
+		(date "2025-04-20")
 		(rev "${VERSION}")
 		(company "Mikhail Matveev")
