File: hardware/turbofrank/usb_hub.kicad_sch (KiCad schematic)
At the start: 2 parts, among them J22 USB HUB Data, U3 MW7211A

Commit message: TurboFRANK 1.04 WIP
Parts:
- added C43: 4.7u, FRANK:Capacitor (0805), symbol Device:C_Small
Connections:
- net GND: now also C43.2
- net VBUS: now also C43.1
Other:
- moved on the sheet: J22
Changed lines of the file:
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@@
+		(color 0 0 0 0)
+	)
+	(junction
+		(at 110.49 41.91)
+		(diameter 0)
 		(color 0 0 0 0)
 	)
@@
 	(wire
 		(pts
-			(xy 87.63 41.91) (xy 97.79 41.91)
+			(xy 110.49 59.69) (xy 110.49 58.42)
+		)
+		(stroke
+			(width 0)
+			(type default)
+		)
+	)
+	(wire
+		(pts
+			(xy 87.63 41.91) (xy 110.49 41.91)
 		)
 		(stroke
@@
 	(wire
 		(pts
-			(xy 127 36.83) (xy 146.05 36.83)
+			(xy 64.77 87.63) (xy 83.82 87.63)
 		)
 		(stroke
@@
 	(wire
 		(pts
-			(xy 127 34.29) (xy 146.05 34.29)
+			(xy 64.77 85.09) (xy 83.82 85.09)
 		)
 		(stroke
@@
 	(wire
 		(pts
+			(xy 110.49 41.91) (xy 113.03 41.91)
+		)
+		(stroke
+			(width 0)
+			(type default)
+		)
+	)
+	(wire
+		(pts
 			(xy 44.45 46.99) (xy 49.53 46.99)
 		)
@@
 	(wire
 		(pts
-			(xy 87.63 46.99) (xy 106.68 46.99)
-		)
-		(stroke
-			(width 0)
-			(type default)
-		)
-	)
-	(wire
-		(pts
-			(xy 87.63 49.53) (xy 106.68 49.53)
+			(xy 87.63 46.99) (xy 129.54 46.99)
+		)
+		(stroke
+			(width 0)
+			(type default)
+		)
+	)
+	(wire
+		(pts
+			(xy 87.63 49.53) (xy 129.54 49.53)
 		)
 		(stroke
@@
 		)
 	)
+	(wire
+		(pts
+			(xy 110.49 41.91) (xy 110.49 53.34)
+		)
+		(stroke
+			(width 0)
+			(type default)
+		)
+	)
 	(label "DP_IN"
-		(at 106.68 46.99 180)
+		(at 129.54 46.99 180)
 		(effects
 			(font
@@
 	)
 	(label "DM_IN"
-		(at 106.68 49.53 180)
+		(at 129.54 49.53 180)
 		(effects
 			(font
@@
 	)
 	(label "DM_IN"
-		(at 146.05 36.83 180)
+		(at 83.82 87.63 180)
 		(effects
 			(font
@@
 	)
 	(label "DP_IN"
-		(at 146.05 34.29 180)
+		(at 83.82 85.09 180)
 		(effects
 			(font
@@
 			)
 			(justify right)
+		)
+	)
+	(symbol
+		(lib_id "power:GND")
+		(at 110.49 59.69 0)
+		(unit 1)
+		(exclude_from_sim no)
+		(in_bom yes)
+		(on_board yes)
+		(dnp no)
+		(fields_autoplaced yes)
+		(property "Reference" "#PWR0140"
+			(at 110.49 66.04 0)
+			(effects
+				(font
+					(size 1.27 1.27)
+				)
+				(hide yes)
+			)
+		)
+		(property "Value" "GND"
+			(at 110.49 64.77 0)
+			(effects
+				(font
+					(size 1.27 1.27)
+				)
+			)
+		)
+		(property "Footprint" ""
+			(at 110.49 59.69 0)
+			(effects
+				(font
+					(size 1.27 1.27)
+				)
+				(hide yes)
+			)
+		)
+		(property "Datasheet" ""
+			(at 110.49 59.69 0)
+			(effects
+				(font
+					(size 1.27 1.27)
+				)
+				(hide yes)
+			)
+		)
+		(property "Description" "Power symbol creates a global label with name \"GND\" , ground"
+			(at 110.49 59.69 0)
+			(effects
+				(font
+					(size 1.27 1.27)
+				)
+				(hide yes)
+			)
+		)
+		(pin "1"
+		)
+		(instances
+			(project "turbofrank"
+				(path "/8c0b3d8b-46d3-4173-ab1e-a61765f77d61/2b27f9a5-aaa8-45c5-9eab-ce9c55507cf0"
+					(reference "#PWR0140")
+					(unit 1)
+				)
+			)
 		)
 	)
 	(symbol
 		(lib_id "power:VBUS")
-		(at 97.79 41.91 270)
+		(at 113.03 41.91 270)
 		(unit 1)
 		(exclude_from_sim no)
@@
 		(fields_autoplaced yes)
 		(property "Reference" "#PWR079"
-			(at 93.98 41.91 0)
+			(at 109.22 41.91 0)
 			(effects
 				(font
@@
 		)
 		(property "Value" "VBUS"
-			(at 101.6 41.9099 90)
+			(at 116.84 41.9099 90)
 			(effects
 				(font
@@
 		)
 		(property "Footprint" ""
-			(at 97.79 41.91 0)
+			(at 113.03 41.91 0)
 			(effects
 				(font
@@
 		)
 		(property "Datasheet" ""
-			(at 97.79 41.91 0)
+			(at 113.03 41.91 0)
 			(effects
 				(font
@@
 		)
 		(property "Description" "Power symbol creates a global label with name \"VBUS\""
-			(at 97.79 41.91 0)
+			(at 113.03 41.91 0)
 			(effects
 				(font
@@
 	)
 	(symbol
+		(lib_id "Device:C_Small")
+		(at 110.49 55.88 0)
+		(unit 1)
+		(exclude_from_sim no)
+		(in_bom yes)
+		(on_board yes)
+		(dnp no)
+		(property "Reference" "C43"
+			(at 113.538 56.134 90)
+			(effects
+				(font
+					(size 1.27 1.27)
+				)
+			)
+		)
+		(property "Value" "4.7u"
+			(at 107.696 56.134 90)
+			(effects
+				(font
+					(size 1.27 1.27)
+				)
+			)
+		)
+		(property "Footprint" "FRANK:Capacitor (0805)"
+			(at 110.49 55.88 0)
+			(effects
+				(font
+					(size 1.27 1.27)
+				)
+				(hide yes)
+			)
+		)
+		(property "Datasheet" "~"
+			(at 110.49 55.88 0)
+			(effects
+				(font
+					(size 1.27 1.27)
+				)
+				(hide yes)
+			)
+		)
+		(property "Description" "Unpolarized capacitor, small symbol"
+			(at 110.49 55.88 0)
+			(effects
+				(font
+					(size 1.27 1.27)
+				)
+				(hide yes)
+			)
+		)
+		(property "AliExpress" "https://www.aliexpress.com/item/33008008276.html"
+			(at 110.49 55.88 0)
+			(effects
+				(font
+					(size 1.27 1.27)
+				)
+				(hide yes)
+			)
+		)
+		(pin "1"
+		)
+		(pin "2"
+		)
+		(instances
+			(project "turbofrank"
+				(path "/8c0b3d8b-46d3-4173-ab1e-a61765f77d61/2b27f9a5-aaa8-45c5-9eab-ce9c55507cf0"
+					(reference "C43")
+					(unit 1)
+				)
+			)
+		)
+	)
+	(symbol
 		(lib_id "Connector:Conn_01x02_Pin")
-		(at 121.92 34.29 0)
+		(at 59.69 85.09 0)
 		(unit 1)
 		(exclude_from_sim no)
@@
 		(fields_autoplaced yes)
 		(property "Reference" "J22"
-			(at 122.555 29.21 0)
+			(at 60.325 80.01 0)
 			(effects
 				(font
@@
 		)
 		(property "Value" "USB HUB Data"
-			(at 122.555 31.75 0)
+			(at 60.325 82.55 0)
 			(effects
 				(font
@@
 		)
 		(property "Footprint" "FRANK:Connector Female ZH 1.50mm (2 pins)"
-			(at 121.92 34.29 0)
+			(at 59.69 85.09 0)
 			(effects
 				(font
@@
 		)
 		(property "Datasheet" "~"
-			(at 121.92 34.29 0)
+			(at 59.69 85.09 0)
 			(effects
 				(font
@@
 		)
 		(property "Description" "Generic connector, single row, 01x02, script generated"
-			(at 121.92 34.29 0)
-			(effects
-				(font
+			(at 59.69 85.09 0)
+			(effects
+				(font

Commit message: TurboFRANK HW 1.04 (release)
Parts:
- J22: footprint FRANK:Connector Female ZH 1.50mm (2 pins) -> FRANK:Connector Female ZH 1.50mm (2 pins + tracks)
- U3: footprint FRANK:SO-16 -> FRANK:SOP-16
Changed lines of the file:
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@@
 	(title_block
 		(title "TurboFRANK")
-		(date "2025-03-17")
+		(date "2025-03-19")
 		(rev "1.04")
 		(company "Mikhail Matveev")
@@
 			)
 		)
-		(property "Footprint" "FRANK:Connector Female ZH 1.50mm (2 pins)"
+		(property "Footprint" "FRANK:Connector Female ZH 1.50mm (2 pins + tracks)"
 			(at 59.69 85.09 0)
 			(effects
@@
 			)
 		)
-		(property "Footprint" "FRANK:SO-16"
+		(property "Footprint" "FRANK:SOP-16"
 			(at 68.58 43.18 0)
 			(effects

Commit message: TurboFRANK WIP
Parts:
- renumbered C43 to C14, J22 to J21
Changed lines of the file:
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@@
 		(dnp no)
 		(fields_autoplaced yes)
-		(property "Reference" "#PWR0140"
+		(property "Reference" "#PWR080"
 			(at 110.49 66.04 0)
 			(effects
@@
 			(project "turbofrank"
 				(path "/8c0b3d8b-46d3-4173-ab1e-a61765f77d61/2b27f9a5-aaa8-45c5-9eab-ce9c55507cf0"
-					(reference "#PWR0140")
+					(reference "#PWR080")
 					(unit 1)
 				)
@@
 		(on_board yes)
 		(dnp no)
-		(property "Reference" "C43"
+		(property "Reference" "C14"
 			(at 113.538 56.134 90)
 			(effects
@@
 			(project "turbofrank"
 				(path "/8c0b3d8b-46d3-4173-ab1e-a61765f77d61/2b27f9a5-aaa8-45c5-9eab-ce9c55507cf0"
-					(reference "C43")
+					(reference "C14")
 					(unit 1)
 				)
@@
 		(dnp no)
 		(fields_autoplaced yes)
-		(property "Reference" "J22"
+		(property "Reference" "J21"
 			(at 60.325 80.01 0)
 			(effects
@@
 			(project ""
 				(path "/8c0b3d8b-46d3-4173-ab1e-a61765f77d61/2b27f9a5-aaa8-45c5-9eab-ce9c55507cf0"
-					(reference "J22")
-					(unit 1)
-				)
+					(reference "J21")
+					(unit 1)
+				)

Commit message: TurboFRANK 1.05 HW
Parts:
- renumbered C14 to C40, U3 to U12
Other:
- moved on the sheet: J21
Changed lines of the file:
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@@
 	(title_block
 		(title "TurboFRANK")
-		(date "2025-03-19")
-		(rev "1.04")
+		(date "2025-04-04")
+		(rev "${VERSION}")
 		(company "Mikhail Matveev")
 		(comment 1 "https://github.com/xtremespb/frank")
@@
 	(wire
 		(pts
-			(xy 64.77 87.63) (xy 83.82 87.63)
+			(xy 62.23 72.39) (xy 80.01 72.39)
 		)
 		(stroke
@@
 	(wire
 		(pts
-			(xy 64.77 85.09) (xy 83.82 85.09)
+			(xy 62.23 69.85) (xy 80.01 69.85)
 		)
 		(stroke
@@
 	)
 	(label "DM_IN"
-		(at 83.82 87.63 180)
+		(at 80.01 72.39 180)
 		(effects
 			(font
@@
 	)
 	(label "DP_IN"
-		(at 83.82 85.09 180)
+		(at 80.01 69.85 180)
 		(effects
 			(font
@@
 		(dnp no)
 		(fields_autoplaced yes)
-		(property "Reference" "#PWR080"
+		(property "Reference" "#PWR0136"
 			(at 110.49 66.04 0)
 			(effects
@@
 		(instances
 			(project "turbofrank"
-				(path "/8c0b3d8b-46d3-4173-ab1e-a61765f77d61/2b27f9a5-aaa8-45c5-9eab-ce9c55507cf0"
-					(reference "#PWR080")
+				(path "/8c0b3d8b-46d3-4173-ab1e-a61765f77d61/c2769f78-f968-472a-a3d7-89c385b7d62d"
+					(reference "#PWR0136")
 					(unit 1)
 				)
@@
 		(dnp no)
 		(fields_autoplaced yes)
-		(property "Reference" "#PWR079"
+		(property "Reference" "#PWR0135"
 			(at 109.22 41.91 0)
 			(effects
@@
 		(instances
 			(project ""
-				(path "/8c0b3d8b-46d3-4173-ab1e-a61765f77d61/2b27f9a5-aaa8-45c5-9eab-ce9c55507cf0"
-					(reference "#PWR079")
+				(path "/8c0b3d8b-46d3-4173-ab1e-a61765f77d61/c2769f78-f968-472a-a3d7-89c385b7d62d"
+					(reference "#PWR0135")
 					(unit 1)
 				)
@@
 		(dnp no)
 		(fields_autoplaced yes)
-		(property "Reference" "#PWR078"
+		(property "Reference" "#PWR0134"
 			(at 104.14 34.29 0)
 			(effects
@@
 		(instances
 			(project "turbofrank"
-				(path "/8c0b3d8b-46d3-4173-ab1e-a61765f77d61/2b27f9a5-aaa8-45c5-9eab-ce9c55507cf0"
-					(reference "#PWR078")
+				(path "/8c0b3d8b-46d3-4173-ab1e-a61765f77d61/c2769f78-f968-472a-a3d7-89c385b7d62d"
+					(reference "#PWR0134")
 					(unit 1)
 				)
@@
 		(on_board yes)
 		(dnp no)
-		(property "Reference" "C14"
+		(property "Reference" "C40"
 			(at 113.538 56.134 90)
 			(effects
@@
 		(instances
 			(project "turbofrank"
-				(path "/8c0b3d8b-46d3-4173-ab1e-a61765f77d61/2b27f9a5-aaa8-45c5-9eab-ce9c55507cf0"
-					(reference "C14")
+				(path "/8c0b3d8b-46d3-4173-ab1e-a61765f77d61/c2769f78-f968-472a-a3d7-89c385b7d62d"
+					(reference "C40")
 					(unit 1)
 				)
@@
 	(symbol
 		(lib_id "Connector:Conn_01x02_Pin")
-		(at 59.69 85.09 0)
+		(at 57.15 69.85 0)
 		(unit 1)
 		(exclude_from_sim no)
@@
 		(fields_autoplaced yes)
 		(property "Reference" "J21"
-			(at 60.325 80.01 0)
+			(at 57.785 64.77 0)
 			(effects
 				(font
@@
 		)
 		(property "Value" "USB HUB Data"
-			(at 60.325 82.55 0)
+			(at 57.785 67.31 0)
 			(effects
 				(font
@@
 		)
 		(property "Footprint" "FRANK:Connector Female ZH 1.50mm (2 pins + tracks)"
-			(at 59.69 85.09 0)
+			(at 57.15 69.85 0)
 			(effects
 				(font
@@
 		)
 		(property "Datasheet" "~"
-			(at 59.69 85.09 0)
+			(at 57.15 69.85 0)
 			(effects
 				(font
@@
 		)
 		(property "Description" "Generic connector, single row, 01x02, script generated"
-			(at 59.69 85.09 0)
+			(at 57.15 69.85 0)
 			(effects
 				(font
@@
 		(instances
 			(project ""
-				(path "/8c0b3d8b-46d3-4173-ab1e-a61765f77d61/2b27f9a5-aaa8-45c5-9eab-ce9c55507cf0"
+				(path "/8c0b3d8b-46d3-4173-ab1e-a61765f77d61/c2769f78-f968-472a-a3d7-89c385b7d62d"
 					(reference "J21")
 					(unit 1)
@@
 		(dnp no)
 		(fields_autoplaced yes)
-		(property "Reference" "U3"
+		(property "Reference" "U12"
 			(at 68.58 24.13 0)
 			(effects
@@
 		(instances
 			(project "turbofrank"
-				(path "/8c0b3d8b-46d3-4173-ab1e-a61765f77d61/2b27f9a5-aaa8-45c5-9eab-ce9c55507cf0"
-					(reference "U3")
+				(path "/8c0b3d8b-46d3-4173-ab1e-a61765f77d61/c2769f78-f968-472a-a3d7-89c385b7d62d"
+					(reference "U12")
 					(unit 1)
 				)

Commit message: TurboFRANK HW 1.05 Release
Parts:
- J21: AliExpress (none) -> https://www.aliexpress.com/item/1005001649158434.html
- U12: AliExpress (none) -> https://www.aliexpress.com/item/1005007446137541.html
Other:
- moved on the sheet: C40, J21, U12

Commit message: Bugfixes
Other:
- title: TurboFRANK -> ${NAME}
Changed lines of the file:
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@@
 	(paper "A4")
 	(title_block
-		(title "TurboFRANK")
-		(date "2025-04-04")
+		(title "${NAME}")
+		(date "2025-04-20")
 		(rev "${VERSION}")
 		(company "Mikhail Matveev")
@@
 	(wire
 		(pts
-			(xy 179.07 85.09) (xy 181.61 85.09)
+			(xy 179.07 85.09) (xy 191.77 85.09)
 		)
 		(stroke
@@
 			)
 			(justify right)
+		)
+	)
+	(hierarchical_label "VBUS"
+		(shape input)
+		(at 191.77 85.09 0)
+		(effects
+			(font
+				(size 1.27 1.27)
+			)
+			(justify left)
 		)
 	)
@@
 	)
 	(symbol
-		(lib_id "power:VBUS")
-		(at 181.61 85.09 270)
-		(unit 1)
-		(exclude_from_sim no)
-		(in_bom yes)
-		(on_board yes)
-		(dnp no)
-		(fields_autoplaced yes)
-		(property "Reference" "#PWR0135"
-			(at 177.8 85.09 0)
-			(effects
-				(font
-					(size 1.27 1.27)
-				)
-				(hide yes)
-			)
-		)
-		(property "Value" "VBUS"
-			(at 185.42 85.0899 90)
-			(effects
-				(font
-					(size 1.27 1.27)
-				)
-				(justify left)
-			)
-		)
-		(property "Footprint" ""
-			(at 181.61 85.09 0)
-			(effects
-				(font
-					(size 1.27 1.27)
-				)
-				(hide yes)
-			)
-		)
-		(property "Datasheet" ""
-			(at 181.61 85.09 0)
-			(effects
-				(font
-					(size 1.27 1.27)
-				)
-				(hide yes)
-			)
-		)
-		(property "Description" "Power symbol creates a global label with name \"VBUS\""
-			(at 181.61 85.09 0)
-			(effects
-				(font
-					(size 1.27 1.27)
-				)
-				(hide yes)
-			)
-		)
-		(pin "1"
-		)
-		(instances
-			(project ""
-				(path "/8c0b3d8b-46d3-4173-ab1e-a61765f77d61/c2769f78-f968-472a-a3d7-89c385b7d62d"
-					(reference "#PWR0135")
-					(unit 1)
-				)
-			)
-		)
-	)
-	(symbol
 		(lib_id "power:GND")
 		(at 166.37 77.47 90)
@@
 					(size 1.27 1.27)
 				)
+				(hide yes)
 			)
 		)
@@
 					(size 1.27 1.27)
 				)
-			)
-		)
+				(hide yes)
+			)
+		)

Commit message: TurboFRANK HW 1.07
Parts:
- renumbered C40 to C23, U12 to U9
Changed lines of the file:
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@@
 	(title_block
 		(title "${NAME}")
-		(date "2025-04-20")
+		(date "2025-05-01")
 		(rev "${VERSION}")
 		(company "Mikhail Matveev")
@@
 		(dnp no)
 		(fields_autoplaced yes)
-		(property "Reference" "#PWR0136"
+		(property "Reference" "#PWR0109"
 			(at 179.07 109.22 0)
 			(effects
@@
 			(project "turbofrank"
 				(path "/8c0b3d8b-46d3-4173-ab1e-a61765f77d61/c2769f78-f968-472a-a3d7-89c385b7d62d"
-					(reference "#PWR0136")
+					(reference "#PWR0109")
 					(unit 1)
 				)
@@
 		(dnp no)
 		(fields_autoplaced yes)
-		(property "Reference" "#PWR0134"
+		(property "Reference" "#PWR0108"
 			(at 172.72 77.47 0)
 			(effects
@@
 			(project "turbofrank"
 				(path "/8c0b3d8b-46d3-4173-ab1e-a61765f77d61/c2769f78-f968-472a-a3d7-89c385b7d62d"
-					(reference "#PWR0134")
+					(reference "#PWR0108")
 					(unit 1)
 				)
@@
 		(on_board yes)
 		(dnp no)
-		(property "Reference" "C40"
+		(property "Reference" "C23"
 			(at 182.118 99.314 90)
 			(effects
@@
 			(project "turbofrank"
 				(path "/8c0b3d8b-46d3-4173-ab1e-a61765f77d61/c2769f78-f968-472a-a3d7-89c385b7d62d"
-					(reference "C40")
+					(reference "C23")
 					(unit 1)
 				)
@@
 		(dnp no)
 		(fields_autoplaced yes)
-		(property "Reference" "U12"
+		(property "Reference" "U9"
 			(at 137.16 67.31 0)
 			(effects
@@
 			(project "turbofrank"
 				(path "/8c0b3d8b-46d3-4173-ab1e-a61765f77d61/c2769f78-f968-472a-a3d7-89c385b7d62d"
-					(reference "U12")
+					(reference "U9")
 					(unit 1)
 				)
