File: hardware/turbofrank/usbstack.kicad_sch (KiCad schematic)
At the start: 7 parts

Commit message: TurboFRANK 1.04 WIP
Parts:
- renumbered C30 to C6, C31 to C7, USB2 to J7, R82 to R12, R83 to R13, R84 to R14, R85 to R15
Changed lines of the file:
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@@
 	(title_block
 		(title "TurboFRANK")
-		(date "2025-03-03")
-		(rev "1.03")
+		(date "2025-03-17")
+		(rev "1.04")
 		(company "Mikhail Matveev")
 		(comment 1 "https://github.com/xtremespb/frank")
@@
 		(dnp no)
 		(fields_autoplaced yes)
-		(property "Reference" "USB2"
+		(property "Reference" "J7"
 			(at 38.1 30.48 0)
 			(effects
@@
 		)
 		(instances
-			(project "usb2ps2"
+			(project "turbofrank"
+				(path "/8c0b3d8b-46d3-4173-ab1e-a61765f77d61/363c63a2-6afd-440e-9891-102dc1fa9944"
+					(reference "J7")
+					(unit 1)
+				)
 				(path "/8c0b3d8b-46d3-4173-ab1e-a61765f77d61/b237c830-8b62-42ca-9271-338aede27b72"
-					(reference "USB2")
+					(reference "J18")
 					(unit 1)
 				)
@@
 		(on_board yes)
 		(dnp no)
-		(property "Reference" "C30"
+		(property "Reference" "C6"
 			(at 84.201 44.5516 0)
 			(effects
@@
 		)
 		(instances
-			(project "usb2ps2"
+			(project "turbofrank"
+				(path "/8c0b3d8b-46d3-4173-ab1e-a61765f77d61/363c63a2-6afd-440e-9891-102dc1fa9944"
+					(reference "C6")
+					(unit 1)
+				)
 				(path "/8c0b3d8b-46d3-4173-ab1e-a61765f77d61/b237c830-8b62-42ca-9271-338aede27b72"
-					(reference "C30")
+					(reference "C12")
 					(unit 1)
 				)
@@
 		(on_board yes)
 		(dnp no)
-		(property "Reference" "R84"
+		(property "Reference" "R14"
 			(at 61.722 66.04 90)
 			(effects
@@
 		)
 		(instances
-			(project "usb2ps2"
+			(project "turbofrank"
+				(path "/8c0b3d8b-46d3-4173-ab1e-a61765f77d61/363c63a2-6afd-440e-9891-102dc1fa9944"
+					(reference "R14")
+					(unit 1)
+				)
 				(path "/8c0b3d8b-46d3-4173-ab1e-a61765f77d61/b237c830-8b62-42ca-9271-338aede27b72"
-					(reference "R84")
+					(reference "R33")
 					(unit 1)
 				)
@@
 		(on_board yes)
 		(dnp no)
-		(property "Reference" "C31"
+		(property "Reference" "C7"
 			(at 95.631 44.5516 0)
 			(effects
@@
 		)
 		(instances
-			(project "usb2ps2"
+			(project "turbofrank"
+				(path "/8c0b3d8b-46d3-4173-ab1e-a61765f77d61/363c63a2-6afd-440e-9891-102dc1fa9944"
+					(reference "C7")
+					(unit 1)
+				)
 				(path "/8c0b3d8b-46d3-4173-ab1e-a61765f77d61/b237c830-8b62-42ca-9271-338aede27b72"
-					(reference "C31")
+					(reference "C13")
 					(unit 1)
 				)
@@
 		(on_board yes)
 		(dnp no)
-		(property "Reference" "#PWR098"
+		(property "Reference" "#PWR033"
 			(at 52.07 40.64 0)
 			(effects
@@
 		)
 		(instances
-			(project "usb2ps2"
+			(project "turbofrank"
+				(path "/8c0b3d8b-46d3-4173-ab1e-a61765f77d61/363c63a2-6afd-440e-9891-102dc1fa9944"
+					(reference "#PWR033")
+					(unit 1)
+				)
 				(path "/8c0b3d8b-46d3-4173-ab1e-a61765f77d61/b237c830-8b62-42ca-9271-338aede27b72"
-					(reference "#PWR098")
+					(reference "#PWR068")
 					(unit 1)
 				)
@@
 		(on_board yes)
 		(dnp no)
-		(property "Reference" "#PWR0100"
+		(property "Reference" "#PWR035"
 			(at 81.28 57.15 0)
 			(effects
@@
 		)
 		(instances
-			(project "usb2ps2"
+			(project "turbofrank"
+				(path "/8c0b3d8b-46d3-4173-ab1e-a61765f77d61/363c63a2-6afd-440e-9891-102dc1fa9944"
+					(reference "#PWR035")
+					(unit 1)
+				)
 				(path "/8c0b3d8b-46d3-4173-ab1e-a61765f77d61/b237c830-8b62-42ca-9271-338aede27b72"
-					(reference "#PWR0100")
+					(reference "#PWR070")
 					(unit 1)
 				)
@@
 		(on_board yes)
 		(dnp no)
-		(property "Reference" "R83"
+		(property "Reference" "R13"
 			(at 70.612 64.77 90)
 			(effects
@@
 		)
 		(instances
-			(project "usb2ps2"
+			(project "turbofrank"
+				(path "/8c0b3d8b-46d3-4173-ab1e-a61765f77d61/363c63a2-6afd-440e-9891-102dc1fa9944"
+					(reference "R13")
+					(unit 1)
+				)
 				(path "/8c0b3d8b-46d3-4173-ab1e-a61765f77d61/b237c830-8b62-42ca-9271-338aede27b72"
-					(reference "R83")
+					(reference "R32")
 					(unit 1)
 				)
@@
 		(on_board yes)
 		(dnp no)
-		(property "Reference" "#PWR0101"
+		(property "Reference" "#PWR036"
 			(at 92.71 57.15 0)
 			(effects
@@
 		)
 		(instances
-			(project "usb2ps2"
+			(project "turbofrank"
+				(path "/8c0b3d8b-46d3-4173-ab1e-a61765f77d61/363c63a2-6afd-440e-9891-102dc1fa9944"
+					(reference "#PWR036")
+					(unit 1)
+				)
 				(path "/8c0b3d8b-46d3-4173-ab1e-a61765f77d61/b237c830-8b62-42ca-9271-338aede27b72"
-					(reference "#PWR0101")
+					(reference "#PWR071")
 					(unit 1)
 				)
@@
 		(on_board yes)
 		(dnp no)
-		(property "Reference" "R82"
+		(property "Reference" "R12"
 			(at 57.912 59.69 90)
 			(effects
@@
 		)
 		(instances
-			(project "usb2ps2"
+			(project "turbofrank"
+				(path "/8c0b3d8b-46d3-4173-ab1e-a61765f77d61/363c63a2-6afd-440e-9891-102dc1fa9944"
+					(reference "R12")
+					(unit 1)
+				)
 				(path "/8c0b3d8b-46d3-4173-ab1e-a61765f77d61/b237c830-8b62-42ca-9271-338aede27b72"
-					(reference "R82")
+					(reference "R31")
 					(unit 1)
 				)
@@
 		(on_board yes)
 		(dnp no)
-		(property "Reference" "#PWR099"
+		(property "Reference" "#PWR034"
 			(at 58.42 40.64 0)
 			(effects
@@
 		)
 		(instances
-			(project "usb2ps2"
+			(project "turbofrank"
+				(path "/8c0b3d8b-46d3-4173-ab1e-a61765f77d61/363c63a2-6afd-440e-9891-102dc1fa9944"
+					(reference "#PWR034")
+					(unit 1)
+				)
 				(path "/8c0b3d8b-46d3-4173-ab1e-a61765f77d61/b237c830-8b62-42ca-9271-338aede27b72"
-					(reference "#PWR099")
+					(reference "#PWR069")
 					(unit 1)
 				)
@@
 		(dnp no)
 		(fields_autoplaced yes)
-		(property "Reference" "#PWR0102"
+		(property "Reference" "#PWR037"
 			(at 38.1 73.66 0)
 			(effects
@@
 		)
 		(instances
-			(project ""
+			(project "turbofrank"
+				(path "/8c0b3d8b-46d3-4173-ab1e-a61765f77d61/363c63a2-6afd-440e-9891-102dc1fa9944"
+					(reference "#PWR037")
+					(unit 1)
+				)
 				(path "/8c0b3d8b-46d3-4173-ab1e-a61765f77d61/b237c830-8b62-42ca-9271-338aede27b72"
-					(reference "#PWR0102")
+					(reference "#PWR072")
 					(unit 1)
 				)
@@
 		(on_board yes)
 		(dnp no)
-		(property "Reference" "R85"
+		(property "Reference" "R15"
 			(at 74.422 71.12 90)
 			(effects
@@
 		)
 		(instances
-			(project "usb2ps2"
+			(project "turbofrank"
+				(path "/8c0b3d8b-46d3-4173-ab1e-a61765f77d61/363c63a2-6afd-440e-9891-102dc1fa9944"
+					(reference "R15")
+					(unit 1)
+				)
 				(path "/8c0b3d8b-46d3-4173-ab1e-a61765f77d61/b237c830-8b62-42ca-9271-338aede27b72"
-					(reference "R85")
-					(unit 1)
-				)
+					(reference "R34")
+					(unit 1)
+				)

Commit message: TurboFRANK WIP
Parts:
- renumbered C7 to C10, C6 to C9, J7 to J16, R12 to R27, R13 to R28, R14 to R29, R15 to R30
Other:
- moved on the sheet: C10, C9, J16, R27, R28, R29, R30

Commit message: Bugfixes
Other:
- title: TurboFRANK -> ${NAME}
Changed lines of the file:
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@@
 	(paper "A4")
 	(title_block
-		(title "TurboFRANK")
-		(date "2025-04-04")
+		(title "${NAME}")
+		(date "2025-04-20")
 		(rev "${VERSION}")
 		(company "Mikhail Matveev")
