File: hardware/hdmi2vga/softcomp.kicad_sch (KiCad schematic)
At the start: 10 parts

Commit message: Minor updates
Parts:
- renumbered SC1 to J6
Changed lines of the file:
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@@
 	(title_block
 		(title "HDMI to VGA Passive Adapter")
-		(date "2025-03-04")
-		(rev "2.01")
+		(date "2025-04-01")
+		(rev "2.02")
 		(company "Mikhail Matveev")
 		(comment 1 "https://github.com/xtremespb/frank")
@@
 		(dnp no)
 		(fields_autoplaced yes)
-		(property "Reference" "SC1"
+		(property "Reference" "J6"
 			(at 100.33 31.7499 0)
 			(effects
@@
 			(project "CMZJ2"
 				(path "/8c0b3d8b-46d3-4173-ab1e-a61765f77d61/41f3c986-8cc8-43f4-917d-7c89a2c675d6"
-					(reference "SC1")
+					(reference "J6")
 					(unit 1)
 				)
