File: hardware/hdmi2vga/hdmi2vga.kicad_pcb (KiCad board)
At the start: 2 copper layers, 0 parts

Commit message: Revision 2.03
Parts:
- added H1: MountingHole, FRANK:Mounting Hole (2.7mm), F.Cu at (119.0, 54.2)
- added H2: MountingHole, FRANK:Mounting Hole (2.7mm), F.Cu at (142.5, 54.2)
- added J1: HDMI, FRANK:HDMI (male), F.Cu at (130.8, 48.2)
- added J2: VGA, FRANK:D-SUB (15 pin, female), F.Cu at (135.0, 61.2)
- added L1: HDMI LED, FRANK:LED (0805), F.Cu at (126.0, 56.0)
- added R1: 1K, FRANK:Resistor (0805), F.Cu at (128.2, 56.0)
- added R2: 820R, FRANK:Resistor (0805), F.Cu at (135.0, 56.0)
- added R3: 820R, FRANK:Resistor (0805), F.Cu at (132.8, 56.0)
- added R4: 820R, FRANK:Resistor (0805), F.Cu at (130.5, 56.0)
Routing:
- net /D2P_VGA_VS: track 0.00 -> 31.1 mm
- net /D2N_VGA_HS: track 0.00 -> 27.6 mm
- net GND: track 0.00 -> 19.0 mm, vias 0 -> 6
- net /CLKP_VGA_BH: track 0.00 -> 18.1 mm
- net /D1P_VGA_RH: track 0.00 -> 16.2 mm, vias 0 -> 1
- net /D0P_VGA_GH: track 0.00 -> 14.5 mm
- net /D1N_VGA_R: track 0.00 -> 12.5 mm, vias 0 -> 1
- net Net-(J1-+5V): track 0.00 -> 9.70 mm, vias 0 -> 1
- net /CLKN_VGA_B: track 0.00 -> 9.39 mm, vias 0 -> 1
- net /D0N_VGA_G: track 0.00 -> 7.72 mm
- net Net-(L1-A): track 0.00 -> 2.27 mm
Other:
- board outline added: 31.1 x 21.8 mm
