File: hardware/minifrank_rm1/reset.kicad_sch (KiCad schematic)
At the start: 1 part, among them SW2 Reset Button

Commit message: Minor updates
Parts:
- SW3: renamed from SW2; value Reset Button -> KLS7-TS3302; AliExpress https://www.aliexpress.com/item/1005001629293584.html -> https://www.aliexpress.com/item/1005007359248990.html
Other:
- title: MiniFRANK RM1 -> TurboFRANK
Changed lines of the file:
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@@
 	(paper "A4")
 	(title_block
-		(title "MiniFRANK RM1")
-		(date "2025-03-16")
-		(rev "2.02")
+		(title "TurboFRANK")
+		(date "2025-03-03")
+		(rev "1.02")
 		(company "Mikhail Matveev")
 		(comment 1 "https://github.com/xtremespb/frank")
@@
 		(on_board yes)
 		(dnp no)
-		(property "Reference" "SW2"
+		(property "Reference" "SW3"
 			(at 62.484 49.022 0)
 			(effects
@@
 			)
 		)
-		(property "Value" "Reset Button"
+		(property "Value" "KLS7-TS3302"
 			(at 62.484 51.562 0)
 			(effects
@@
 			)
 		)
-		(property "AliExpress" "https://www.aliexpress.com/item/1005001629293584.html"
+		(property "AliExpress" "https://www.aliexpress.com/item/1005007359248990.html"
 			(at 48.26 59.69 0)
 			(effects
@@
 			(project "frank2"
 				(path "/8c0b3d8b-46d3-4173-ab1e-a61765f77d61/44b0fc63-213a-4da4-a0e4-3ab9f837f02d"
-					(reference "SW2")
+					(reference "SW3")
 					(unit 1)
 				)
@@
 		(dnp no)
 		(fields_autoplaced yes)
-		(property "Reference" "#PWR044"
+		(property "Reference" "#PWR068"
 			(at 48.26 41.91 0)
 			(effects
@@
 			(project "frank2"
 				(path "/8c0b3d8b-46d3-4173-ab1e-a61765f77d61/44b0fc63-213a-4da4-a0e4-3ab9f837f02d"
-					(reference "#PWR044")
+					(reference "#PWR068")
 					(unit 1)
 				)
