File: hardware/minifrank_rm1/minifrank_rm1.kicad_pcb (KiCad board)
At the start: 2 copper layers, 76 x 56.5 mm, 102 parts, among them J1 D-SUB 9 Male, J2 0475710001, J3 104031-0811, J4 PJ-320D, J5 FRANK:Jack (3.5mm, PJ-320D), J6 D-SUB 9 Male, J7 MDC-036, J8 DC3RX19JA2, Q1 BC850, Q2 BC850, U1 NCP1117 3.3, U2 W25Q128JVSIQ, U3 RP2040, U4 TDA1387T, U5 ESP-PSRAM32, Y1 12 MHz

Commit message: Update minifrank_rm1.kicad_pcb
Parts:
- moved C19 0.62 mm to (169.9, 47.8)
- moved C22 0.62 mm to (169.9, 52.5)
- moved R11 0.50 mm to (175.0, 53.5)
- moved R12 0.50 mm to (179.2, 53.5)
- moved J4 0.20 mm to (172.8, 72.2)
- moved J5 0.20 mm to (172.8, 62.2)
Routing:
- net VBUS: track 0.00 -> 279.7 mm
- net +3V3: track 5.78 -> 116.2 mm, vias 2 -> 5
- net /GPIO14: track 5.42 -> 100.3 mm, vias 0 -> 1
- net /GPIO15: track 5.59 -> 93.7 mm, vias 0 -> 2
- net /RP2040/GPIO25: track 6.87 -> 57.8 mm, vias 0 -> 2
- net /GPIO28: track 6.94 -> 38.0 mm, vias 0 -> 1
- net /GPIO18: track 7.02 -> 36.9 mm
- net /GPIO27: track 6.91 -> 36.1 mm, vias 0 -> 1
- net /GPIO22: track 7.12 -> 35.7 mm, vias 0 -> 2
- net /GPIO19: track 7.04 -> 33.1 mm, vias 0 -> 2
- net Net-(USB1-SHIELD): track 0.00 -> 24.4 mm
- net /GPIO20: track 7.04 -> 31.4 mm, vias 0 -> 2
- net /D+: track 0.00 -> 16.1 mm
- net /GPIO26: track 6.85 -> 22.4 mm, vias 0 -> 1
- net /D-: track 0.00 -> 14.5 mm
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
Commit message: WIP
Routing:
- net /KB_CLK: track 2.25 -> 63.4 mm, vias 0 -> 3
- net /KB_DATA: track 2.25 -> 56.1 mm, vias 0 -> 1
- net /A_OUTL: track 0.00 -> 42.1 mm, vias 0 -> 2
- net /A_OUTB: track 0.00 -> 41.6 mm, vias 0 -> 1
- net Net-(J6-Pad2): track 0.00 -> 38.9 mm, vias 0 -> 2
- net /Audio Out/L: track 0.00 -> 31.2 mm, vias 0 -> 2
- net /GPIO28: track 38.0 -> 68.7 mm
- net Net-(C22-Pad1): track 0.00 -> 28.2 mm
- net /Audio Out/R: track 0.00 -> 28.1 mm, vias 0 -> 2
- net Net-(J1-Pad2): track 0.00 -> 27.0 mm, vias 0 -> 1
- net /GPIO27: track 36.1 -> 62.7 mm
- net /GPIO26: track 22.4 -> 48.2 mm
- net /MS_DATA: track 0.00 -> 20.6 mm
- net Net-(C19-Pad1): track 0.00 -> 16.5 mm
- net /A_TDAR: track 0.00 -> 16.5 mm, vias 0 -> 1
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
Commit message: WIP
Routing:
- net VBUS: track 289.5 -> 284.0 mm
- net /KB_DATA: track 56.1 -> 54.4 mm
- net /GPIO27: track 62.7 -> 64.3 mm
- net Net-(J8-CLKN): track 11.5 -> 10.0 mm
- net /GPIO4: track 38.6 -> 37.2 mm
- net /RP2040/XIN: track 12.2 -> 10.9 mm
- net Net-(J8-CLKP): track 10.2 -> 9.05 mm
- net Net-(U3-USB_DP): track 10.7 -> 9.62 mm
- net /GPIO13: track 16.3 -> 15.2 mm
- net /GPIO5: track 49.7 -> 48.7 mm
- net Net-(J8-D0N): track 9.10 -> 8.15 mm
- net Net-(J8-D1N): track 8.27 -> 7.32 mm
- net Net-(J8-D2P): track 7.56 -> 6.69 mm
- net Net-(U3-USB_DM): track 12.5 -> 11.7 mm
- net Net-(U3-VREG_VOUT): track 33.2 -> 32.4 mm
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
Commit message: MiniFRANK RM1 2.03
Routing:
- net /RP2040/GPIO25: track 61.3 -> 63.1 mm
- net /GPIO26: track 48.2 -> 49.1 mm
- net Net-(U3-USB_DM): track 11.7 -> 11.1 mm
- net GND: vias 34 -> 35
Other:
- board text added: "2.03"
- board text added: "MiniFRANK"
- board text added: "RM1"
- board text added: "rh1.tech"

Commit message: WIP
Parts:
- removed C26: 100n, FRANK:Capacitor (0805)
- removed JP3: Mouse DATA, FRANK:Pin Header (1x02)
- removed JP4: Jumper (Solder), FRANK:Jumper (solder)
- added C29: 10u, FRANK:Capacitor (0805), F.Cu at (181.7, 69.2)
- added C30: 10u, FRANK:Capacitor (0805), F.Cu at (178.2, 61.0)
- added C31: 47n, FRANK:Capacitor (0805), F.Cu at (185.0, 76.8)
- added C32: 47n, FRANK:Capacitor (0805), F.Cu at (184.0, 79.2)
- added C33: 10u, FRANK:Capacitor (0805), F.Cu at (168.0, 82.8)
- added C34: 10u, FRANK:Capacitor (0805), F.Cu at (168.0, 85.5)
- added C35: 100n, FRANK:Capacitor (0805), F.Cu at (162.8, 87.1)
- added R39: 10K, FRANK:Resistor (0805), F.Cu at (170.8, 61.8)
- added R40: 47K, FRANK:Resistor (0805), F.Cu at (173.0, 61.8)
- added R41: 10K, FRANK:Resistor (0805), F.Cu at (192.5, 75.8)
- added R42: 47K, FRANK:Resistor (0805), F.Cu at (191.0, 73.5)
- added R43: 20K, FRANK:Resistor (0805), F.Cu at (181.8, 71.5)
- added R44: 10K, FRANK:Resistor (0805), F.Cu at (178.2, 58.8)
- added R45: 2K, FRANK:Resistor (0805), F.Cu at (180.5, 76.8)
- added R46: 2K, FRANK:Resistor (0805), F.Cu at (179.5, 79.2)
- added R47: 10K, FRANK:Resistor (0805), F.Cu at (185.0, 74.2)
- added R48: 10K, FRANK:Resistor (0805), F.Cu at (184.0, 82.0)
- added R49: 1K, FRANK:Resistor (0805), F.Cu at (179.5, 82.0)
- added R50: 1K, FRANK:Resistor (0805), F.Cu at (180.5, 74.2)
- added R51: 2K, FRANK:Resistor (0805), F.Cu at (186.5, 71.8)
- added R52: 2K, FRANK:Resistor (0805), F.Cu at (189.2, 81.0)
- added R53: 470R, FRANK:Resistor (0805), F.Cu at (168.0, 80.0)
- added R54: 470R, FRANK:Resistor (0805), F.Cu at (168.0, 88.2)
- added U6: TDA1387T, FRANK:SO-8, F.Cu at (161.0, 81.8)
- C19, C22: value 10u -> 100n; footprint FRANK:Capacitor (3528, tantalum, polar) -> FRANK:Capacitor (0805)
- C20, C23: value 10n -> 100n
- C21: value 10u -> 100n
- C24, C27, C28: value 100n -> 10u
- J4: value PJ-320D -> ~
- JP1: value SW_DIP_x05 -> SW_DIP_x06; footprint FRANK:DIP Switch (5x5) -> FRANK:DIP Switch (6)
- JP2: value Mouse CLK -> Jumper (Solder); footprint FRANK:Pin Header (1x02) -> FRANK:Jumper (solder); moved to B.Cu
- R11: value 1K -> 10K
- R12, R16: value 330R -> 1K
- R13, R14: value 2K -> 10K
- R15, R18, R23: value 1K -> 100R
- R17, R20: value 10K -> 1K
- R19: value 10K -> 100R
- R21: value 100R -> 1K
- R25, R29, R30: value 100R -> 270R
- R26, R27, R28: value 1K -> 270R
- R33, R34: value 270R -> 2K
- R35, R36, R37: value 270R -> 10K
- R38: value 270R -> 20K
- U4: value TDA1387T -> ESP-PSRAM32
- U5: value ESP-PSRAM32 -> LM358
- moved JP2 47.7 mm to (218.8, 82.0), turned to -90 degrees
- moved U5 46.1 mm to (174.1, 70.6), turned to 180 degrees
- moved C23 44.5 mm to (222.5, 47.8)
- moved C28 44.2 mm to (192.5, 78.0), turned to 0 degrees
- moved LD1 43.1 mm to (212.0, 81.2), turned to 180 degrees
- moved U4 42.8 mm to (219.0, 80.5)
- moved R22 41.5 mm to (199.0, 41.5), turned to 90 degrees
- moved R20 41.5 mm to (227.0, 42.0), turned to 90 degrees
- moved R19 41.0 mm to (229.5, 42.0), turned to -90 degrees
- moved C21 40.3 mm to (220.8, 76.5), turned to 180 degrees
- moved R10 39.3 mm to (208.0, 81.2), turned to 180 degrees
- moved R23 38.0 mm to (191.5, 41.5), turned to -90 degrees
- moved R17 35.5 mm to (222.0, 42.0)
- moved R34 33.9 mm to (192.5, 82.5), turned to 180 degrees
- moved C24 33.2 mm to (172.3, 75.2), turned to 180 degrees
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Connections:
- C19 pad 1: Net-(C19-Pad1) -> +3V3
- C19 pad 2: /Audio Out/L -> GND
- C20 pad 1: Net-(C19-Pad1) -> Net-(C20-Pad1)
- C20 pad 2: GND -> Net-(C20-Pad2)
- C21 pad 1: Net-(U4-FLT) -> +3V3
- C22 pad 1: Net-(C22-Pad1) -> VBUS
- C22 pad 2: /Audio Out/R -> GND
- C23 pad 1: Net-(C22-Pad1) -> VBUS
- C24 pad 1: +3V3 -> GND
- C24 pad 2: GND -> VBUS
- C25 pad 1: Net-(C25-Pad1) -> GND
- C25 pad 2: Net-(C25-Pad2) -> VBUS
- C27 pad 1: VBUS -> Net-(C27-Pad1)
- C27 pad 2: GND -> /Audio Out/AMP_OUTL
- C28 pad 1: VBUS -> /AMP_IN_R
- C28 pad 2: GND -> Net-(C28-Pad2)
- J4 pad R: /Audio Out/R -> /Audio Out/AMP_OUTR
- J4 pad T: /Audio Out/L -> /Audio Out/AMP_OUTL
- J5 pad T: Net-(C25-Pad1) -> Net-(C20-Pad1)
- JP1 pad 1: /A_OUTL -> /PWM_OUT_L
- JP1 pad 10: /GPIO27 -> /AMP_IN_L
- JP1 pad 2: /A_OUTR -> /PWM_OUT_R
- JP1 pad 3: /A_OUTB -> /TDA_L
- JP1 pad 4: /A_TDAL -> /TDA_R
- JP1 pad 5: /A_TDAR -> /MS_CLK_3V
- JP1 pad 6: /A_OUTR -> /MS_DATA_3V
- JP1 pad 7: /A_OUTL -> /GPIO15
- JP1 pad 8: /GPIO28 -> /GPIO14
- JP1 pad 9: /GPIO26 -> /AMP_IN_R
- JP2 pad 1: /MS_CLK_3V -> Net-(JP2-A)
- JP2 pad 2: /GPIO14 -> /GPIO21
- R11 pad 1: Net-(C19-Pad1) -> +3V3
- R11 pad 2: /A_OUTL -> Net-(D2-A)
- R12 pad 1: /Audio Out/L -> +3V3
- R12 pad 2: GND -> /GPIO22
- R13 pad 1: Net-(C19-Pad1) -> Net-(D2-A)
- R13 pad 2: /A_OUTB -> Net-(Q1-B)
- R14 pad 1: Net-(C22-Pad1) -> Net-(C20-Pad2)
- R14 pad 2: /A_OUTB -> Net-(D2-K)
- R15 pad 1: Net-(C22-Pad1) -> Net-(C20-Pad1)
- R15 pad 2: /A_OUTR -> GND
- R16 pad 1: /Audio Out/R -> /GPIO16
- R16 pad 2: GND -> Net-(J6-Pad2)
- R17 pad 1: +3V3 -> VBUS
- R17 pad 2: Net-(D2-A) -> /KB_CLK
- R18 pad 1: +3V3 -> /KB_CLK
- R18 pad 2: /GPIO22 -> /GPIO0
- R19 pad 1: Net-(D2-A) -> /KB_DATA
- R19 pad 2: Net-(Q1-B) -> /GPIO1
- R20 pad 1: Net-(C25-Pad2) -> VBUS
- R20 pad 2: Net-(D2-K) -> /KB_DATA
- R21 pad 1: Net-(C25-Pad1) -> VBUS
- R21 pad 2: GND -> /MS_DATA
- R22 pad 1: /GPIO16 -> VBUS
- R22 pad 2: Net-(J6-Pad2) -> /MS_CLK
- R23 pad 1: VBUS -> /MS_DATA
- R23 pad 2: /KB_CLK -> /MS_DATA_3V
- R24 pad 1: /KB_CLK -> /MS_CLK
- R24 pad 2: /GPIO0 -> /MS_CLK_3V
- R25 pad 1: /KB_DATA -> Net-(J8-CLKN)
- R25 pad 2: /GPIO1 -> /GPIO6
- R26 pad 1: VBUS -> Net-(J8-CLKP)
- R26 pad 2: /KB_DATA -> /GPIO7
- R27 pad 1: VBUS -> Net-(J8-D0N)
- R27 pad 2: /MS_DATA -> /GPIO8
- R28 pad 1: VBUS -> Net-(J8-D0P)
- R28 pad 2: /MS_CLK -> /GPIO9
- R29 pad 1: /MS_DATA -> Net-(J8-D1N)
- R29 pad 2: /MS_DATA_3V -> /GPIO10
- R30 pad 1: /MS_CLK -> Net-(J8-D1P)
- R30 pad 2: /MS_CLK_3V -> /GPIO11
- R31 pad 1: Net-(J8-CLKN) -> Net-(J8-D2N)
- R31 pad 2: /GPIO6 -> /GPIO12
- R32 pad 1: Net-(J8-CLKP) -> Net-(J8-D2P)
- R32 pad 2: /GPIO7 -> /GPIO13
- R33 pad 1: Net-(J8-D0N) -> Net-(R33-Pad1)
- R33 pad 2: /GPIO8 -> GND
- R34 pad 1: Net-(J8-D0P) -> Net-(R34-Pad1)
- R34 pad 2: /GPIO9 -> GND
- R35 pad 1: Net-(J8-D1N) -> /AMP_IN_L
- R35 pad 2: /GPIO10 -> Net-(R33-Pad1)
- R36 pad 1: Net-(J8-D1P) -> /AMP_IN_R
- R36 pad 2: /GPIO11 -> Net-(R34-Pad1)
- R37 pad 1: Net-(J8-D2N) -> Net-(U5A-+)
- R37 pad 2: /GPIO12 -> VBUS
- R38 pad 1: Net-(J8-D2P) -> GND
- R38 pad 2: /GPIO13 -> /Audio Out/AMP_OUTL
- U4 pad 1: /GPIO27 -> /GPIO18
- U4 pad 2: /GPIO28 -> Net-(JP2-A)
- U4 pad 3: /GPIO26 -> unconnected-(U4-SIO2-Pad3)
- U4 pad 5: VBUS -> /GPIO20
- U4 pad 6: /A_TDAL -> /GPIO19
- U4 pad 7: Net-(U4-FLT) -> unconnected-(U4-SIO3-Pad7)
- U4 pad 8: /A_TDAR -> +3V3
- U5 pad 1: /GPIO18 -> Net-(C29-Pad1)
- U5 pad 3: unconnected-(U5-SIO2-Pad3) -> Net-(U5A-+)
- U5 pad 5: /GPIO20 -> Net-(U5A-+)
- U5 pad 6: /GPIO19 -> Net-(U5B--)
- U5 pad 7: unconnected-(U5-SIO3-Pad7) -> Net-(C27-Pad1)
- U5 pad 8: +3V3 -> VBUS
Routing:
- net /RP2040/GPIO25: track 63.1 -> 13.3 mm, vias 2 -> 0
- net /GPIO14: track 100.0 -> 55.5 mm, vias 1 -> 0
- net /A_OUTL: track 42.1 -> 0.00 mm, vias 2 -> 0
- net /A_OUTB: track 41.6 -> 0.00 mm, vias 1 -> 0
- net Net-(J6-Pad2): track 38.8 -> 0.00 mm, vias 2 -> 0
- net VBUS: track 284.0 -> 321.7 mm
- net /Audio Out/L: track 31.2 -> 0.00 mm, vias 2 -> 0
- net Net-(C22-Pad1): track 28.1 -> 0.00 mm
- net /Audio Out/R: track 27.3 -> 0.00 mm, vias 2 -> 0
- net Net-(J1-Pad2): track 26.3 -> 0.00 mm, vias 1 -> 0
- net +3V3: track 123.0 -> 149.0 mm, vias 8 -> 6
- net /GPIO15: track 94.0 -> 68.7 mm, vias 2 -> 0
- net /GPIO22: track 35.7 -> 60.6 mm, vias 2 -> 0
- net /KB_CLK: track 63.8 -> 39.5 mm, vias 1 -> 0
- net /MS_DATA: track 20.8 -> 0.00 mm
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Other:
- board size 76 x 56.5 mm -> 86.2 x 56.5 mm

Commit message: TurboFRANK WIP
Parts:
- added C26: 10u, FRANK:Capacitor (0805), F.Cu at (171.2, 56.8)
- moved C22 22.6 mm to (191.4, 48.2), turned to -90 degrees
- moved J7 4.97 mm to (179.9, 46.6), turned to 180 degrees
- moved D6 2.25 mm to (194.0, 48.2)
- moved D7 0.10 mm to (196.6, 48.2)
- renumbered L1 to LD2
Routing:
- net /TDA_L: track 0.00 -> 52.3 mm, vias 0 -> 2
- net /TDA_R: track 0.00 -> 43.2 mm, vias 0 -> 1
- net /AMP_IN_L: track 0.00 -> 37.9 mm, vias 0 -> 4
- net /PWM_OUT_L: track 0.00 -> 36.3 mm, vias 0 -> 1
- net Net-(C27-Pad1): track 0.00 -> 35.9 mm, vias 0 -> 2
- net /GPIO28: track 59.3 -> 91.7 mm
- net Net-(U5A--): track 0.00 -> 32.4 mm
- net /AMP_IN_R: track 0.00 -> 28.4 mm, vias 0 -> 1
- net /PWM_OUT_R: track 0.00 -> 28.2 mm, vias 0 -> 2
- net /GPIO26: track 63.3 -> 90.9 mm, vias 0 -> 2
- net /GPIO14: track 55.5 -> 83.0 mm
- net /GPIO15: track 68.7 -> 96.0 mm
- net /Audio Out/AMP_OUTR: track 0.00 -> 25.1 mm
- net Net-(U5A-+): track 0.00 -> 23.5 mm, vias 0 -> 2
- net /MS_DATA: track 0.00 -> 23.3 mm, vias 0 -> 1
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Other:
- board text added: "2.04"
- board text added: "AUDIO OUT"
- board text added: "BOOT"
- board text added: "GP1"
- board text added: "MS"
- board text added: "PL"
- board text added: "PR"
- board text added: "RST"
- board text added: "TAPE IN"
- board text added: "TL"
- board text added: "TR"
- board text removed: "2.03"

Commit message: MiniFRANK RM1 WIP
Parts:
- added C43: 4.7u, FRANK:Capacitor (0805), F.Cu at (165.2, 69.8)
- added C44: 10u, FRANK:Capacitor (0805), F.Cu at (166.0, 53.8)
- added C45: 10u, FRANK:Capacitor (0805), F.Cu at (161.8, 53.8)
- added J9: SS-52100-004, FRANK:USB Type A (stacked), F.Cu at (166.1, 47.8)
- added R55: 22R, FRANK:Resistor (0805), F.Cu at (154.8, 61.8)
- added R56: 22R, FRANK:Resistor (0805), F.Cu at (154.8, 59.2)
- added R57: 22R, FRANK:Resistor (0805), F.Cu at (154.8, 56.8)
- added R58: 22R, FRANK:Resistor (0805), F.Cu at (154.8, 54.2)
- added U7: MW7211A, FRANK:SOP-16, F.Cu at (162.5, 61.5)
- moved D2 28.1 mm to (166.5, 73.5)
- moved Q2 24.5 mm to (166.3, 76.8)
- moved C20 19.2 mm to (154.8, 64.2), turned to 180 degrees
- moved R15 18.7 mm to (154.8, 66.8), turned to 180 degrees
- moved R14 17.8 mm to (151.0, 64.8), turned to -90 degrees
- moved J4 13.8 mm to (156.4, 83.5)
- moved J5 13.8 mm to (156.3, 73.5)
- moved R13 11.3 mm to (170.0, 54.5)
- moved R53 11.2 mm to (168.0, 91.2), turned to 180 degrees
- moved R11 8.19 mm to (168.0, 60.2), turned to 90 degrees
- moved C34 7.98 mm to (161.2, 89.8), turned to 180 degrees
- moved H3 6.30 mm to (152.5, 41.0)
- moved H4 6.30 mm to (152.5, 91.5)
- moved C33 6.25 mm to (168.0, 89.0), turned to 180 degrees
- moved U6 5.38 mm to (166.2, 83.0), turned to -90 degrees
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Routing:
- net /D-: track 14.7 -> 96.5 mm, vias 0 -> 2
- net /D+: track 16.7 -> 87.8 mm, vias 0 -> 2
- net VBUS: track 333.1 -> 287.5 mm
- net /TDA_L: track 52.3 -> 11.6 mm, vias 2 -> 0
- net /TDA_R: track 43.2 -> 7.28 mm, vias 1 -> 0
- net Net-(D2-A): track 22.1 -> 0.00 mm
- net /GPIO26: track 90.9 -> 70.4 mm, vias 2 -> 1
- net /GPIO28: track 91.7 -> 73.3 mm
- net Net-(C20-Pad2): track 14.3 -> 0.00 mm
- net +3V3: track 156.9 -> 143.2 mm
- net /GPIO27: track 77.3 -> 65.0 mm
- net Net-(D2-K): track 9.83 -> 0.00 mm
- net /Audio Out/AMP_OUTR: track 25.1 -> 16.9 mm
- net Net-(C20-Pad1): track 6.98 -> 0.00 mm
- net Net-(U6-FLT): track 4.03 -> 0.00 mm
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Other:
- board size 86.2 x 56.5 mm -> 92.5 x 56.5 mm

Commit message: MiniFRANK 2.05 Release
Parts:
- J4: value ~ -> PJ-320D
- J5: value FRANK:Jack (3.5mm, PJ-320D) -> PJ-320D
- JP1: value SW_DIP_x06 -> Main Jumpers
- LD1: value BLUE -> Blue
- moved R13 0.56 mm to (170.5, 54.8)
- moved C26 0.25 mm to (171.2, 57.0)
- renumbered USB1 to J10
Routing:
- net /TDA_R: track 7.28 -> 64.4 mm, vias 0 -> 1
- net /TDA_L: track 11.6 -> 55.8 mm, vias 0 -> 1
- net Net-(D2-A): track 0.00 -> 25.7 mm, vias 0 -> 2
- net /Audio Out/AMP_OUTR: track 16.9 -> 39.6 mm, vias 0 -> 2
- net Net-(J9-D1-): track 0.00 -> 21.6 mm
- net Net-(D2-K): track 0.00 -> 20.6 mm
- net /Audio Out/AMP_OUTL: track 12.6 -> 30.8 mm, vias 0 -> 2
- net Net-(J9-D1+): track 0.00 -> 17.0 mm, vias 0 -> 1
- net +3V3: track 143.2 -> 159.7 mm
- net Net-(J9-D2+): track 0.00 -> 16.4 mm
- net VBUS: track 287.5 -> 301.3 mm
- net Net-(J9-D2-): track 0.00 -> 11.4 mm
- net /GPIO28: track 73.3 -> 83.8 mm, vias 0 -> 2
- net /USB_D2-: track 0.00 -> 10.3 mm
- net /GPIO26: track 70.4 -> 79.9 mm, vias 1 -> 2
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Other:
- board text added: "2.05"
- board text removed: "2.04"
