File: hardware/minifrank_rm1/gamepad.kicad_sch (KiCad schematic)
At the start: 3 parts

Commit message: Minor updates
Parts:
- D1: renamed from D3; AliExpress https://www.aliexpress.com/item/32997486634.html -> https://www.aliexpress.com/item/1005006143480992.html
- J1: renamed from GP1; value Gamepad -> D-SUB 9 Male; footprint FRANK:D-SUB (9 pin, male) -> FRANK:D-SUB (9 pin, male, top mount); AliExpress https://www.aliexpress.com/item/4000659356343.html -> https://www.aliexpress.com/item/4001214300548.html
- renumbered R13 to R1
Other:
- note removed: "The gamepad uses standard DB9 male socket."
Changed lines of the file:
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@@
 	(title_block
 		(title "MiniFRANK RM1")
-		(date "2025-03-16")
-		(rev "2.02")
+		(date "2025-04-01")
+		(rev "2.03")
 		(company "Mikhail Matveev")
 		(comment 1 "https://github.com/xtremespb/frank")
-	)
-	(text "The gamepad uses standard DB9 male socket."
-		(exclude_from_sim no)
-		(at 49.53 31.75 0)
-		(effects
-			(font
-				(size 1.27 1.27)
-			)
-			(justify left)
-		)
 	)
 	(junction
@@
 		(on_board yes)
 		(dnp no)
-		(property "Reference" "#PWR040"
+		(property "Reference" "#PWR04"
 			(at 78.74 83.82 0)
 			(effects
@@
 		(instances
 			(project ""
-				(path "/8c0b3d8b-46d3-4173-ab1e-a61765f77d61/91039a09-82d7-4099-8414-fc5647ada98f"
-					(reference "#PWR040")
-					(unit 1)
-				)
-				(path "/8c0b3d8b-46d3-4173-ab1e-a61765f77d61/e9da9b3c-e9c6-4677-bc99-391052f7625b"
-					(reference "#PWR043")
+				(path "/8c0b3d8b-46d3-4173-ab1e-a61765f77d61/2783d91d-5335-4a4c-9a71-d18d6dc2e592"
+					(reference "#PWR053")
+					(unit 1)
+				)
+				(path "/8c0b3d8b-46d3-4173-ab1e-a61765f77d61/d4862ecd-2ed8-4240-ac0c-247fd7d9c41c"
+					(reference "#PWR04")
 					(unit 1)
 				)
@@
 		(on_board yes)
 		(dnp no)
-		(property "Reference" "D3"
+		(property "Reference" "D1"
 			(at 76.2 73.66 0)
 			(effects
@@
 			)
 		)
-		(property "AliExpress" "https://www.aliexpress.com/item/32997486634.html"
+		(property "AliExpress" "https://www.aliexpress.com/item/1005006143480992.html"
 			(at 78.74 73.66 0)
 			(effects
@@
 		(instances
 			(project ""
-				(path "/8c0b3d8b-46d3-4173-ab1e-a61765f77d61/91039a09-82d7-4099-8414-fc5647ada98f"
+				(path "/8c0b3d8b-46d3-4173-ab1e-a61765f77d61/2783d91d-5335-4a4c-9a71-d18d6dc2e592"
 					(reference "D3")
 					(unit 1)
 				)
-				(path "/8c0b3d8b-46d3-4173-ab1e-a61765f77d61/e9da9b3c-e9c6-4677-bc99-391052f7625b"
-					(reference "D4")
+				(path "/8c0b3d8b-46d3-4173-ab1e-a61765f77d61/d4862ecd-2ed8-4240-ac0c-247fd7d9c41c"
+					(reference "D1")
 					(unit 1)
 				)
@@
 		(dnp no)
 		(fields_autoplaced yes)
-		(property "Reference" "#PWR039"
+		(property "Reference" "#PWR03"
 			(at 91.44 67.31 0)
 			(effects
@@
 		(instances
 			(project ""
-				(path "/8c0b3d8b-46d3-4173-ab1e-a61765f77d61/91039a09-82d7-4099-8414-fc5647ada98f"
-					(reference "#PWR039")
-					(unit 1)
-				)
-				(path "/8c0b3d8b-46d3-4173-ab1e-a61765f77d61/e9da9b3c-e9c6-4677-bc99-391052f7625b"
-					(reference "#PWR042")
+				(path "/8c0b3d8b-46d3-4173-ab1e-a61765f77d61/2783d91d-5335-4a4c-9a71-d18d6dc2e592"
+					(reference "#PWR052")
+					(unit 1)
+				)
+				(path "/8c0b3d8b-46d3-4173-ab1e-a61765f77d61/d4862ecd-2ed8-4240-ac0c-247fd7d9c41c"
+					(reference "#PWR03")
 					(unit 1)
 				)
@@
 		(on_board yes)
 		(dnp no)
-		(property "Reference" "GP1"
+		(property "Reference" "J1"
 			(at 109.22 50.8 0)
 			(effects
@@
 			)
 		)
-		(property "Value" "Gamepad"
+		(property "Value" "D-SUB 9 Male"
 			(at 105.41 48.26 0)
 			(effects
@@
 			)
 		)
-		(property "Footprint" "FRANK:D-SUB (9 pin, male)"
+		(property "Footprint" "FRANK:D-SUB (9 pin, male, top mount)"
 			(at 107.95 63.5 0)
 			(effects
@@
 			)
 		)
-		(property "AliExpress" "https://www.aliexpress.com/item/4000659356343.html"
+		(property "AliExpress" "https://www.aliexpress.com/item/4001214300548.html"
 			(at 107.95 63.5 0)
 			(effects
@@
 		(instances
 			(project ""
-				(path "/8c0b3d8b-46d3-4173-ab1e-a61765f77d61/91039a09-82d7-4099-8414-fc5647ada98f"
-					(reference "GP1")
-					(unit 1)
-				)
-				(path "/8c0b3d8b-46d3-4173-ab1e-a61765f77d61/e9da9b3c-e9c6-4677-bc99-391052f7625b"
-					(reference "GP2")
+				(path "/8c0b3d8b-46d3-4173-ab1e-a61765f77d61/2783d91d-5335-4a4c-9a71-d18d6dc2e592"
+					(reference "J6")
+					(unit 1)
+				)
+				(path "/8c0b3d8b-46d3-4173-ab1e-a61765f77d61/d4862ecd-2ed8-4240-ac0c-247fd7d9c41c"
+					(reference "J1")
 					(unit 1)
 				)
@@
 		(dnp no)
 		(fields_autoplaced yes)
-		(property "Reference" "#PWR038"
+		(property "Reference" "#PWR02"
 			(at 86.36 60.96 0)
 			(effects
@@
 		(instances
 			(project ""
-				(path "/8c0b3d8b-46d3-4173-ab1e-a61765f77d61/91039a09-82d7-4099-8414-fc5647ada98f"
-					(reference "#PWR038")
-					(unit 1)
-				)
-				(path "/8c0b3d8b-46d3-4173-ab1e-a61765f77d61/e9da9b3c-e9c6-4677-bc99-391052f7625b"
-					(reference "#PWR041")
+				(path "/8c0b3d8b-46d3-4173-ab1e-a61765f77d61/2783d91d-5335-4a4c-9a71-d18d6dc2e592"
+					(reference "#PWR051")
+					(unit 1)
+				)
+				(path "/8c0b3d8b-46d3-4173-ab1e-a61765f77d61/d4862ecd-2ed8-4240-ac0c-247fd7d9c41c"
+					(reference "#PWR02")
 					(unit 1)
 				)
@@
 		(on_board yes)
 		(dnp no)
-		(property "Reference" "R13"
+		(property "Reference" "R1"
 			(at 81.28 66.04 90)
 			(effects
@@
 		(instances
 			(project ""
-				(path "/8c0b3d8b-46d3-4173-ab1e-a61765f77d61/91039a09-82d7-4099-8414-fc5647ada98f"
-					(reference "R13")
-					(unit 1)
-				)
-				(path "/8c0b3d8b-46d3-4173-ab1e-a61765f77d61/e9da9b3c-e9c6-4677-bc99-391052f7625b"
-					(reference "R14")
-					(unit 1)
-				)
+				(path "/8c0b3d8b-46d3-4173-ab1e-a61765f77d61/2783d91d-5335-4a4c-9a71-d18d6dc2e592"
+					(reference "R22")
+					(unit 1)
+				)
+				(path "/8c0b3d8b-46d3-4173-ab1e-a61765f77d61/d4862ecd-2ed8-4240-ac0c-247fd7d9c41c"
+					(reference "R1")
+					(unit 1)
+				)

Commit message: MiniFRANK 2.05 Release
Parts:
- D1: LCSC (none) -> C19334
- R1: LCSC (none) -> C17513
Changed lines of the file:
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@@
 	(title_block
 		(title "MiniFRANK RM1")
-		(date "2025-04-04")
-		(rev "2.04")
+		(date "2025-04-07")
+		(rev "${VERSION}")
 		(company "Mikhail Matveev")
 		(comment 1 "https://github.com/xtremespb/frank")
@@
 				)
 				(hide yes)
+			)
+		)
+		(property "LCSC" "C19334"
+			(at 78.74 73.66 0)
+			(effects
+				(font
+					(size 1.27 1.27)
+				)
 			)
 		)
@@
 			)
 		)
+		(property "LCSC" "C17513"
+			(at 83.82 68.58 0)
+			(effects
+				(font
+					(size 1.27 1.27)
+				)
+			)
+		)

Commit message: Bugfixes
Other:
- title: MiniFRANK RM1 -> ${NAME}
Changed lines of the file:
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@@
 	(paper "A4")
 	(title_block
-		(title "MiniFRANK RM1")
-		(date "2025-04-09")
+		(title "${NAME}")
+		(date "2025-04-24")
 		(rev "${VERSION}")
 		(company "Mikhail Matveev")
