File: hardware/minifrank_rm1/ps2.kicad_sch (KiCad schematic)
At the start: 8 parts

Commit message: Minor updates
Parts:
- added D6, D7: 3V3, FRANK:Diode (SOD-323), symbol Device:D_Zener
- added R27, R28: 1K, FRANK:Resistor (0805), symbol Device:R
- added R29, R30: 100R, FRANK:Resistor (0805), symbol Device:R
- D4: renamed from D1; AliExpress https://www.aliexpress.com/item/32997486634.html -> https://www.aliexpress.com/item/1005006143480992.html
- D5: renamed from D2; AliExpress https://www.aliexpress.com/item/32997486634.html -> https://www.aliexpress.com/item/1005006143480992.html
- J7: renamed from KB1; value PS/2 Keyboard -> MDC-036
- renumbered C18 to C27, R9 to R23, R10 to R24, R11 to R25, R12 to R26
Connections:
- net GND: now also D6.2 (A), D7.2 (A)
- net VBUS: now also R27.1, R28.1
- net KB_DATA: now reaches J7.1, R25.1, R26.2
- net KB_CLK: now reaches J7.5, R23.2, R24.1
- net MS_DATA: now reaches J7.2
- net MS_DATA: now also R27.2, R29.1
- net MS_CLK: now reaches J7.6
- net MS_CLK: now also R28.2, R30.1
- net CLK renamed KB_CLK_3V
- net DATA renamed KB_DATA_3V
- new net MS_CLK_3V: D7.1 (K), R30.2
- new net MS_DATA_3V: D6.1 (K), R29.2
- no-connect marks 2 -> 0
Other:
- note removed: "PS/2 Keyboard is used here. You can connect USB>PS/2 Adapter in order to use USB keyboards."
- moved on the sheet: C27, D4, D5, J7, R23, R24, R25, R26

Commit message: WIP
Parts:
- renumbered C27 to C22, R23 to R17, R24 to R18, R25 to R19, R26 to R20, R27 to R21, R28 to R22, R29 to R23, R30 to R24
Changed lines of the file:
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@@
 		(dnp no)
 		(fields_autoplaced yes)
-		(property "Reference" "#PWR060"
+		(property "Reference" "#PWR055"
 			(at 107.95 59.69 0)
 			(effects
@@
 			(project "turbofrank"
 				(path "/8c0b3d8b-46d3-4173-ab1e-a61765f77d61/362dd4de-9685-486a-ada7-07852c7bfc7d"
-					(reference "#PWR060")
+					(reference "#PWR055")
 					(unit 1)
 				)
@@
 		(on_board yes)
 		(dnp no)
-		(property "Reference" "#PWR061"
+		(property "Reference" "#PWR056"
 			(at 31.75 81.28 0)
 			(effects
@@
 			(project "turbofrank"
 				(path "/8c0b3d8b-46d3-4173-ab1e-a61765f77d61/362dd4de-9685-486a-ada7-07852c7bfc7d"
-					(reference "#PWR061")
+					(reference "#PWR056")
 					(unit 1)
 				)
@@
 		(on_board yes)
 		(dnp no)
-		(property "Reference" "R27"
+		(property "Reference" "R21"
 			(at 52.07 100.33 90)
 			(effects
@@
 			(project "turbofrank"
 				(path "/8c0b3d8b-46d3-4173-ab1e-a61765f77d61/362dd4de-9685-486a-ada7-07852c7bfc7d"
-					(reference "R27")
+					(reference "R21")
 					(unit 1)
 				)
@@
 		(dnp no)
 		(fields_autoplaced yes)
-		(property "Reference" "#PWR063"
+		(property "Reference" "#PWR058"
 			(at 69.85 148.59 0)
 			(effects
@@
 			(project "turbofrank"
 				(path "/8c0b3d8b-46d3-4173-ab1e-a61765f77d61/362dd4de-9685-486a-ada7-07852c7bfc7d"
-					(reference "#PWR063")
+					(reference "#PWR058")
 					(unit 1)
 				)
@@
 		(on_board yes)
 		(dnp no)
-		(property "Reference" "R25"
+		(property "Reference" "R19"
 			(at 77.47 50.8 90)
 			(effects
@@
 			(project "turbofrank"
 				(path "/8c0b3d8b-46d3-4173-ab1e-a61765f77d61/362dd4de-9685-486a-ada7-07852c7bfc7d"
-					(reference "R25")
+					(reference "R19")
 					(unit 1)
 				)
@@
 		(on_board yes)
 		(dnp no)
-		(property "Reference" "R28"
+		(property "Reference" "R22"
 			(at 72.39 100.33 90)
 			(effects
@@
 			(project "turbofrank"
 				(path "/8c0b3d8b-46d3-4173-ab1e-a61765f77d61/362dd4de-9685-486a-ada7-07852c7bfc7d"
-					(reference "R28")
+					(reference "R22")
 					(unit 1)
 				)
@@
 		(on_board yes)
 		(dnp no)
-		(property "Reference" "R24"
+		(property "Reference" "R18"
 			(at 77.47 45.72 90)
 			(effects
@@
 			(project "turbofrank"
 				(path "/8c0b3d8b-46d3-4173-ab1e-a61765f77d61/362dd4de-9685-486a-ada7-07852c7bfc7d"
-					(reference "R24")
+					(reference "R18")
 					(unit 1)
 				)
@@
 		(on_board yes)
 		(dnp no)
-		(property "Reference" "R29"
+		(property "Reference" "R23"
 			(at 58.42 114.3 90)
 			(effects
@@
 			(project "turbofrank"
 				(path "/8c0b3d8b-46d3-4173-ab1e-a61765f77d61/362dd4de-9685-486a-ada7-07852c7bfc7d"
-					(reference "R29")
+					(reference "R23")
 					(unit 1)
 				)
@@
 		(dnp no)
 		(fields_autoplaced yes)
-		(property "Reference" "#PWR057"
+		(property "Reference" "#PWR052"
 			(at 111.76 39.37 0)
 			(effects
@@
 			(project "turbofrank"
 				(path "/8c0b3d8b-46d3-4173-ab1e-a61765f77d61/362dd4de-9685-486a-ada7-07852c7bfc7d"
-					(reference "#PWR057")
+					(reference "#PWR052")
 					(unit 1)
 				)
@@
 		(dnp no)
 		(fields_autoplaced yes)
-		(property "Reference" "#PWR058"
+		(property "Reference" "#PWR053"
 			(at 27.94 53.34 0)
 			(effects
@@
 			(project "turbofrank"
 				(path "/8c0b3d8b-46d3-4173-ab1e-a61765f77d61/362dd4de-9685-486a-ada7-07852c7bfc7d"
-					(reference "#PWR058")
+					(reference "#PWR053")
 					(unit 1)
 				)
@@
 		(on_board yes)
 		(dnp no)
-		(property "Reference" "R26"
+		(property "Reference" "R20"
 			(at 63.5 57.15 90)
 			(effects
@@
 			(project "turbofrank"
 				(path "/8c0b3d8b-46d3-4173-ab1e-a61765f77d61/362dd4de-9685-486a-ada7-07852c7bfc7d"
-					(reference "R26")
+					(reference "R20")
 					(unit 1)
 				)
@@
 		(on_board yes)
 		(dnp no)
-		(property "Reference" "R23"
+		(property "Reference" "R17"
 			(at 63.5 36.83 90)
 			(effects
@@
 			(project "turbofrank"
 				(path "/8c0b3d8b-46d3-4173-ab1e-a61765f77d61/362dd4de-9685-486a-ada7-07852c7bfc7d"
-					(reference "R23")
+					(reference "R17")
 					(unit 1)
 				)
@@
 		(on_board yes)
 		(dnp no)
-		(property "Reference" "#PWR059"
+		(property "Reference" "#PWR054"
 			(at 59.69 49.53 0)
 			(effects
@@
 			(project "turbofrank"
 				(path "/8c0b3d8b-46d3-4173-ab1e-a61765f77d61/362dd4de-9685-486a-ada7-07852c7bfc7d"
-					(reference "#PWR059")
+					(reference "#PWR054")
 					(unit 1)
 				)
@@
 		(dnp no)
 		(fields_autoplaced yes)
-		(property "Reference" "#PWR062"
+		(property "Reference" "#PWR057"
 			(at 49.53 144.78 0)
 			(effects
@@
 			(project "turbofrank"
 				(path "/8c0b3d8b-46d3-4173-ab1e-a61765f77d61/362dd4de-9685-486a-ada7-07852c7bfc7d"
-					(reference "#PWR062")
+					(reference "#PWR057")
 					(unit 1)
 				)
@@
 		(on_board yes)
 		(dnp no)
-		(property "Reference" "R30"
+		(property "Reference" "R24"
 			(at 63.5 114.3 90)
 			(effects
@@
 			(project "turbofrank"
 				(path "/8c0b3d8b-46d3-4173-ab1e-a61765f77d61/362dd4de-9685-486a-ada7-07852c7bfc7d"
-					(reference "R30")
+					(reference "R24")
 					(unit 1)
 				)
@@
 		(on_board yes)
 		(dnp no)
-		(property "Reference" "C27"
+		(property "Reference" "C22"
 			(at 34.671 66.1416 0)
 			(effects
@@
 			(project "turbofrank"
 				(path "/8c0b3d8b-46d3-4173-ab1e-a61765f77d61/362dd4de-9685-486a-ada7-07852c7bfc7d"
-					(reference "C27")
-					(unit 1)
-				)
+					(reference "C22")
+					(unit 1)
+				)

Commit message: MiniFRANK 2.05 Release
Parts:
- C22: LCSC (none) -> C1711
- D4, D5, D6, D7: LCSC (none) -> C19334
- R17, R20, R21, R22: LCSC (none) -> C17513
- R18, R19, R23, R24: LCSC (none) -> C3152174
Changed lines of the file:
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@@
 	(title_block
 		(title "MiniFRANK RM1")
-		(date "2025-04-04")
-		(rev "2.04")
+		(date "2025-04-07")
+		(rev "${VERSION}")
 		(company "Mikhail Matveev")
 		(comment 1 "https://github.com/xtremespb/frank")
@@
 			)
 		)
+		(property "LCSC" "C19334"
+			(at 97.79 59.69 0)
+			(effects
+				(font
+					(size 1.27 1.27)
+				)
+			)
+		)
 		(pin "1"
 		)
@@
 				)
 				(hide yes)
+			)
+		)
+		(property "LCSC" "C17513"
+			(at 49.53 100.33 0)
+			(effects
+				(font
+					(size 1.27 1.27)
+				)
 			)
 		)
@@
 			)
 		)
+		(property "LCSC" "C3152174"
+			(at 83.82 52.07 0)
+			(effects
+				(font
+					(size 1.27 1.27)
+				)
+			)
+		)
 		(pin "1"
 		)
@@
 			)
 		)
+		(property "LCSC" "C17513"
+			(at 69.85 100.33 0)
+			(effects
+				(font
+					(size 1.27 1.27)
+				)
+			)
+		)
 		(pin "1"
 		)
@@
 			)
 		)
+		(property "LCSC" "C3152174"
+			(at 83.82 46.99 0)
+			(effects
+				(font
+					(size 1.27 1.27)
+				)
+			)
+		)
 		(pin "1"
 		)
@@
 				)
 				(hide yes)
+			)
+		)
+		(property "LCSC" "C3152174"
+			(at 57.15 120.65 0)
+			(effects
+				(font
+					(size 1.27 1.27)
+				)
 			)
 		)
@@
 			)
 		)
+		(property "LCSC" "C19334"
+			(at 49.53 134.62 0)
+			(effects
+				(font
+					(size 1.27 1.27)
+				)
+			)
+		)
 		(pin "1"
 		)
@@
 			)
 		)
+		(property "LCSC" "C17513"
+			(at 63.5 59.69 0)
+			(effects
+				(font
+					(size 1.27 1.27)
+				)
+			)
+		)
 		(pin "1"
 		)
@@
 				)
 				(hide yes)
+			)
+		)
+		(property "LCSC" "C17513"
+			(at 63.5 39.37 0)
+			(effects
+				(font
+					(size 1.27 1.27)
+				)
 			)
 		)
@@
 			)
 		)
+		(property "LCSC" "C19334"
+			(at 97.79 39.37 0)
+			(effects
+				(font
+					(size 1.27 1.27)
+				)
+			)
+		)
 		(pin "1"
 		)
@@
 			)
 		)
+		(property "LCSC" "C3152174"
+			(at 62.23 120.65 0)
+			(effects
+				(font
+					(size 1.27 1.27)
+				)
+			)
+		)
 		(pin "1"
 		)
@@
 			)
 		)
+		(property "LCSC" "C19334"
+			(at 69.85 134.62 0)
+			(effects
+				(font
+					(size 1.27 1.27)
+				)
+			)
+		)
 		(pin "1"
 		)
@@
 			)
 		)
+		(property "LCSC" "C1711"
+			(at 31.75 67.31 0)
+			(effects
+				(font
+					(size 1.27 1.27)
+				)
+			)
+		)

Commit message: Bugfixes
Other:
- title: MiniFRANK RM1 -> ${NAME}
Changed lines of the file:
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@@
 	(paper "A4")
 	(title_block
-		(title "MiniFRANK RM1")
-		(date "2025-04-09")
+		(title "${NAME}")
+		(date "2025-04-24")
 		(rev "${VERSION}")
 		(company "Mikhail Matveev")
