File: hardware/minifrank_rm1/usb_hub.kicad_sch (KiCad schematic)
At the start: 3 parts, among them J22 USB HUB Data, U3 MW7211A

Commit message: MiniFRANK RM1 WIP
Parts:
- removed J22: USB HUB Data, FRANK:Connector Female ZH 1.50mm (2 pins + tracks), symbol Connector:Conn_01x02_Pin
- renumbered U3 to U7
Other:
- moved on the sheet: C43, U7

Commit message: MiniFRANK 2.05 Release
Parts:
- C43: LCSC (none) -> C1746
- U7: AliExpress (none) -> https://www.aliexpress.com/item/1005007446137541.html
Other:
- title: TurboFRANK -> MiniFRANK RM1
Changed lines of the file:
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@@
 	(paper "A4")
 	(title_block
-		(title "TurboFRANK")
-		(date "2025-03-19")
-		(rev "1.04")
+		(title "MiniFRANK RM1")
+		(date "2025-04-07")
+		(rev "${VERSION}")
 		(company "Mikhail Matveev")
 		(comment 1 "https://github.com/xtremespb/frank")
@@
 			)
 		)
-		(property "Datasheet" "~"
+		(property "Datasheet" "https://eu.mouser.com/datasheet/2/40/KGM_X7R-3223212.pdf"
 			(at 176.53 99.06 0)
 			(effects
@@
 				)
 				(hide yes)
+			)
+		)
+		(property "LCSC" "C1746"
+			(at 176.53 99.06 0)
+			(effects
+				(font
+					(size 1.27 1.27)
+				)
 			)
 		)
@@
 			)
 		)
-		(property "Datasheet" "DOCUMENTATION"
+		(property "Datasheet" "https://content.instructables.com/FTQ/K2JY/KW6E9NZ8/FTQK2JYKW6E9NZ8.pdf"
 			(at 134.62 86.36 0)
 			(effects
@@
 			)
 		)
+		(property "AliExpress" "https://www.aliexpress.com/item/1005007446137541.html"
+			(at 134.62 86.36 0)
+			(effects
+				(font
+					(size 1.27 1.27)
+				)
+				(hide yes)
+			)
+		)

Commit message: Bugfixes
Parts:
- renumbered C43 to C37
Other:
- title: MiniFRANK RM1 -> ${NAME}
Changed lines of the file:
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@@
 	(paper "A4")
 	(title_block
-		(title "MiniFRANK RM1")
-		(date "2025-04-09")
+		(title "${NAME}")
+		(date "2025-04-24")
 		(rev "${VERSION}")
 		(company "Mikhail Matveev")
@@
 		(on_board yes)
 		(dnp no)
-		(property "Reference" "C43"
+		(property "Reference" "C37"
 			(at 179.578 99.314 90)
 			(effects
@@
 					(size 1.27 1.27)
 				)
+				(hide yes)
 			)
 		)
@@
 			(project "turbofrank"
 				(path "/8c0b3d8b-46d3-4173-ab1e-a61765f77d61/38dacd66-5330-4209-a1a1-c2b704ef5733"
-					(reference "C43")
+					(reference "C37")
 					(unit 1)
 				)
