File: hardware/minifrank_rm1/audio_multiplexer.kicad_sch (KiCad schematic)
At the start: 3 parts, among them U8 74HC4052D

Commit message: MiniFRANK RM1 2.07
Parts:
- U8: symbol 74HC4052D_653:74HC4052D,653 -> FRANK:74HC4052D
Changed lines of the file:
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@@
 	)
 	(symbol
-		(lib_id "74HC4052D_653:74HC4052D,653")
+		(lib_id "FRANK:74HC4052D")
 		(at 142.24 91.44 0)
 		(unit 1)
