File: lab/protea/protea.kicad_pcb (KiCad board)
At the start: 2 copper layers, 80.1 x 44 mm, 73 parts, among them J1 USB4215-03-A, J2 D-SUB 9 Male, J3 676430910, J4 HDMI Female, J5 ESP8266 Prog, U1 NCP1117 3.3, U2 W25Q128JVSIQ, U3 RP2040, U4 MAX232CSE+, U5 ESP8266-12E_ESP-12E, Y1 12 MHz

Commit message: Fixes
Parts:
- removed JP1: HDMI Jumper, FRANK:Jumper (solder)
- removed S2: Defaults, FRANK:Button (SMD, 3x3mm, 1-1)
- added J6: SD04H0SB, FRANK:DIP Switch (5x5), F.Cu at (113.6, 54.0)
- R1, R3: moved to F.Cu
- moved R11 68.6 mm to (127.2, 59.8)
- moved D2 68.4 mm to (132.0, 59.8), turned to 180 degrees
- moved R22 63.9 mm to (120.2, 43.5), turned to 180 degrees
- moved R23 61.4 mm to (120.2, 41.0), turned to 180 degrees
- moved D1 59.8 mm to (124.2, 47.0)
- moved R24 42.0 mm to (93.5, 48.3)
- moved S5 41.9 mm to (85.8, 23.8)
- moved R21 39.0 mm to (93.2, 35.5)
- moved R20 38.3 mm to (93.2, 31.5)
- moved S3 36.1 mm to (130.2, 63.0)
- moved C24 32.3 mm to (93.5, 44.8), turned to 180 degrees
- moved C21 29.4 mm to (94.8, 64.5), turned to 180 degrees
- moved J3 25.2 mm to (159.9, 32.4)
- moved C22 24.6 mm to (143.0, 25.8), turned to -90 degrees
- moved C23 23.8 mm to (146.2, 25.8), turned to 90 degrees
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Connections:
- net /ESP8266/ADC renamed /ESP_ADC
- net /ESP8266/CSO renamed /ESP_CSO
- net /ESP8266/GPIO10 renamed /ESP_GPIO10
- net /ESP8266/GPIO12 renamed /ESP_GPIO12
- net /ESP8266/GPIO13 renamed /ESP_GPIO13
- net /ESP8266/GPIO14 renamed /ESP_GPIO14
- net /ESP8266/GPIO16 renamed /ESP_GPIO16
- net /ESP8266/GPIO4 renamed /ESP_GPIO4
- net /ESP8266/GPIO5 renamed /ESP_GPIO5
- net /ESP8266/GPIO9 renamed /ESP_GPIO9
- net /ESP8266/MISO renamed /ESP_MISO
- net /ESP8266/MOSI renamed /ESP_MOSI
- net /ESP8266/RXD renamed /ESP_RXD
- net /ESP8266/SCLK renamed /ESP_SCLK
- net /ESP8266/TXD renamed /ESP_TXD
- C18 pad 2: VBUS -> /RS232_VBUS
- U4 pad 16: VBUS -> /RS232_VBUS
Routing:
- net +3V3: track 0.00 -> 180.4 mm, vias 6 -> 9
- net VBUS: track 0.00 -> 130.7 mm, vias 0 -> 1
- net /GPIO17: track 6.67 -> 37.9 mm, vias 0 -> 2
- net /GPIO16: track 7.63 -> 35.5 mm
- net Net-(J1-SHIELD): track 0.00 -> 21.3 mm
- net /D-: track 0.00 -> 21.2 mm, vias 0 -> 1
- net /GPIO18: track 22.0 -> 43.1 mm, vias 0 -> 2
- net /GPIO15: track 4.30 -> 24.2 mm
- net /RP2040/QSPI_SD3: track 8.51 -> 26.8 mm, vias 0 -> 2
- net /D+: track 0.00 -> 18.0 mm, vias 0 -> 1
- net /RP2040/QSPI_SCLK: track 8.33 -> 26.0 mm, vias 0 -> 2
- net /GPIO19: track 33.8 -> 51.1 mm
- net /RP2040/QSPI_SD0: track 8.37 -> 22.6 mm, vias 0 -> 2
- net /GPIO14: track 17.1 -> 30.4 mm
- net Net-(J4-CLKN): track 0.00 -> 12.2 mm
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Other:
- board size 80.1 x 44 mm -> 92 x 44 mm

Commit message: WIP
Parts:
- moved R10 2.25 mm to (127.8, 49.2)
- moved R1 0.75 mm to (159.0, 55.0)
- moved R3 0.28 mm to (159.0, 46.5)
- moved C2 0.25 mm to (163.2, 60.2)
Routing:
- net Net-(U5-IO0): track 0.00 -> 56.1 mm, vias 0 -> 2
- net Net-(R6-Pad2): track 4.21 -> 45.9 mm, vias 0 -> 2
- net /ESP_TXD: track 0.00 -> 40.8 mm, vias 0 -> 1
- net /RS232/CTS_IN: track 0.00 -> 39.2 mm, vias 0 -> 1
- net /RS232/RTS_IN: track 0.00 -> 36.9 mm, vias 0 -> 1
- net /RS232/TX_IN: track 0.00 -> 35.7 mm, vias 0 -> 1
- net /RS232/CTS_MAX: track 0.00 -> 33.9 mm, vias 0 -> 2
- net /ESP_RXD: track 0.00 -> 32.8 mm
- net /RS232/RX_IN: track 0.00 -> 31.0 mm
- net /RS232/RX_MAX: track 0.00 -> 30.4 mm
- net Net-(U5-RESET): track 0.00 -> 30.2 mm, vias 0 -> 2
- net /RS232_VBUS: track 0.00 -> 25.3 mm, vias 0 -> 1
- net /GPIO18: track 43.1 -> 63.0 mm
- net /RP2040/QSPI_SS: track 11.1 -> 30.0 mm
- net /GPIO16: track 35.5 -> 54.1 mm
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Other:
- board text added: "+5V"
- board text added: "2.04"
- board text added: "BOOT"
- board text added: "DEF"
- board text added: "HDMI"
- board text added: "Protea"
- board text added: "RDX"
- board text added: "RST"
- board text added: "TDX"
- board text added: "rh1.tech"
