File: hardware/frank_m1/CMZJ2.kicad_sch (KiCad schematic)
At the start: 7 parts, among them CON1 Pin Header 1x03, CON2 Pin Header 1x03, J1 Pin Header 2x18

Commit message: FRANK M1 1.16 WIP
Parts:
- removed J1: Pin Header 2x18, FRANK:Pin Header (2x16), symbol Connector_Generic:Conn_02x16_Odd_Even
- added JP1: SW_DIP_x06, DIP Switch (6), symbol Switch:SW_DIP_x06
- added JP2: SW_DIP_x10, DIP Switch (10), symbol Switch:SW_DIP_x10
- added S1: TS-1233, FRANK:Button (SMD, 3x3mm, 1-1), symbol Switch:SW_Push
- renumbered CON1 to J1, CON2 to J2
Connections:
- net A_OUTB: now also JP1.3
- net A_OUTL: now also JP1.1, JP1.9
- net A_OUTR: now also JP1.2, JP1.8
- net A_TDAL: now also JP1.4
- net A_TDAR: now also JP1.5
- net GND: now also S1.2
- net GP1_DATA: now also JP2.3
- net GP2_DATA: now also JP2.4
- net GPIO14: now also JP2.19
- net GPIO15: now also JP2.20
- net GPIO16: now also JP2.14, JP2.18
- net GPIO17: now also JP2.13, JP2.17
- net GPIO18: now also JP2.12
- net GPIO19: now also JP2.11
- net GPIO21: now also JP2.16
- net GPIO22: now also JP1.7
- net GPIO26: now also JP1.11
- net GPIO27: now also JP1.12
- net GPIO28: now also JP1.10
- net LOAD_IN_D: now also JP1.6
- net MS_CLK_3V: now also JP2.2
- net MS_DATA_3V: now also JP2.1
- net PSR_SOSIO: now also JP2.5
- net RS232_CTS: now also JP2.9
- net RS232_RTS: now also JP2.10
- net RS232_RX: now also JP2.8
- net RS232_TX: now also JP2.7
- net RUN: now also S1.1
- net VBUS: now also JP2.15
- net ZERO_VBUS: now also JP2.6
Other:
- removed sheet Reset
- moved on the sheet: J1, J2

Commit message: FRANK M1 1.16
Parts:
- JP1: footprint DIP Switch (6) -> FRANK:DIP Switch (6)
- JP2: footprint DIP Switch (10) -> FRANK:DIP Switch (10)
Changed lines of the file:
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@@
 			)
 		)
-		(property "Footprint" "DIP Switch (10)"
+		(property "Footprint" "FRANK:DIP Switch (10)"
 			(at 213.36 64.77 0)
 			(effects
@@
 			)
 		)
-		(property "Footprint" "DIP Switch (6)"
+		(property "Footprint" "FRANK:DIP Switch (6)"
 			(at 213.36 33.02 0)
 			(effects
