File: hardware/frank_m1/audio.kicad_sch (KiCad schematic)
At the start: 13 parts

Commit message: Fixed tape loading bug on all PCBs
Parts:
- TDA1: footprint FRANK:SOIC-8 -> FRANK:SO-8
Changed lines of the file:
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@@
 	(title_block
 		(title "FRANK M1")
-		(date "2025-03-03")
-		(rev "1.14")
+		(date "2025-03-16")
+		(rev "1.15")
 		(company "Mikhail Matveev")
 		(comment 1 "https://github.com/xtremespb/frank")
@@
 			)
 		)
-		(property "Footprint" "FRANK:SOIC-8"
+		(property "Footprint" "FRANK:SO-8"
 			(at 186.69 59.69 0)
 			(effects

Commit message: Bugfixes
Parts:
- added C21, C24: 10u, FRANK:Capacitor (0805), symbol Device:C
- added C22: 1n, FRANK:Capacitor (0805), symbol Device:C
- added C23: 10u, FRANK:Capacitor (3528, tantalum, polar), symbol Device:C
- added J14: AUDIO, FRANK:RCA, symbol Connector_Generic:Conn_01x02
- added Q3: BC850, FRANK:SOT-23, symbol Transistor_BJT:BC850
- added R61, R62: 10k(3k), FRANK:Resistor (0805), symbol Device:R
- added R63: 47k(10k), FRANK:Resistor (0805), symbol Device:R
- added R64: 20k(2k), Resistor_SMD:R_0805_2012Metric_Pad1.20x1.40mm_HandSolder, symbol Device:R
- added R65: 20K, Resistor_SMD:R_0805_2012Metric_Pad1.20x1.40mm_HandSolder, symbol Device:R
- added R66: 10k, Resistor_SMD:R_0805_2012Metric_Pad1.20x1.40mm_HandSolder, symbol Device:R
- added R67: 200R, FRANK:Resistor (0805), symbol Device:R
Connections:
- net GND: now also C22.2, C24.1, J14.2 (Pin_2), R64.1, R65.1, R67.1
- net VBUS: now also C24.2, Q3.3 (C), R66.1
- new net: C21.1, R61.1, R62.1, R63.1, R64.2
- new net: C21.2, C22.1, Q3.1 (B), R65.2, R66.2
- new net: C23.1, Q3.2 (E), R67.2
- new net BEEP_OUT: R63.2
- new net LEFT_OUT: R62.2
- new net L_OUT: C23.2, J14.1 (Pin_1)
- new net RIGHT_OUT: R61.2

Commit message: FRANK M1 1.16 WIP
Parts:
- removed C21, C24: 10u, FRANK:Capacitor (0805), symbol Device:C
- removed C22: 1n, FRANK:Capacitor (0805), symbol Device:C
- removed C23: 10u, FRANK:Capacitor (3528, tantalum, polar), symbol Device:C
- removed C9: 10u, FRANK:Capacitor (3528, tantalum, polar), symbol Device:C_Polarized
- removed J14: AUDIO, FRANK:RCA, symbol Connector_Generic:Conn_01x02
- removed Q3: BC850, FRANK:SOT-23, symbol Transistor_BJT:BC850
- removed R61, R62: 10k(3k), FRANK:Resistor (0805), symbol Device:R
- removed R63: 47k(10k), FRANK:Resistor (0805), symbol Device:R
- removed R64: 20k(2k), Resistor_SMD:R_0805_2012Metric_Pad1.20x1.40mm_HandSolder, symbol Device:R
- removed R65: 20K, Resistor_SMD:R_0805_2012Metric_Pad1.20x1.40mm_HandSolder, symbol Device:R
- removed R66: 10k, Resistor_SMD:R_0805_2012Metric_Pad1.20x1.40mm_HandSolder, symbol Device:R
- removed R67: 200R, FRANK:Resistor (0805), symbol Device:R
- added C9: 10u, FRANK:Capacitor (0805), symbol Device:C
- renumbered AJ1 to J10, TDA1 to U3
Connections:
- net GND: now also C9.2
- net at U3.7 (FLT): now also C9.1

Commit message: Minor updates
Other:
- moved on the sheet: C10, C11, C7, C8, C9, J10, R22, R23, R24, R25, R26, R27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
