File: hardware/frank_m1/hdmi.kicad_sch (KiCad schematic)
At the start: 10 parts

Commit message: FRANK M1 1.16 WIP
Parts:
- renumbered HDMI1 to J9
Changed lines of the file:
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@@
 	(title_block
 		(title "FRANK M1")
-		(date "2025-03-16")
-		(rev "1.15")
+		(date "2025-03-26")
+		(rev "1.16")
 		(company "Mikhail Matveev")
 		(comment 1 "https://github.com/xtremespb/frank")
@@
 		(dnp no)
 		(fields_autoplaced yes)
-		(property "Reference" "HDMI1"
+		(property "Reference" "J9"
 			(at 43.18 91.4399 0)
 			(effects
@@
 			(project "frank2"
 				(path "/8c0b3d8b-46d3-4173-ab1e-a61765f77d61/db853a64-9343-4a36-b5b8-71001392b936"
-					(reference "HDMI1")
+					(reference "J9")
 					(unit 1)
 				)

Commit message: Minor updates
Other:
- note removed: "HDMI video output requires the resistors to be close to the HDMI socket in order to work properly."
- moved on the sheet: C5, J9, R14, R15, R16, R17, R18, R19, R20, R21
