File: hardware/frank_m1/pico.kicad_sch (KiCad schematic)
At the start: 2 parts

Commit message: FRANK M1 1.16 WIP
Parts:
- renumbered JP2 to JP4, RP1 to U4
Changed lines of the file:
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@@
 	(title_block
 		(title "FRANK M1")
-		(date "2025-03-16")
-		(rev "1.15")
+		(date "2025-03-26")
+		(rev "1.16")
 		(company "Mikhail Matveev")
 		(comment 1 "https://github.com/xtremespb/frank")
@@
 		(dnp no)
 		(fields_autoplaced yes)
-		(property "Reference" "RP1"
+		(property "Reference" "U4"
 			(at 74.93 24.13 0)
 			(effects
@@
 			(project ""
 				(path "/8c0b3d8b-46d3-4173-ab1e-a61765f77d61/8cfcdea6-a6da-4433-b1cd-9be5bedbd2f0"
-					(reference "RP1")
+					(reference "U4")
 					(unit 1)
 				)
@@
 		(on_board yes)
 		(dnp no)
-		(property "Reference" "JP2"
+		(property "Reference" "JP4"
 			(at 120.65 44.45 0)
 			(effects
@@
 			(project "turbofrank"
 				(path "/8c0b3d8b-46d3-4173-ab1e-a61765f77d61/8cfcdea6-a6da-4433-b1cd-9be5bedbd2f0"
-					(reference "JP2")
-					(unit 1)
-				)
+					(reference "JP4")
+					(unit 1)
+				)

Commit message: Minor updates
Other:
- moved on the sheet: JP4, U4
