File: hardware/frank_m1/sd.kicad_sch (KiCad schematic)
At the start: 3 parts

Commit message: FRANK M1 1.16 WIP
Parts:
- renumbered SD1 to J5, SD2 to J6
Changed lines of the file:
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@@
 	(title_block
 		(title "FRANK M1")
-		(date "2025-03-16")
-		(rev "1.15")
+		(date "2025-03-26")
+		(rev "1.16")
 		(company "Mikhail Matveev")
 		(comment 1 "https://github.com/xtremespb/frank")
@@
 		(dnp no)
 		(fields_autoplaced yes)
-		(property "Reference" "#PWR026"
+		(property "Reference" "#PWR027"
 			(at 128.27 57.15 0)
 			(effects
@@
 			(project "core"
 				(path "/8c0b3d8b-46d3-4173-ab1e-a61765f77d61/2e81912e-397c-4129-8da5-abf37a4f2667"
-					(reference "#PWR026")
+					(reference "#PWR027")
 					(unit 1)
 				)
@@
 		(on_board yes)
 		(dnp no)
-		(property "Reference" "#PWR027"
+		(property "Reference" "#PWR028"
 			(at 148.59 53.34 0)
 			(effects
@@
 			(project "core"
 				(path "/8c0b3d8b-46d3-4173-ab1e-a61765f77d61/2e81912e-397c-4129-8da5-abf37a4f2667"
-					(reference "#PWR027")
+					(reference "#PWR028")
 					(unit 1)
 				)
@@
 		(dnp no)
 		(fields_autoplaced yes)
-		(property "Reference" "#PWR025"
+		(property "Reference" "#PWR026"
 			(at 55.88 53.34 0)
 			(effects
@@
 			(project "core"
 				(path "/8c0b3d8b-46d3-4173-ab1e-a61765f77d61/2e81912e-397c-4129-8da5-abf37a4f2667"
-					(reference "#PWR025")
+					(reference "#PWR026")
 					(unit 1)
 				)
@@
 		(dnp no)
 		(fields_autoplaced yes)
-		(property "Reference" "SD1"
+		(property "Reference" "J5"
 			(at 78.74 43.18 0)
 			(effects
@@
 			(project ""
 				(path "/8c0b3d8b-46d3-4173-ab1e-a61765f77d61/2e81912e-397c-4129-8da5-abf37a4f2667"
-					(reference "SD1")
+					(reference "J5")
 					(unit 1)
 				)
@@
 		(dnp no)
 		(fields_autoplaced yes)
-		(property "Reference" "#PWR029"
+		(property "Reference" "#PWR030"
 			(at 101.6 58.42 0)
 			(effects
@@
 			(project "core"
 				(path "/8c0b3d8b-46d3-4173-ab1e-a61765f77d61/2e81912e-397c-4129-8da5-abf37a4f2667"
-					(reference "#PWR029")
+					(reference "#PWR030")
 					(unit 1)
 				)
@@
 		(dnp no)
 		(fields_autoplaced yes)
-		(property "Reference" "#PWR030"
+		(property "Reference" "#PWR031"
 			(at 132.08 99.06 0)
 			(effects
@@
 			(project "turbofrank"
 				(path "/8c0b3d8b-46d3-4173-ab1e-a61765f77d61/2e81912e-397c-4129-8da5-abf37a4f2667"
-					(reference "#PWR030")
+					(reference "#PWR031")
 					(unit 1)
 				)
@@
 		(dnp no)
 		(fields_autoplaced yes)
-		(property "Reference" "SD2"
+		(property "Reference" "J6"
 			(at 161.925 74.93 0)
 			(effects
@@
 			(project "turbofrank"
 				(path "/8c0b3d8b-46d3-4173-ab1e-a61765f77d61/2e81912e-397c-4129-8da5-abf37a4f2667"
-					(reference "SD2")
+					(reference "J6")
 					(unit 1)
 				)
@@
 		(dnp no)
 		(fields_autoplaced yes)
-		(property "Reference" "#PWR028"
+		(property "Reference" "#PWR029"
 			(at 55.88 55.88 0)
 			(effects
@@
 			(project "core"
 				(path "/8c0b3d8b-46d3-4173-ab1e-a61765f77d61/2e81912e-397c-4129-8da5-abf37a4f2667"
-					(reference "#PWR028")
+					(reference "#PWR029")
 					(unit 1)
 				)
@@
 		(dnp no)
 		(fields_autoplaced yes)
-		(property "Reference" "#PWR024"
+		(property "Reference" "#PWR025"
 			(at 55.88 50.8 0)
 			(effects
@@
 			(project ""
 				(path "/8c0b3d8b-46d3-4173-ab1e-a61765f77d61/2e81912e-397c-4129-8da5-abf37a4f2667"
-					(reference "#PWR024")
+					(reference "#PWR025")
 					(unit 1)
 				)

Commit message: Minor updates
Other:
- note removed: "Short TF Card slot is used to save some space on the PCB."
- moved on the sheet: C4, J5, J6
