File: hardware/minifrank_rm24/gamepad.kicad_sch (KiCad schematic)
At the start: 6 parts

Commit message: RM24 WIP
Parts:
- renumbered GP1 to J11
Other:
- moved on the sheet: C28, D5, D6, J11, R35, R36

Commit message: MiniFRANK RM24 1.01
Parts:
- renumbered J11 to J1
Changed lines of the file:
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@@
 	(title_block
 		(title "MiniFRANK RM24")
-		(date "2025-03-14")
-		(rev "1.00")
+		(date "2025-04-09")
+		(rev "${VERSION}")
 		(company "Mikhail Matveev")
 		(comment 1 "https://github.com/xtremespb/frank")
@@
 		(on_board yes)
 		(dnp no)
-		(property "Reference" "J11"
+		(property "Reference" "J1"
 			(at 171.45 67.31 0)
 			(effects
@@
 			(project "valera-2350A"
 				(path "/8c0b3d8b-46d3-4173-ab1e-a61765f77d61/e3bc68fc-1a90-4165-9d37-467f5079ac2b"
-					(reference "J11")
-					(unit 1)
-				)
+					(reference "J1")
+					(unit 1)
+				)
