File: hardware/minifrank_rm24/hdmi.kicad_sch (KiCad schematic)
At the start: 10 parts

Commit message: RM24 WIP
Parts:
- renumbered HDMI1 to J8
Other:
- moved on the sheet: C26, J8, R27, R28, R29, R30, R31, R32, R33, R34
