File: hardware/minifrank_rm24/tape.kicad_sch (KiCad schematic)
At the start: 11 parts, among them Q1 BC850, Q2 BC850

Commit message: RM24 WIP
Parts:
- C35: renamed from C1; LCSC (none) -> C1711
- C36: renamed from C2; LCSC (none) -> C1711
- D7: renamed from D1; LCSC (none) -> C5443967
- J4: renamed from AJ1; value PJ-325C -> PJ-320D; footprint FRANK:Jack (3.5mm) -> FRANK:Jack (3.5mm, PJ-320D); AliExpress https://www.aliexpress.com/item/1005006710837751.html -> https://www.aliexpress.com/item/4001158231104.html; LCSC (none) -> C95562
- Q1, Q2: AliExpress https://www.aliexpress.com/item/33017911878.html -> https://www.aliexpress.com/item/1005005008637286.html; LCSC (none) -> C78484
- R59: renamed from R1; LCSC (none) -> C17414
- R60: renamed from R2; AliExpress https://www.vishay.com/docs/28952/mcs0402at-mct0603at-mcu08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 -> https://www.aliexpress.com/item/1005005945735199.html; LCSC (none) -> C17513
- R61: renamed from R3; LCSC (none) -> C17414
- R62: renamed from R4; LCSC (none) -> C17414
- R63: renamed from R5; LCSC (none) -> C3152174
Connections:
- net LOAD_IN: no longer C36.1, J4.T, R63.1
- new net: C36.1, J4.T, R63.1
- no-connect marks 3 -> 1
Other:
- title: Frank M2 -> MiniFRANK RM1

Commit message: MiniFRANK RM24 1.01
Other:
- title: MiniFRANK RM1 -> MiniFRANK RM24
Changed lines of the file:
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@@
 	(paper "A4")
 	(title_block
-		(title "MiniFRANK RM1")
-		(date "2025-04-07")
+		(title "MiniFRANK RM24")
+		(date "2025-04-09")
 		(rev "${VERSION}")
 		(company "Mikhail Matveev")
