File: hardware/minifrank_rm24/usb_hub.kicad_sch (KiCad schematic)
At the start: 2 parts, among them U7 MW7211A

Commit message: MiniFRANK RM24 1.01
Other:
- title: MiniFRANK RM1 -> MiniFRANK RM24
Changed lines of the file:
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@@
 	(paper "A4")
 	(title_block
-		(title "MiniFRANK RM1")
-		(date "2025-04-07")
+		(title "MiniFRANK RM24")
+		(date "2025-04-09")
 		(rev "${VERSION}")
 		(company "Mikhail Matveev")
