File: hardware/minifrank_rm24/usbstack.kicad_sch (KiCad schematic)
At the start: 0 parts

Commit message: RM24 WIP
Parts:
- added C38, C39: 10u, FRANK:Capacitor (0805), symbol Device:C
- added J6: SS-52100-004, FRANK:USB Type A (stacked), symbol Connector:USB_A_Stacked
- added R55, R56, R57, R58: 22R, FRANK:Resistor (0805), symbol Device:R
Connections:
- new net: J6.2 (D1-), R56.2
- new net: J6.3 (D1+), R55.2
- new net: J6.6 (D2-), R58.2
- new net: J6.7 (D2+), R57.2
- new net D1+: R55.1
- new net D1-: R56.1
- new net D2+: R57.1
- new net D2-: R58.1
- new net GND: C38.2, C39.2, J6.4 (GND1), J6.8 (GND2), J6.9 (Shield)
- new net VBUS: C38.1, C39.1, J6.1 (VBUS1), J6.5 (VBUS2)
Other:
- company: (none) -> Mikhail Matveev
- title: (none) -> MiniFRANK RM1

Commit message: MiniFRANK RM24 1.01
Other:
- title: MiniFRANK RM1 -> MiniFRANK RM24
Changed lines of the file:
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@@
 	(paper "A4")
 	(title_block
-		(title "MiniFRANK RM1")
-		(date "2025-04-07")
+		(title "MiniFRANK RM24")
+		(date "2025-04-09")
 		(rev "${VERSION}")
 		(company "Mikhail Matveev")
