File: lab/minifrank_rm1e/minifrank_rm1e.kicad_pcb (KiCad board)
At the start: 2 copper layers, 85.6 x 54 mm, 135 parts, among them J10 USB4215-03-A, J2 0475710001, J3 104031-0811, J4 PJ-320D, J5 PJ-320D, J6 D-SUB 9 Male, J7 MDC-036, J8 DC3RX19JA2, J9 SS-52100-004, Q1 BC850, Q2 BC850, U1 NCP1117 3.3, U2 W25Q128JVSIQ, U3 RP2040, U4 ESP-PSRAM32, U5 LM358, U6 TDA1387T, U7 MW7211A, U8 74HC4052D,653, Y1 12 MHz

Commit message: WIP
Parts:
- moved C4 1.46 mm to (214.7, 100.8)
- moved C3 0.85 mm to (214.8, 105.6)
- moved C14 0.41 mm to (212.3, 105.6)
- moved C10 0.36 mm to (212.3, 106.8)
- moved C11 0.30 mm to (212.3, 101.8)
Routing:
- net Net-(C29-Pad1): track 0.00 -> 80.3 mm, vias 0 -> 4
- net /Audio Out/AMP_OUTL: track 0.00 -> 68.1 mm, vias 0 -> 6
- net Net-(U5A--): track 0.00 -> 65.4 mm, vias 0 -> 4
- net /MS_DATA_3V: track 0.00 -> 64.1 mm, vias 0 -> 4
- net /MS_CLK_3V: track 0.00 -> 61.9 mm, vias 0 -> 4
- net /PWM_OUT_L: track 0.00 -> 51.5 mm, vias 0 -> 2
- net Net-(J6-Pad2): track 0.00 -> 46.0 mm, vias 0 -> 1
- net /GPIO28: track 40.6 -> 82.9 mm, vias 2 -> 6
- net Net-(C32-Pad1): track 0.00 -> 40.8 mm, vias 0 -> 2
- net /AMP_IN_R: track 0.00 -> 38.6 mm, vias 0 -> 2
- net Net-(C26-Pad2): track 0.00 -> 34.9 mm, vias 0 -> 2
- net Net-(C20-Pad1): track 0.00 -> 34.6 mm, vias 0 -> 2
- net /PS2/MS_CLK: track 0.00 -> 33.8 mm, vias 0 -> 2
- net /GPIO14: track 26.7 -> 60.0 mm, vias 0 -> 2
- net /KB_DATA: track 0.00 -> 33.2 mm, vias 0 -> 2
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
Commit message: Update minifrank_rm1e.kicad_pcb
Routing:
- net /GPIO22: track 27.1 -> 28.6 mm
- net /TDA_L: track 20.7 -> 21.7 mm
- net /KB_CLK: track 29.6 -> 30.5 mm
- net Net-(J10-CC2): track 5.66 -> 6.63 mm
- net /RP2040/QSPI_SD3: track 13.8 -> 14.7 mm
- net /RP2040/QSPI_SD1: track 26.8 -> 27.5 mm
- net VBUS: track 276.4 -> 277.0 mm
- net /RUN: track 48.4 -> 48.9 mm
Other:
- board text added: "ASW"
- board text added: "BOOT"
- board text added: "MCK"
- board text added: "MDA"
- board text added: "RESET"
- board text added: "TIN"
