File: lab/minifrank_rm1e/hdmi.kicad_sch (KiCad schematic)
At the start: 10 parts, among them J8 DC3RX19JA2

Commit message: Experimental boards added
Other:
- title: MiniFRANK RM1E -> ${NAME}
Changed lines of the file:
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@@
 	(paper "A4")
 	(title_block
-		(title "MiniFRANK RM1E")
-		(date "2025-04-15")
+		(title "${NAME}")
+		(date "2025-04-16")
 		(rev "${VERSION}")
 		(company "Mikhail Matveev")
