File: lab/minifrank_rm1e/power.kicad_sch (KiCad schematic)
At the start: 9 parts, among them J10 USB4215-03-A, U1 NCP1117 3.3

Commit message: Experimental boards added
Other:
- title: MiniFRANK RM1E -> ${NAME}
Changed lines of the file:
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@@
 	(paper "A4")
 	(title_block
-		(title "MiniFRANK RM1E")
-		(date "2025-04-15")
+		(title "${NAME}")
+		(date "2025-04-16")
 		(rev "${VERSION}")
 		(company "Mikhail Matveev")
