File: lab/picofrank2/rp2350a.kicad_sch (KiCad schematic)
At the start: 33 parts, among them U2 RP2350, U3 ESP-PSRAM32, U4 W25Q128JVS, Y1 ASE-12MHz

Commit message: PicoFRANK2 WIP
Changed lines of the file:
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@@
 	(wire
 		(pts
-			(xy 214.63 134.62) (xy 246.38 134.62)
+			(xy 214.63 134.62) (xy 229.87 134.62)
 		)
 		(stroke
@@
 		)
 	)
-	(label "GPIO25"
-		(at 246.38 134.62 180)
-		(effects
-			(font
-				(size 1.27 1.27)
-			)
-			(justify right bottom)
-		)
-	)
 	(label "QSPI_SD0"
 		(at 106.68 171.45 180)
@@
 		(effects
 			(font
+				(size 1.27 1.27)
+			)
+			(justify left)
+		)
+	)
+	(hierarchical_label "GPIO25"
+		(shape input)
+		(at 229.87 134.62 0)
+		(effects
+			(font
