File: hardware/protea/rp2040.kicad_sch (KiCad schematic)
At the start: 25 parts, among them SW1 Flash Button, Y1 12 MHz

Commit message: Minor updates
Parts:
- removed SW1: Flash Button, FRANK:Button (SMD, 3x3mm), symbol Switch:SW_Push_Dual
- added S2: TS-1233, FRANK:Button (SMD, 3x3mm, 1-1), symbol Switch:SW_Push
- renumbered C1 to C11, C2 to C12, C3 to C13, C4 to C14, C5 to C15, C6 to C16, C7 to C17, C8 to C18, C9 to C19, C10 to C20, C11 to C21, C12 to C22, C13 to C23, C14 to C24, C15 to C25, L1 to LD2, R1 to R31, R2 to R32, R3 to R33, R4 to R34, R5 to R35, FL1 to U3, RP1 to U4
Connections:
- net GND: now also S2.1
- net ~{USB_BOOT}: now also S2.2
Other:
- title: Protea -> MiniFRANK RM1E
- moved on the sheet: C24, C25, LD2, R34, R35, Y1

Commit message: Cleanup
Parts:
- removed S2: TS-1233, FRANK:Button (SMD, 3x3mm, 1-1), symbol Switch:SW_Push
- added S3: Boot, FRANK:Button (SMD, 3x3mm, 1-1), symbol Switch:SW_Push
- LD2: value Blue -> BLUE
- renumbered C18 to C10, C19 to C11, C20 to C12, C21 to C13, C22 to C14, C23 to C15, C24 to C16, C25 to C17, C11 to C3, C12 to C4, C13 to C5, C14 to C6, C15 to C7, C16 to C8, C17 to C9, R31 to R5, R32 to R6, R33 to R7, R34 to R8, R35 to R9, U3 to U2, U4 to U3
Connections:
- net GND: now also S3.2
- net ~{USB_BOOT}: no longer names the net of R6.2
- net ~{USB_BOOT}: now also S3.1
Other:
- title: MiniFRANK RM1E -> Protea
- moved on the sheet: C16, C17, LD2, R8, R9, Y1

Commit message: Bugfixes
Other:
- title: Protea -> ${NAME}
Changed lines of the file:
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@@
 	(paper "A4")
 	(title_block
-		(title "Protea")
-		(date "2025-04-03")
-		(rev "2.04")
+		(title "${NAME}")
+		(date "2025-04-21")
+		(rev "${VERSION}")
 		(company "Mikhail Matveev")
 		(comment 1 "https://github.com/xtremespb/frank")
