File: hardware/protea/rs232.kicad_sch (KiCad schematic)
At the start: 10 parts

Commit message: Cleanup
Parts:
- renumbered C19 to C18, C20 to C19, C21 to C20, C22 to C21, D3 to D1, D4 to D2, COM1 to J2, R13 to R10, R14 to R11, MAX1 to U4
Connections:
- net VBUS renamed RS232_VBUS

Commit message: Bugfixes
Other:
- title: Protea -> ${NAME}
Changed lines of the file:
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@@
 	(paper "A4")
 	(title_block
-		(title "Protea")
-		(date "2025-04-03")
-		(rev "2.04")
+		(title "${NAME}")
+		(date "2025-04-21")
+		(rev "${VERSION}")
 		(company "Mikhail Matveev")
 		(comment 1 "https://github.com/xtremespb/frank")
