File: lab/nyx2/rp2350a.kicad_sch (KiCad schematic)
At the start: 33 parts, among them U2 RP2350, U3 ESP-PSRAM32, U4 W25Q128JVS, Y1 ASE-12MHz

Commit message: Experimental boards added
Other:
- title: MiniFRANK RM24 -> ${NAME}
Changed lines of the file:
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@@
 	(paper "A4")
 	(title_block
-		(title "MiniFRANK RM24")
-		(date "2025-04-09")
+		(title "${NAME}")
+		(date "2025-04-16")
 		(rev "${VERSION}")
 		(company "Mikhail Matveev")

Commit message: Nyx2 HW 1.03
Parts:
- C12: renamed from C14; footprint FRANK:Capacitor (0402) -> FRANK:Capacitor (0805)
- C13: renamed from C15; footprint FRANK:Capacitor (0402) -> FRANK:Capacitor (0805)
- C14: renamed from C16; footprint FRANK:Capacitor (0402) -> FRANK:Capacitor (0805)
- C2: renamed from C4; footprint FRANK:Capacitor (0402) -> FRANK:Capacitor (0805)
- L1: footprint FRANK:Inductor (3225) -> FRANK:IND_LQH2MCN100K02L
- R9: renamed from R13; value 0 -> 0R
- renumbered C3 to C1, C12 to C10, C13 to C11, C17 to C15, C18 to C16, C5 to C3, C6 to C4, C7 to C5, C8 to C6, C9 to C7, C10 to C8, C11 to C9, LD2 to LD1, R5 to R1, R14 to R10, R6 to R2, R7 to R3, R8 to R4, R9 to R5, R10 to R6, R11 to R7, R12 to R8, U2 to U1, U3 to U2, U4 to U3
