File: lab/minifrank_rm2/audio.kicad_sch (KiCad schematic)
At the start: 1 part, among them J2 PJ-320D

Commit message: MiniFRANK RM2 1.02
Parts:
- J2: LCSC C95562 -> (none)
Changed lines of the file:
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@@
 			)
 		)
-		(property "LCSC" "C95562"
+		(property "LCSC" ""
 			(at 212.09 66.04 0)
 			(effects
