File: hardware/frank_m2/HR3FQ.kicad_sch (KiCad schematic)
At the start: 7 parts, among them CON1 Pin Header 1x03, CON2 Pin Header 1x03, J1 Pin Header 2x18

Commit message: Minor updates
Parts:
- renumbered CON1 to J1, CON2 to J2, J1 to JP1
Changed lines of the file:
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@@
 		(dnp no)
 		(fields_autoplaced yes)
-		(property "Reference" "CON1"
+		(property "Reference" "J1"
 			(at 212.725 71.12 0)
 			(effects
@@
 			(project ""
 				(path "/8c0b3d8b-46d3-4173-ab1e-a61765f77d61"
-					(reference "CON1")
+					(reference "J1")
 					(unit 1)
 				)
@@
 		(dnp no)
 		(fields_autoplaced yes)
-		(property "Reference" "J1"
+		(property "Reference" "JP1"
 			(at 212.09 21.59 0)
 			(effects
@@
 			(project "HR3FQ"
 				(path "/8c0b3d8b-46d3-4173-ab1e-a61765f77d61"
-					(reference "J1")
+					(reference "JP1")
 					(unit 1)
 				)
@@
 		(dnp no)
 		(fields_autoplaced yes)
-		(property "Reference" "CON2"
+		(property "Reference" "J2"
 			(at 212.725 86.36 0)
 			(effects
@@
 			(project "turbofrank"
 				(path "/8c0b3d8b-46d3-4173-ab1e-a61765f77d61"
-					(reference "CON2")
-					(unit 1)
-				)
+					(reference "J2")
+					(unit 1)
+				)
