File: hardware/frank_m2/composite.kicad_sch (KiCad schematic)
At the start: 16 parts

Commit message: Minor updates
Parts:
- renumbered C16 to C15, SC1 to J15
Other:
- moved on the sheet: C15, J15, R45, R46, R47, R48, R49, R50, R51, R52, R53, R54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
