File: hardware/frank_m2/gamepad.kicad_sch (KiCad schematic)
At the start: 3 parts

Commit message: Minor updates
Parts:
- renumbered GP1 to J7
Other:
- note removed: "The gamepad uses standard DB9 male socket."
- moved on the sheet: D5, J7, R12
