File: hardware/frank_m2/power.kicad_sch (KiCad schematic)
At the start: 8 parts, among them U1 NCP1117 3.3

Commit message: Minor updates
Parts:
- renumbered USB1 to J3, L1 to LD1
Other:
- note removed: "The LED indicates +3V power availability. Usually it's green, but you decide ;-)"
- note removed: "The power source is USB-C connector. The NCP1117 transforms +5V to +3V3."
- moved on the sheet: C1, C2, LD1, R1, R2, R3, U1
