File: hardware/frank_m2/sd.kicad_sch (KiCad schematic)
At the start: 3 parts

Commit message: Minor updates
Parts:
- renumbered SD1 to J5, SD2 to J6
Other:
- note removed: "Short TF Card slot is used to save some space on the PCB."
- moved on the sheet: C4, J5, J6
